Commit message: move ar3 meshes and add ar4 meshes

File: ar_description/urdf/ar3.urdf (robot description, URDF)
Before this commit: robot ar3, 7 links, 6 joints
Links:
- link base_link: geometry collision mesh filename=package://ar_description/meshes/ar3/base_link.STL; visual mesh filename=package://ar_description/meshes/ar3/base_link.STL
- link link_1: geometry collision mesh filename=package://ar_description/meshes/ar3/link_1.STL; visual mesh filename=package://ar_description/meshes/ar3/link_1.STL
- link link_2: geometry collision mesh filename=package://ar_description/meshes/ar3/link_2.STL; visual mesh filename=package://ar_description/meshes/ar3/link_2.STL
- link link_3: geometry collision mesh filename=package://ar_description/meshes/ar3/link_3.STL; visual mesh filename=package://ar_description/meshes/ar3/link_3.STL
- link link_4: geometry collision mesh filename=package://ar_description/meshes/ar3/link_4.STL; visual mesh filename=package://ar_description/meshes/ar3/link_4.STL
- link link_5: geometry collision mesh filename=package://ar_description/meshes/ar3/link_5.STL; visual mesh filename=package://ar_description/meshes/ar3/link_5.STL
- link link_6: geometry collision mesh filename=package://ar_description/meshes/ar3/link_6.STL; visual mesh filename=package://ar_description/meshes/ar3/link_6.STL

File: ar_description/urdf/ar3.urdf.xacro (robot description, xacro)
@@ -14,14 +14,14 @@
       <origin rpy="0 0 0" xyz="0 0 0"/>
       <geometry>
-        <mesh filename="package://ar_description/meshes/base_link.STL"/>
-      </geometry>
-      <material name="">
-        <color rgba="1 1 0 1"/>
-      </material>
-    </visual>
-    <collision>
-      <origin rpy="0 0 0" xyz="0 0 0"/>
-      <geometry>
-        <mesh filename="package://ar_description/meshes/base_link.STL"/>
+        <mesh filename="package://ar_description/meshes/ar3/base_link.STL"/>
+      </geometry>
+      <material name="">
+        <color rgba="1 1 0 1"/>
+      </material>
+    </visual>
+    <collision>
+      <origin rpy="0 0 0" xyz="0 0 0"/>
+      <geometry>
+        <mesh filename="package://ar_description/meshes/ar3/base_link.STL"/>
       </geometry>
     </collision>
@@ -36,14 +36,14 @@
       <origin rpy="0 0 0" xyz="0 0 0"/>
       <geometry>
-        <mesh filename="package://ar_description/meshes/link_1.STL"/>
-      </geometry>
-      <material name="">
-        <color rgba="1 1 0 1"/>
-      </material>
-    </visual>
-    <collision>
-      <origin rpy="0 0 0" xyz="0 0 0"/>
-      <geometry>
-        <mesh filename="package://ar_description/meshes/link_1.STL"/>
+        <mesh filename="package://ar_description/meshes/ar3/link_1.STL"/>
+      </geometry>
+      <material name="">
+        <color rgba="1 1 0 1"/>
+      </material>
+    </visual>
+    <collision>
+      <origin rpy="0 0 0" xyz="0 0 0"/>
+      <geometry>
+        <mesh filename="package://ar_description/meshes/ar3/link_1.STL"/>
       </geometry>
     </collision>
@@ -65,14 +65,14 @@
       <origin rpy="0 0 0" xyz="0 0 0"/>
       <geometry>
-        <mesh filename="package://ar_description/meshes/link_2.STL"/>
-      </geometry>
-      <material name="">
-        <color rgba="1 1 0 1"/>
-      </material>
-    </visual>
-    <collision>
-      <origin rpy="0 0 0" xyz="0 0 0"/>
-      <geometry>
-        <mesh filename="package://ar_description/meshes/link_2.STL"/>
+        <mesh filename="package://ar_description/meshes/ar3/link_2.STL"/>
+      </geometry>
+      <material name="">
+        <color rgba="1 1 0 1"/>
+      </material>
+    </visual>
+    <collision>
+      <origin rpy="0 0 0" xyz="0 0 0"/>
+      <geometry>
+        <mesh filename="package://ar_description/meshes/ar3/link_2.STL"/>
       </geometry>
     </collision>
@@ -94,14 +94,14 @@
       <origin rpy="0 0 0" xyz="0 0 0"/>
       <geometry>
-        <mesh filename="package://ar_description/meshes/link_3.STL"/>
-      </geometry>
-      <material name="">
-        <color rgba="1 1 0 1"/>
-      </material>
-    </visual>
-    <collision>
-      <origin rpy="0 0 0" xyz="0 0 0"/>
-      <geometry>
-        <mesh filename="package://ar_description/meshes/link_3.STL"/>
+        <mesh filename="package://ar_description/meshes/ar3/link_3.STL"/>
+      </geometry>
+      <material name="">
+        <color rgba="1 1 0 1"/>
+      </material>
+    </visual>
+    <collision>
+      <origin rpy="0 0 0" xyz="0 0 0"/>
+      <geometry>
+        <mesh filename="package://ar_description/meshes/ar3/link_3.STL"/>
       </geometry>
     </collision>
@@ -123,14 +123,14 @@
       <origin rpy="0 0 0" xyz="0 0 0"/>
       <geometry>
-        <mesh filename="package://ar_description/meshes/link_4.STL"/>
-      </geometry>
-      <material name="">
-        <color rgba="1 1 0 1"/>
-      </material>
-    </visual>
-    <collision>
-      <origin rpy="0 0 0" xyz="0 0 0"/>
-      <geometry>
-        <mesh filename="package://ar_description/meshes/link_4.STL"/>
+        <mesh filename="package://ar_description/meshes/ar3/link_4.STL"/>
+      </geometry>
+      <material name="">
+        <color rgba="1 1 0 1"/>
+      </material>
+    </visual>
+    <collision>
+      <origin rpy="0 0 0" xyz="0 0 0"/>
+      <geometry>
+        <mesh filename="package://ar_description/meshes/ar3/link_4.STL"/>
       </geometry>
     </collision>
@@ -152,14 +152,14 @@
       <origin rpy="0 0 0" xyz="0 0 0"/>
       <geometry>
-        <mesh filename="package://ar_description/meshes/link_5.STL"/>
-      </geometry>
-      <material name="">
-        <color rgba="1 1 0 1"/>
-      </material>
-    </visual>
-    <collision>
-      <origin rpy="0 0 0" xyz="0 0 0"/>
-      <geometry>
-        <mesh filename="package://ar_description/meshes/link_5.STL"/>
+        <mesh filename="package://ar_description/meshes/ar3/link_5.STL"/>
+      </geometry>
+      <material name="">
+        <color rgba="1 1 0 1"/>
+      </material>
+    </visual>
+    <collision>
+      <origin rpy="0 0 0" xyz="0 0 0"/>
+      <geometry>
+        <mesh filename="package://ar_description/meshes/ar3/link_5.STL"/>
       </geometry>
     </collision>
@@ -181,14 +181,14 @@
       <origin rpy="0 0 0" xyz="0 0 0"/>
       <geometry>
-        <mesh filename="package://ar_description/meshes/link_6.STL"/>
-      </geometry>
-      <material name="">
-        <color rgba="1 1 0 1"/>
-      </material>
-    </visual>
-    <collision>
-      <origin rpy="0 0 0" xyz="0 0 0"/>
-      <geometry>
-        <mesh filename="package://ar_description/meshes/link_6.STL"/>
+        <mesh filename="package://ar_description/meshes/ar3/link_6.STL"/>
+      </geometry>
+      <material name="">
+        <color rgba="1 1 0 1"/>
+      </material>
+    </visual>
+    <collision>
+      <origin rpy="0 0 0" xyz="0 0 0"/>
+      <geometry>
+        <mesh filename="package://ar_description/meshes/ar3/link_6.STL"/>
       </geometry>
     </collision>

File: ar_description/urdf/ar3_gazebo.urdf.xacro (robot description, xacro)
@@ -15,14 +15,14 @@
       <origin rpy="0 0 0" xyz="0 0 0"/>
       <geometry>
-        <mesh filename="package://ar_description/meshes/base_link.STL"/>
-      </geometry>
-      <material name="">
-        <color rgba="1 1 0 1"/>
-      </material>
-    </visual>
-    <collision>
-      <origin rpy="0 0 0" xyz="0 0 0"/>
-      <geometry>
-        <mesh filename="package://ar_description/meshes/base_link.STL"/>
+        <mesh filename="package://ar_description/meshes/ar3/base_link.STL"/>
+      </geometry>
+      <material name="">
+        <color rgba="1 1 0 1"/>
+      </material>
+    </visual>
+    <collision>
+      <origin rpy="0 0 0" xyz="0 0 0"/>
+      <geometry>
+        <mesh filename="package://ar_description/meshes/ar3/base_link.STL"/>
       </geometry>
     </collision>
@@ -42,14 +42,14 @@
       <origin rpy="0 0 0" xyz="0 0 0"/>
       <geometry>
-        <mesh filename="package://ar_description/meshes/link_1.STL"/>
-      </geometry>
-      <material name="">
-        <color rgba="1 1 0 1"/>
-      </material>
-    </visual>
-    <collision>
-      <origin rpy="0 0 0" xyz="0 0 0"/>
-      <geometry>
-        <mesh filename="package://ar_description/meshes/link_1.STL"/>
+        <mesh filename="package://ar_description/meshes/ar3/link_1.STL"/>
+      </geometry>
+      <material name="">
+        <color rgba="1 1 0 1"/>
+      </material>
+    </visual>
+    <collision>
+      <origin rpy="0 0 0" xyz="0 0 0"/>
+      <geometry>
+        <mesh filename="package://ar_description/meshes/ar3/link_1.STL"/>
       </geometry>
     </collision>
@@ -71,14 +71,14 @@
       <origin rpy="0 0 0" xyz="0 0 0"/>
       <geometry>
-        <mesh filename="package://ar_description/meshes/link_2.STL"/>
-      </geometry>
-      <material name="">
-        <color rgba="1 1 0 1"/>
-      </material>
-    </visual>
-    <collision>
-      <origin rpy="0 0 0" xyz="0 0 0"/>
-      <geometry>
-        <mesh filename="package://ar_description/meshes/link_2.STL"/>
+        <mesh filename="package://ar_description/meshes/ar3/link_2.STL"/>
+      </geometry>
+      <material name="">
+        <color rgba="1 1 0 1"/>
+      </material>
+    </visual>
+    <collision>
+      <origin rpy="0 0 0" xyz="0 0 0"/>
+      <geometry>
+        <mesh filename="package://ar_description/meshes/ar3/link_2.STL"/>
       </geometry>
     </collision>
@@ -100,14 +100,14 @@
       <origin rpy="0 0 0" xyz="0 0 0"/>
       <geometry>
-        <mesh filename="package://ar_description/meshes/link_3.STL"/>
-      </geometry>
-      <material name="">
-        <color rgba="1 1 0 1"/>
-      </material>
-    </visual>
-    <collision>
-      <origin rpy="0 0 0" xyz="0 0 0"/>
-      <geometry>
-        <mesh filename="package://ar_description/meshes/link_3.STL"/>
+        <mesh filename="package://ar_description/meshes/ar3/link_3.STL"/>
+      </geometry>
+      <material name="">
+        <color rgba="1 1 0 1"/>
+      </material>
+    </visual>
+    <collision>
+      <origin rpy="0 0 0" xyz="0 0 0"/>
+      <geometry>
+        <mesh filename="package://ar_description/meshes/ar3/link_3.STL"/>
       </geometry>
     </collision>
@@ -129,14 +129,14 @@
       <origin rpy="0 0 0" xyz="0 0 0"/>
       <geometry>
-        <mesh filename="package://ar_description/meshes/link_4.STL"/>
-      </geometry>
-      <material name="">
-        <color rgba="1 1 0 1"/>
-      </material>
-    </visual>
-    <collision>
-      <origin rpy="0 0 0" xyz="0 0 0"/>
-      <geometry>
-        <mesh filename="package://ar_description/meshes/link_4.STL"/>
+        <mesh filename="package://ar_description/meshes/ar3/link_4.STL"/>
+      </geometry>
+      <material name="">
+        <color rgba="1 1 0 1"/>
+      </material>
+    </visual>
+    <collision>
+      <origin rpy="0 0 0" xyz="0 0 0"/>
+      <geometry>
+        <mesh filename="package://ar_description/meshes/ar3/link_4.STL"/>
       </geometry>
     </collision>
@@ -158,14 +158,14 @@
       <origin rpy="0 0 0" xyz="0 0 0"/>
       <geometry>
-        <mesh filename="package://ar_description/meshes/link_5.STL"/>
-      </geometry>
-      <material name="">
-        <color rgba="1 1 0 1"/>
-      </material>
-    </visual>
-    <collision>
-      <origin rpy="0 0 0" xyz="0 0 0"/>
-      <geometry>
-        <mesh filename="package://ar_description/meshes/link_5.STL"/>
+        <mesh filename="package://ar_description/meshes/ar3/link_5.STL"/>
+      </geometry>
+      <material name="">
+        <color rgba="1 1 0 1"/>
+      </material>
+    </visual>
+    <collision>
+      <origin rpy="0 0 0" xyz="0 0 0"/>
+      <geometry>
+        <mesh filename="package://ar_description/meshes/ar3/link_5.STL"/>
       </geometry>
     </collision>
@@ -187,14 +187,14 @@
       <origin rpy="0 0 0" xyz="0 0 0"/>
       <geometry>
-        <mesh filename="package://ar_description/meshes/link_6.STL"/>
-      </geometry>
-      <material name="">
-        <color rgba="1 1 0 1"/>
-      </material>
-    </visual>
-    <collision>
-      <origin rpy="0 0 0" xyz="0 0 0"/>
-      <geometry>
-        <mesh filename="package://ar_description/meshes/link_6.STL"/>
+        <mesh filename="package://ar_description/meshes/ar3/link_6.STL"/>
+      </geometry>
+      <material name="">
+        <color rgba="1 1 0 1"/>
+      </material>
+    </visual>
+    <collision>
+      <origin rpy="0 0 0" xyz="0 0 0"/>
+      <geometry>
+        <mesh filename="package://ar_description/meshes/ar3/link_6.STL"/>
       </geometry>
     </collision>
