Commit message: fix a couple of warnings

File: ar_description/urdf/ar3.urdf.xacro (robot description, xacro)
@@ -4,200 +4,207 @@
 <!-- |    EDITING THIS FILE BY HAND IS NOT RECOMMENDED                                 | -->
 <!-- =================================================================================== -->
-<robot name="ar3">
-  <link name="base_link">
-    <inertial>
-      <origin rpy="0 0 0" xyz="-4.6941E-06 0.054174 0.038824"/>
-      <mass value="0.7102"/>
-      <inertia ixx="0.0039943" ixy="3.697E-07" ixz="-5.7364E-08" iyy="0.0014946" iyz="-0.00036051" izz="0.0042554"/>
-    </inertial>
-    <visual>
-      <origin rpy="0 0 0" xyz="0 0 0"/>
-      <geometry>
-        <mesh filename="package://ar_description/meshes/ar3/base_link.STL"/>
-      </geometry>
-      <material name="">
-        <color rgba="1 1 0 1"/>
-      </material>
-    </visual>
-    <collision>
-      <origin rpy="0 0 0" xyz="0 0 0"/>
-      <geometry>
-        <mesh filename="package://ar_description/meshes/ar3/base_link.STL"/>
-      </geometry>
-    </collision>
-  </link>
-  <link name="link_1">
-    <inertial>
-      <origin rpy="0 0 0" xyz="-0.022706 0.04294 -0.12205"/>
-      <mass value="0.88065"/>
-      <inertia ixx="0.0034" ixy="0.00042296" ixz="-0.00089231" iyy="0.0041778" iyz="0.0010848" izz="0.0027077"/>
-    </inertial>
-    <visual>
-      <origin rpy="0 0 0" xyz="0 0 0"/>
-      <geometry>
-        <mesh filename="package://ar_description/meshes/ar3/link_1.STL"/>
-      </geometry>
-      <material name="">
-        <color rgba="1 1 0 1"/>
-      </material>
-    </visual>
-    <collision>
-      <origin rpy="0 0 0" xyz="0 0 0"/>
-      <geometry>
-        <mesh filename="package://ar_description/meshes/ar3/link_1.STL"/>
-      </geometry>
-    </collision>
-  </link>
-  <joint name="joint_1" type="revolute">
-    <origin rpy="${pi} 0 0" xyz="0 0 0.003445"/>
-    <parent link="base_link"/>
-    <child link="link_1"/>
-    <axis xyz="0 0 1"/>
-    <limit lower="-2.96706" upper="2.96706" effort="0" velocity="0"/>
-  </joint>
-  <link name="link_2">
-    <inertial>
-      <origin rpy="0 0 0" xyz="0.064818 -0.11189 -0.038671"/>
-      <mass value="0.57738"/>
-      <inertia ixx="0.0047312" ixy="0.0022624" ixz="0.00032144" iyy="0.0020836" iyz="-0.00056569" izz="0.0056129"/>
-    </inertial>
-    <visual>
-      <origin rpy="0 0 0" xyz="0 0 0"/>
-      <geometry>
-        <mesh filename="package://ar_description/meshes/ar3/link_2.STL"/>
-      </geometry>
-      <material name="">
-        <color rgba="1 1 0 1"/>
-      </material>
-    </visual>
-    <collision>
-      <origin rpy="0 0 0" xyz="0 0 0"/>
-      <geometry>
-        <mesh filename="package://ar_description/meshes/ar3/link_2.STL"/>
-      </geometry>
-    </collision>
-  </link>
-  <joint name="joint_2" type="revolute">
-    <origin rpy="1.5708 0.5236 -1.5708" xyz="0 0.064146 -0.16608"/>
-    <parent link="link_1"/>
-    <child link="link_2"/>
-    <axis xyz="0 0 -1"/>
-    <limit lower="${-39.6 / 180.0 * pi}" upper="${pi / 2.0}" effort="0" velocity="0"/>
-  </joint>
-  <link name="link_3">
-    <inertial>
-      <origin rpy="0 0 0" xyz="-0.00029765 -0.023661 -0.0019125"/>
-      <mass value="0.1787"/>
-      <inertia ixx="0.0001685" ixy="-2.7713E-05" ixz="5.6885E-06" iyy="0.00012865" iyz="2.9256E-05" izz="0.00020744"/>
-    </inertial>
-    <visual>
-      <origin rpy="0 0 0" xyz="0 0 0"/>
-      <geometry>
-        <mesh filename="package://ar_description/meshes/ar3/link_3.STL"/>
-      </geometry>
-      <material name="">
-        <color rgba="1 1 0 1"/>
-      </material>
-    </visual>
-    <collision>
-      <origin rpy="0 0 0" xyz="0 0 0"/>
-      <geometry>
-        <mesh filename="package://ar_description/meshes/ar3/link_3.STL"/>
-      </geometry>
-    </collision>
-  </link>
-  <joint name="joint_3" type="revolute">
-    <origin rpy="0 0 -1.04720367321" xyz="0.1525 -0.26414 0"/>
-    <parent link="link_2"/>
-    <child link="link_3"/>
-    <axis xyz="0 0 -1"/>
-    <limit lower="0.0174533" upper="2.5080381" effort="0" velocity="0"/>
-  </joint>
-  <link name="link_4">
-    <inertial>
-      <origin rpy="0 0 0" xyz="-0.0016798 -0.00057319 -0.074404"/>
-      <mass value="0.34936"/>
-      <inertia ixx="0.0030532" ixy="-1.8615E-05" ixz="-7.0047E-05" iyy="0.0031033" iyz="-2.3301E-05" izz="0.00022264"/>
-    </inertial>
-    <visual>
-      <origin rpy="0 0 0" xyz="0 0 0"/>
-      <geometry>
-        <mesh filename="package://ar_description/meshes/ar3/link_4.STL"/>
-      </geometry>
-      <material name="">
-        <color rgba="1 1 0 1"/>
-      </material>
-    </visual>
-    <collision>
-      <origin rpy="0 0 0" xyz="0 0 0"/>
-      <geometry>
-        <mesh filename="package://ar_description/meshes/ar3/link_4.STL"/>
-      </geometry>
-    </collision>
-  </link>
-  <joint name="joint_4" type="revolute">
-    <origin rpy="1.5708 -1.2554 -1.5708" xyz="0 0 0.00675"/>
-    <parent link="link_3"/>
-    <child link="link_4"/>
-    <axis xyz="0 0 -1"/>
-    <limit lower="-2.8710666" upper="2.8710666" effort="0" velocity="0"/>
-  </joint>
-  <link name="link_5">
-    <inertial>
-      <origin rpy="0 0 0" xyz="0.0015066 -1.3102E-05 -0.012585"/>
-      <mass value="0.11562"/>
-      <inertia ixx="5.5035E-05" ixy="-1.019E-08" ixz="-2.6243E-06" iyy="8.2921E-05" iyz="1.4437E-08" izz="5.2518E-05"/>
-    </inertial>
-    <visual>
-      <origin rpy="0 0 0" xyz="0 0 0"/>
-      <geometry>
-        <mesh filename="package://ar_description/meshes/ar3/link_5.STL"/>
-      </geometry>
-      <material name="">
-        <color rgba="1 1 0 1"/>
-      </material>
-    </visual>
-    <collision>
-      <origin rpy="0 0 0" xyz="0 0 0"/>
-      <geometry>
-        <mesh filename="package://ar_description/meshes/ar3/link_5.STL"/>
-      </geometry>
-    </collision>
-  </link>
-  <joint name="joint_5" type="revolute">
-    <origin rpy="${pi} 0 -2.8262" xyz="0 0 -0.22225"/>
-    <parent link="link_4"/>
-    <child link="link_5"/>
-    <axis xyz="1 0 0"/>
-    <limit lower="-1.81776042" upper="1.81776042" effort="0" velocity="0"/>
-  </joint>
-  <link name="link_6">
-    <inertial>
-      <origin rpy="0 0 0" xyz="2.9287E-10 -1.6472E-09 0.0091432"/>
-      <mass value="0.013863"/>
-      <inertia ixx="1.3596E-06" ixy="3.0585E-13" ixz="5.7102E-14" iyy="1.7157E-06" iyz="6.3369E-09" izz="2.4332E-06"/>
-    </inertial>
-    <visual>
-      <origin rpy="0 0 0" xyz="0 0 0"/>
-      <geometry>
-        <mesh filename="package://ar_description/meshes/ar3/link_6.STL"/>
-      </geometry>
-      <material name="">
-        <color rgba="1 1 0 1"/>
-      </material>
-    </visual>
-    <collision>
-      <origin rpy="0 0 0" xyz="0 0 0"/>
-      <geometry>
-        <mesh filename="package://ar_description/meshes/ar3/link_6.STL"/>
-      </geometry>
-    </collision>
-  </link>
-  <joint name="joint_6" type="revolute">
-    <origin rpy="0 0 3.1416" xyz="-0.000294 0 0.02117"/>
-    <parent link="link_5"/>
-    <child link="link_6"/>
-    <axis xyz="0 0 1"/>
-    <limit lower="-2.5848326" upper="2.5848326" effort="0" velocity="0"/>
-  </joint>
+<robot xmlns:xacro="http://wiki.ros.org/xacro">
+  <xacro:macro name="ar3_robot" params="parent *origin">
+    <joint name="base_joint" type="fixed">
+      <xacro:insert_block name="origin" />
+      <parent link="${parent}"/>
+      <child link="base_link" />
+    </joint>
+    <link name="base_link">
+      <inertial>
+        <origin rpy="0 0 0" xyz="-4.6941E-06 0.054174 0.038824"/>
+        <mass value="0.7102"/>
+        <inertia ixx="0.0039943" ixy="3.697E-07" ixz="-5.7364E-08" iyy="0.0014946" iyz="-0.00036051" izz="0.0042554"/>
+      </inertial>
+      <visual>
+        <origin rpy="0 0 0" xyz="0 0 0"/>
+        <geometry>
+          <mesh filename="package://ar_description/meshes/ar3/base_link.STL"/>
+        </geometry>
+        <material name="">
+          <color rgba="1 1 0 1"/>
+        </material>
+      </visual>
+      <collision>
+        <origin rpy="0 0 0" xyz="0 0 0"/>
+        <geometry>
+          <mesh filename="package://ar_description/meshes/ar3/base_link.STL"/>
+        </geometry>
+      </collision>
+    </link>
+    <link name="link_1">
+      <inertial>
+        <origin rpy="0 0 0" xyz="-0.022706 0.04294 -0.12205"/>
+        <mass value="0.88065"/>
+        <inertia ixx="0.0034" ixy="0.00042296" ixz="-0.00089231" iyy="0.0041778" iyz="0.0010848" izz="0.0027077"/>
+      </inertial>
+      <visual>
+        <origin rpy="0 0 0" xyz="0 0 0"/>
+        <geometry>
+          <mesh filename="package://ar_description/meshes/ar3/link_1.STL"/>
+        </geometry>
+        <material name="">
+          <color rgba="1 1 0 1"/>
+        </material>
+      </visual>
+      <collision>
+        <origin rpy="0 0 0" xyz="0 0 0"/>
+        <geometry>
+          <mesh filename="package://ar_description/meshes/ar3/link_1.STL"/>
+        </geometry>
+      </collision>
+    </link>
+    <joint name="joint_1" type="revolute">
+      <origin rpy="${pi} 0 0" xyz="0 0 0.003445"/>
+      <parent link="base_link"/>
+      <child link="link_1"/>
+      <axis xyz="0 0 1"/>
+      <limit lower="-2.96706" upper="2.96706" effort="0" velocity="0"/>
+    </joint>
+    <link name="link_2">
+      <inertial>
+        <origin rpy="0 0 0" xyz="0.064818 -0.11189 -0.038671"/>
+        <mass value="0.57738"/>
+        <inertia ixx="0.0047312" ixy="0.0022624" ixz="0.00032144" iyy="0.0020836" iyz="-0.00056569" izz="0.0056129"/>
+      </inertial>
+      <visual>
+        <origin rpy="0 0 0" xyz="0 0 0"/>
+        <geometry>
+          <mesh filename="package://ar_description/meshes/ar3/link_2.STL"/>
+        </geometry>
+        <material name="">
+          <color rgba="1 1 0 1"/>
+        </material>
+      </visual>
+      <collision>
+        <origin rpy="0 0 0" xyz="0 0 0"/>
+        <geometry>
+          <mesh filename="package://ar_description/meshes/ar3/link_2.STL"/>
+        </geometry>
+      </collision>
+    </link>
+    <joint name="joint_2" type="revolute">
+      <origin rpy="1.5708 0.5236 -1.5708" xyz="0 0.064146 -0.16608"/>
+      <parent link="link_1"/>
+      <child link="link_2"/>
+      <axis xyz="0 0 -1"/>
+      <limit lower="${-39.6 / 180.0 * pi}" upper="${pi / 2.0}" effort="0" velocity="0"/>
+    </joint>
+    <link name="link_3">
+      <inertial>
+        <origin rpy="0 0 0" xyz="-0.00029765 -0.023661 -0.0019125"/>
+        <mass value="0.1787"/>
+        <inertia ixx="0.0001685" ixy="-2.7713E-05" ixz="5.6885E-06" iyy="0.00012865" iyz="2.9256E-05" izz="0.00020744"/>
+      </inertial>
+      <visual>
+        <origin rpy="0 0 0" xyz="0 0 0"/>
+        <geometry>
+          <mesh filename="package://ar_description/meshes/ar3/link_3.STL"/>
+        </geometry>
+        <material name="">
+          <color rgba="1 1 0 1"/>
+        </material>
+      </visual>
+      <collision>
+        <origin rpy="0 0 0" xyz="0 0 0"/>
+        <geometry>
+          <mesh filename="package://ar_description/meshes/ar3/link_3.STL"/>
+        </geometry>
+      </collision>
+    </link>
+    <joint name="joint_3" type="revolute">
+      <origin rpy="0 0 -1.04720367321" xyz="0.1525 -0.26414 0"/>
+      <parent link="link_2"/>
+      <child link="link_3"/>
+      <axis xyz="0 0 -1"/>
+      <limit lower="0.0174533" upper="2.5080381" effort="0" velocity="0"/>
+    </joint>
+    <link name="link_4">
+      <inertial>
+        <origin rpy="0 0 0" xyz="-0.0016798 -0.00057319 -0.074404"/>
+        <mass value="0.34936"/>
+        <inertia ixx="0.0030532" ixy="-1.8615E-05" ixz="-7.0047E-05" iyy="0.0031033" iyz="-2.3301E-05" izz="0.00022264"/>
+      </inertial>
+      <visual>
+        <origin rpy="0 0 0" xyz="0 0 0"/>
+        <geometry>
+          <mesh filename="package://ar_description/meshes/ar3/link_4.STL"/>
+        </geometry>
+        <material name="">
+          <color rgba="1 1 0 1"/>
+        </material>
+      </visual>
+      <collision>
+        <origin rpy="0 0 0" xyz="0 0 0"/>
+        <geometry>
+          <mesh filename="package://ar_description/meshes/ar3/link_4.STL"/>
+        </geometry>
+      </collision>
+    </link>
+    <joint name="joint_4" type="revolute">
+      <origin rpy="1.5708 -1.2554 -1.5708" xyz="0 0 0.00675"/>
+      <parent link="link_3"/>
+      <child link="link_4"/>
+      <axis xyz="0 0 -1"/>
+      <limit lower="-2.8710666" upper="2.8710666" effort="0" velocity="0"/>
+    </joint>
+    <link name="link_5">
+      <inertial>
+        <origin rpy="0 0 0" xyz="0.0015066 -1.3102E-05 -0.012585"/>
+        <mass value="0.11562"/>
+        <inertia ixx="5.5035E-05" ixy="-1.019E-08" ixz="-2.6243E-06" iyy="8.2921E-05" iyz="1.4437E-08" izz="5.2518E-05"/>
+      </inertial>
+      <visual>
+        <origin rpy="0 0 0" xyz="0 0 0"/>
+        <geometry>
+          <mesh filename="package://ar_description/meshes/ar3/link_5.STL"/>
+        </geometry>
+        <material name="">
+          <color rgba="1 1 0 1"/>
+        </material>
+      </visual>
+      <collision>
+        <origin rpy="0 0 0" xyz="0 0 0"/>
+        <geometry>
+          <mesh filename="package://ar_description/meshes/ar3/link_5.STL"/>
+        </geometry>
+      </collision>
+    </link>
+    <joint name="joint_5" type="revolute">
+      <origin rpy="${pi} 0 -2.8262" xyz="0 0 -0.22225"/>
+      <parent link="link_4"/>
+      <child link="link_5"/>
+      <axis xyz="1 0 0"/>
+      <limit lower="-1.81776042" upper="1.81776042" effort="0" velocity="0"/>
+    </joint>
+    <link name="link_6">
+      <inertial>
+        <origin rpy="0 0 0" xyz="2.9287E-10 -1.6472E-09 0.0091432"/>
+        <mass value="0.013863"/>
+        <inertia ixx="1.3596E-06" ixy="3.0585E-13" ixz="5.7102E-14" iyy="1.7157E-06" iyz="6.3369E-09" izz="2.4332E-06"/>
+      </inertial>
+      <visual>
+        <origin rpy="0 0 0" xyz="0 0 0"/>
+        <geometry>
+          <mesh filename="package://ar_description/meshes/ar3/link_6.STL"/>
+        </geometry>
+        <material name="">
+          <color rgba="1 1 0 1"/>
+        </material>
+      </visual>
+      <collision>
+        <origin rpy="0 0 0" xyz="0 0 0"/>
+        <geometry>
+          <mesh filename="package://ar_description/meshes/ar3/link_6.STL"/>
+        </geometry>
+      </collision>
+    </link>
+    <joint name="joint_6" type="revolute">
+      <origin rpy="0 0 3.1416" xyz="-0.000294 0 0.02117"/>
+      <parent link="link_5"/>
+      <child link="link_6"/>
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
File: ar_hardware_interface/urdf/ar3.urdf.xacro (robot description, xacro)
@@ -9,4 +9,8 @@
   <!-- convert to property to use substitution in function -->
   <xacro:property name="initial_positions_file" default="$(arg initial_positions_file)"/>
+  <link name="world" />
+  <xacro:ar3_robot parent="world">
+    <origin xyz="0 0 0" rpy="0 0 0" />
+  </xacro:ar3_robot>
   <xacro:ar_ros2_control name="$(arg name)"/>
 </robot>
