Commit message: robot showing in rviz and accepting plans

File: ar_description/urdf/ar3_macro.xacro (robot description, xacro)
@@ -56,5 +56,5 @@
       <child link="link_1"/>
       <axis xyz="0 0 1"/>
-      <limit lower="-2.96706" upper="2.96706" effort="0" velocity="0"/>
+      <limit lower="-2.96706" upper="2.96706" effort="0" velocity="0.5" acceleration="0.5"/>
     </joint>
     <link name="link_2">
@@ -85,5 +85,5 @@
       <child link="link_2"/>
       <axis xyz="0 0 -1"/>
-      <limit lower="${-39.6 / 180.0 * pi}" upper="${pi / 2.0}" effort="0" velocity="0"/>
+      <limit lower="${-39.6 / 180.0 * pi}" upper="${pi / 2.0}" effort="0.5" velocity="0" acceleration="0.5"/>
     </joint>
     <link name="link_3">
@@ -114,5 +114,5 @@
       <child link="link_3"/>
       <axis xyz="0 0 -1"/>
-      <limit lower="0.0174533" upper="2.5080381" effort="0" velocity="0"/>
+      <limit lower="0.0174533" upper="2.5080381" effort="0" velocity="0.5" acceleration="0.5"/>
     </joint>
     <link name="link_4">
@@ -143,5 +143,5 @@
       <child link="link_4"/>
       <axis xyz="0 0 -1"/>
-      <limit lower="-2.8710666" upper="2.8710666" effort="0" velocity="0"/>
+      <limit lower="-2.8710666" upper="2.8710666" effort="0" velocity="0.5" acceleration="0.5"/>
     </joint>
     <link name="link_5">
@@ -172,5 +172,5 @@
       <child link="link_5"/>
       <axis xyz="1 0 0"/>
-      <limit lower="-1.81776042" upper="1.81776042" effort="0" velocity="0"/>
+      <limit lower="-1.81776042" upper="1.81776042" effort="0" velocity="0.5" acceleration="0.5"/>
     </joint>
     <link name="link_6">
@@ -201,5 +201,5 @@
       <child link="link_6"/>
       <axis xyz="0 0 1"/>
-      <limit lower="-2.5848326" upper="2.5848326" effort="0" velocity="0"/>
+      <limit lower="-2.5848326" upper="2.5848326" effort="0" velocity="0.5" acceleration="0.5"/>
     </joint>
   </xacro:macro>

Commit message: working movement in rviz

File: ar_description/urdf/ar3_macro.xacro (robot description, xacro)
@@ -56,5 +56,5 @@
       <child link="link_1"/>
       <axis xyz="0 0 1"/>
-      <limit lower="-2.96706" upper="2.96706" effort="0" velocity="0.5" acceleration="0.5"/>
+      <limit lower="${-170.0 / 180.0 * pi}" upper="${170.0 / 180.0 * pi}" effort="0" velocity="0.5"/>
     </joint>
     <link name="link_2">
@@ -85,5 +85,5 @@
       <child link="link_2"/>
       <axis xyz="0 0 -1"/>
-      <limit lower="${-39.6 / 180.0 * pi}" upper="${pi / 2.0}" effort="0.5" velocity="0" acceleration="0.5"/>
+      <limit lower="${-42.0 / 180.0 * pi}" upper="${90.0 / 180.0 * pi}" effort="0.5" velocity="0"/>
     </joint>
     <link name="link_3">
@@ -110,9 +110,9 @@
     </link>
     <joint name="joint_3" type="revolute">
-      <origin rpy="0 0 -1.04720367321" xyz="0.1525 -0.26414 0"/>
+      <origin rpy="0 0 -2.61799" xyz="0.1525 -0.26414 0"/>
       <parent link="link_2"/>
       <child link="link_3"/>
       <axis xyz="0 0 -1"/>
-      <limit lower="0.0174533" upper="2.5080381" effort="0" velocity="0.5" acceleration="0.5"/>
+      <limit lower="${-89.0 / 180.0 * pi}" upper="${52.0 / 180.0 * pi}" effort="0" velocity="0.5"/>
     </joint>
     <link name="link_4">
@@ -143,5 +143,5 @@
       <child link="link_4"/>
       <axis xyz="0 0 -1"/>
-      <limit lower="-2.8710666" upper="2.8710666" effort="0" velocity="0.5" acceleration="0.5"/>
+      <limit lower="${-165.0 / 180.0 * pi}" upper="${165.0 / 180.0 * pi}" effort="0" velocity="0.5"/>
     </joint>
     <link name="link_5">
@@ -172,5 +172,5 @@
       <child link="link_5"/>
       <axis xyz="1 0 0"/>
-      <limit lower="-1.81776042" upper="1.81776042" effort="0" velocity="0.5" acceleration="0.5"/>
+      <limit lower="${-105.0 / 180.0 * pi}" upper="${105.0 / 180.0 * pi}" effort="0" velocity="0.5"/>
     </joint>
     <link name="link_6">
@@ -201,5 +201,5 @@
       <child link="link_6"/>
       <axis xyz="0 0 1"/>
-      <limit lower="-2.5848326" upper="2.5848326" effort="0" velocity="0.5" acceleration="0.5"/>
+      <limit lower="${-155.0 / 180.0 * pi}" upper="${155.0 / 180.0 * pi}" effort="0" velocity="0.5"/>
     </joint>
   </xacro:macro>
