Commit message: working gazebo simulation

File: ar_description/urdf/ar_gazebo.urdf.xacro (robot description, xacro)
@@ -1,294 +1,22 @@
-<?xml version="1.0" encoding="utf-8"?>
-<!-- =================================================================================== -->
-<!-- |    This document was autogenerated by xacro from ar4.urdf                       | -->
-<!-- |    EDITING THIS FILE BY HAND IS NOT RECOMMENDED but it was unfortunately        | -->
-<!-- =================================================================================== -->
-<robot name="ar">
+<?xml version="1.0"?>
+<robot xmlns:xacro="http://wiki.ros.org/xacro" name="$(arg name)">
+  <xacro:include filename="$(find ar_description)/urdf/ar_macro.xacro"/>
+  <xacro:include filename="$(find ar_description)/urdf/ar.ros2_control.xacro"/>
+  <xacro:arg name="simulation_controllers" default="" />
   <link name="world" />
-  <link name="base_link">
-    <inertial>
-      <origin rpy="0 0 0" xyz="-4.6941E-06 0.054174 0.038824"/>
-      <mass value="0.7102"/>
-      <inertia ixx="0.0039943" ixy="3.697E-07" ixz="-5.7364E-08" iyy="0.0014946" iyz="-0.00036051" izz="0.0042554"/>
-    </inertial>
-    <visual>
-      <origin rpy="0 0 0" xyz="0 0 0"/>
-      <geometry>
-        <mesh filename="package://ar_description/meshes/ar4/base_link.STL"/>
-      </geometry>
-      <material name="">
-        <color rgba="1 1 0 1"/>
-      </material>
-    </visual>
-    <collision>
-      <origin rpy="0 0 0" xyz="0 0 0"/>
-      <geometry>
-        <mesh filename="package://ar_description/meshes/ar4/base_link.STL"/>
-      </geometry>
-    </collision>
-  </link>
-  <joint name="joint_world" type="fixed">
-    <parent link="world"/>
-    <child link="base_link"/>
+  <xacro:ar_robot parent="world">
     <origin xyz="0 0 0" rpy="0 0 0" />
-  </joint>
-  <link name="link_1">
-    <inertial>
-      <origin rpy="0 0 0" xyz="-0.022706 0.04294 -0.12205"/>
-      <mass value="0.88065"/>
-      <inertia ixx="0.0034" ixy="0.00042296" ixz="-0.00089231" iyy="0.0041778" iyz="0.0010848" izz="0.0027077"/>
-    </inertial>
-    <visual>
-      <origin rpy="0 0 0" xyz="0 0 0"/>
-      <geometry>
-        <mesh filename="package://ar_description/meshes/ar4/link_1.STL"/>
-      </geometry>
-      <material name="">
-        <color rgba="1 1 0 1"/>
-      </material>
-    </visual>
-    <collision>
-      <origin rpy="0 0 0" xyz="0 0 0"/>
-      <geometry>
-        <mesh filename="package://ar_description/meshes/ar4/link_1.STL"/>
-      </geometry>
-    </collision>
-  </link>
-  <joint name="joint_1" type="revolute">
-    <origin rpy="${pi} 0 0" xyz="0 0 0.003445"/>
-    <parent link="base_link"/>
-    <child link="link_1"/>
-    <axis xyz="0 0 1"/>
-    <limit lower="-2.96706" upper="2.96706" effort="100" velocity="100"/>
-  </joint>
-  <link name="link_2">
-    <inertial>
-      <origin rpy="0 0 0" xyz="0.064818 -0.11189 -0.038671"/>
-      <mass value="0.57738"/>
-      <inertia ixx="0.0047312" ixy="0.0022624" ixz="0.00032144" iyy="0.0020836" iyz="-0.00056569" izz="0.0056129"/>
-    </inertial>
-    <visual>
-      <origin rpy="0 0 0" xyz="0 0 0"/>
-      <geometry>
-        <mesh filename="package://ar_description/meshes/ar4/link_2.STL"/>
-      </geometry>
-      <material name="">
-        <color rgba="1 1 0 1"/>
-      </material>
-    </visual>
-    <collision>
-      <origin rpy="0 0 0" xyz="0 0 0"/>
-      <geometry>
-        <mesh filename="package://ar_description/meshes/ar4/link_2.STL"/>
-      </geometry>
-    </collision>
-  </link>
-  <joint name="joint_2" type="revolute">
-    <origin rpy="1.5708 0.5236 -1.5708" xyz="0 0.064146 -0.16608"/>
-    <parent link="link_1"/>
-    <child link="link_2"/>
-    <axis xyz="0 0 -1"/>
-    <limit lower="${-39.6 / 180.0 * pi}" upper="${pi / 2.0}" effort="100" velocity="100"/>
-  </joint>
-  <link name="link_3">
-    <inertial>
-      <origin rpy="0 0 0" xyz="-0.00029765 -0.023661 -0.0019125"/>
-      <mass value="0.1787"/>
-      <inertia ixx="0.0001685" ixy="-2.7713E-05" ixz="5.6885E-06" iyy="0.00012865" iyz="2.9256E-05" izz="0.00020744"/>
-    </inertial>
-    <visual>
-      <origin rpy="0 0 0" xyz="0 0 0"/>
-      <geometry>
-        <mesh filename="package://ar_description/meshes/ar4/link_3.STL"/>
-      </geometry>
-      <material name="">
-        <color rgba="1 1 0 1"/>
-      </material>
-    </visual>
-    <collision>
-      <origin rpy="0 0 0" xyz="0 0 0"/>
-      <geometry>
-        <mesh filename="package://ar_description/meshes/ar4/link_3.STL"/>
-      </geometry>
-    </collision>
-  </link>
-  <joint name="joint_3" type="revolute">
-    <origin rpy="0 0 -1.04720367321" xyz="0.1525 -0.26414 0"/>
-    <parent link="link_2"/>
-    <child link="link_3"/>
-    <axis xyz="0 0 -1"/>
-    <limit lower="0.0174533" upper="2.5080381" effort="100" velocity="100"/>
-  </joint>
-  <link name="link_4">
-    <inertial>
-      <origin rpy="0 0 0" xyz="-0.0016798 -0.00057319 -0.074404"/>
-      <mass value="0.34936"/>
-      <inertia ixx="0.0030532" ixy="-1.8615E-05" ixz="-7.0047E-05" iyy="0.0031033" iyz="-2.3301E-05" izz="0.00022264"/>
-    </inertial>
-    <visual>
-      <origin rpy="0 0 0" xyz="0 0 0"/>
-      <geometry>
-        <mesh filename="package://ar_description/meshes/ar4/link_4.STL"/>
-      </geometry>
-      <material name="">
-        <color rgba="1 1 0 1"/>
-      </material>
-    </visual>
-    <collision>
-      <origin rpy="0 0 0" xyz="0 0 0"/>
-      <geometry>
-        <mesh filename="package://ar_description/meshes/ar4/link_4.STL"/>
-      </geometry>
-    </collision>
-  </link>
-  <joint name="joint_4" type="revolute">
-    <origin rpy="1.5708 -1.2554 -1.5708" xyz="0 0 0.00675"/>
-    <parent link="link_3"/>
-    <child link="link_4"/>
-    <axis xyz="0 0 -1"/>
-    <limit lower="-2.8710666" upper="2.8710666" effort="100" velocity="100"/>
-  </joint>
-  <link name="link_5">
-    <inertial>
-      <origin rpy="0 0 0" xyz="0.0015066 -1.3102E-05 -0.012585"/>
-      <mass value="0.11562"/>
-      <inertia ixx="5.5035E-05" ixy="-1.019E-08" ixz="-2.6243E-06" iyy="8.2921E-05" iyz="1.4437E-08" izz="5.2518E-05"/>
-    </inertial>
-    <visual>
-      <origin rpy="0 0 0" xyz="0 0 0"/>
-      <geometry>
-        <mesh filename="package://ar_description/meshes/ar4/link_5.STL"/>
-      </geometry>
-      <material name="">
-        <color rgba="1 1 0 1"/>
-      </material>
-    </visual>
-    <collision>
-      <origin rpy="0 0 0" xyz="0 0 0"/>
-      <geometry>
-        <mesh filename="package://ar_description/meshes/ar4/link_5.STL"/>
-      </geometry>
-    </collision>
-  </link>
-  <joint name="joint_5" type="revolute">
-    <origin rpy="${pi} 0 -2.8262" xyz="0 0 -0.22225"/>
-    <parent link="link_4"/>
-    <child link="link_5"/>
-    <axis xyz="1 0 0"/>
-    <limit lower="-1.81776042" upper="1.81776042" effort="100" velocity="100"/>
-  </joint>
-  <link name="link_6">
-    <inertial>
-      <origin rpy="0 0 0" xyz="2.9287E-10 -1.6472E-09 0.0091432"/>
-      <mass value="0.013863"/>
-      <inertia ixx="1.3596E-06" ixy="3.0585E-13" ixz="5.7102E-14" iyy="1.7157E-06" iyz="6.3369E-09" izz="2.4332E-06"/>
-    </inertial>
-    <visual>
-      <origin rpy="0 0 0" xyz="0 0 0"/>
-      <geometry>
-        <mesh filename="package://ar_description/meshes/ar4/link_6.STL"/>
-      </geometry>
-      <material name="">
-        <color rgba="1 1 0 1"/>
-      </material>
-    </visual>
-    <collision>
-      <origin rpy="0 0 0" xyz="0 0 0"/>
-      <geometry>
-        <mesh filename="package://ar_description/meshes/ar4/link_6.STL"/>
-      </geometry>
-    </collision>
-  </link>
-  <joint name="joint_6" type="revolute">
-    <origin rpy="0 0 3.1416" xyz="-0.000294 0 0.02117"/>
-    <parent link="link_5"/>
-    <child link="link_6"/>
-    <axis xyz="0 0 1"/>
-    <limit lower="-2.5848326" upper="2.5848326" effort="100" velocity="100"/>
-  </joint>
-  <transmission name="transmission_1">
-    <type>transmission_interface/SimpleTransmission</type>
-    <joint name="joint_1">
-        <hardwareInterface>hardware_interface/PositionJointInterface</hardwareInterface>
-    </joint>
-    <actuator name="motor_1">
-        <hardwareInterface>hardware_interface/PositionJointInterface</hardwareInterface>
-        <mechanicalReduction>1</mechanicalReduction>
-    </actuator>
-  </transmission>
-  <transmission name="transmission_2">
-      <type>transmission_interface/SimpleTransmission</type>
-      <joint name="joint_2">
-          <hardwareInterface>hardware_interface/PositionJointInterface</hardwareInterface>
-      </joint>
-      <actuator name="motor_2">
-          <hardwareInterface>hardware_interface/PositionJointInterface</hardwareInterface>
-          <mechanicalReduction>1</mechanicalReduction>
-      </actuator>
-  </transmission>
-  <transmission name="transmission_3">
-      <type>transmission_interface/SimpleTransmission</type>
-      <joint name="joint_3">
-          <hardwareInterface>hardware_interface/PositionJointInterface</hardwareInterface>
-      </joint>
-      <actuator name="motor_3">
-          <hardwareInterface>hardware_interface/PositionJointInterface</hardwareInterface>
-          <mechanicalReduction>1</mechanicalReduction>
-      </actuator>
-  </transmission>
-  <transmission name="transmission_4">
-      <type>transmission_interface/SimpleTransmission</type>
-      <joint name="joint_4">
-          <hardwareInterface>hardware_interface/PositionJointInterface</hardwareInterface>
-      </joint>
-      <actuator name="motor_4">
-          <hardwareInterface>hardware_interface/PositionJointInterface</hardwareInterface>
-          <mechanicalReduction>1</mechanicalReduction>
-      </actuator>
-  </transmission>
-  <transmission name="transmission_5">
-      <type>transmission_interface/SimpleTransmission</type>
-      <joint name="joint_5">
-          <hardwareInterface>hardware_interface/PositionJointInterface</hardwareInterface>
-      </joint>
-      <actuator name="motor_5">
-          <hardwareInterface>hardware_interface/PositionJointInterface</hardwareInterface>
-          <mechanicalReduction>1</mechanicalReduction>
-      </actuator>
-  </transmission>
-  <transmission name="transmission_6">
-      <type>transmission_interface/SimpleTransmission</type>
-      <joint name="joint_6">
-          <hardwareInterface>hardware_interface/PositionJointInterface</hardwareInterface>
-      </joint>
-      <actuator name="motor_6">
-          <hardwareInterface>hardware_interface/PositionJointInterface</hardwareInterface>
-          <mechanicalReduction>1</mechanicalReduction>
-      </actuator>
-  </transmission>
+  </xacro:ar_robot>
+  <xacro:ar_ros2_control
+    name="$(arg name)"
+    plugin_name="gazebo_ros2_control/GazeboSystem"
+    serial_port="None"
+    calibrate="False"
+  />
+  <gazebo reference="world" />
   <gazebo>
-    <plugin name="gazebo_ros2_control" filename="libgazebo_ros2_control.so">
+    <plugin filename="libgazebo_ros2_control.so" name="gazebo_ros2_control">
+      <parameters>$(arg simulation_controllers)</parameters>
     </plugin>
   </gazebo>
-  <gazebo reference="base_link">
-      <selfCollide>true</selfCollide>
-  </gazebo>
-  <gazebo reference="link_1">
-      <selfCollide>true</selfCollide>
-  </gazebo>
-  <gazebo reference="link_2">
-      <selfCollide>true</selfCollide>
-  </gazebo>
-  <gazebo reference="link_3">
-      <selfCollide>true</selfCollide>
-  </gazebo>
-  <gazebo reference="link_4">
-      <selfCollide>true</selfCollide>
-  </gazebo>
-  <gazebo reference="link_5">
-      <selfCollide>true</selfCollide>
-  </gazebo>
-  <gazebo reference="link_6">
-      <selfCollide>true</selfCollide>
-  </gazebo>
 </robot>

File: ar_description/urdf/ar_macro.xacro (robot description, xacro)
@@ -16,14 +16,14 @@
         <origin rpy="0 0 0" xyz="0 0 0"/>
         <geometry>
-          <mesh filename="package://ar_description/meshes/ar4/base_link.STL"/>
-        </geometry>
-        <material name="">
-          <color rgba="1 1 0 1"/>
-        </material>
-      </visual>
-      <collision>
-        <origin rpy="0 0 0" xyz="0 0 0"/>
-        <geometry>
-          <mesh filename="package://ar_description/meshes/ar4/base_link.STL"/>
+          <mesh filename="file://$(find ar_description)/meshes/ar4/base_link.STL"/>
+        </geometry>
+        <material name="">
+          <color rgba="1 1 0 1"/>
+        </material>
+      </visual>
+      <collision>
+        <origin rpy="0 0 0" xyz="0 0 0"/>
+        <geometry>
+          <mesh filename="file://$(find ar_description)/meshes/ar4/base_link.STL"/>
         </geometry>
       </collision>
@@ -38,14 +38,14 @@
         <origin rpy="0 0 0" xyz="0 0 0"/>
         <geometry>
-          <mesh filename="package://ar_description/meshes/ar4/link_1.STL"/>
-        </geometry>
-        <material name="">
-          <color rgba="1 1 0 1"/>
-        </material>
-      </visual>
-      <collision>
-        <origin rpy="0 0 0" xyz="0 0 0"/>
-        <geometry>
-          <mesh filename="package://ar_description/meshes/ar4/link_1.STL"/>
+          <mesh filename="file://$(find ar_description)/meshes/ar4/link_1.STL"/>
+        </geometry>
+        <material name="">
+          <color rgba="1 1 0 1"/>
+        </material>
+      </visual>
+      <collision>
+        <origin rpy="0 0 0" xyz="0 0 0"/>
+        <geometry>
+          <mesh filename="file://$(find ar_description)/meshes/ar4/link_1.STL"/>
         </geometry>
       </collision>
@@ -67,14 +67,14 @@
         <origin rpy="0 0 0" xyz="0 0 0"/>
         <geometry>
-          <mesh filename="package://ar_description/meshes/ar4/link_2.STL"/>
-        </geometry>
-        <material name="">
-          <color rgba="1 1 0 1"/>
-        </material>
-      </visual>
-      <collision>
-        <origin rpy="0 0 0" xyz="0 0 0"/>
-        <geometry>
-          <mesh filename="package://ar_description/meshes/ar4/link_2.STL"/>
+          <mesh filename="file://$(find ar_description)/meshes/ar4/link_2.STL"/>
+        </geometry>
+        <material name="">
+          <color rgba="1 1 0 1"/>
+        </material>
+      </visual>
+      <collision>
+        <origin rpy="0 0 0" xyz="0 0 0"/>
+        <geometry>
+          <mesh filename="file://$(find ar_description)/meshes/ar4/link_2.STL"/>
         </geometry>
       </collision>
@@ -96,14 +96,14 @@
         <origin rpy="0 0 0" xyz="0 0 0"/>
         <geometry>
-          <mesh filename="package://ar_description/meshes/ar4/link_3.STL"/>
-        </geometry>
-        <material name="">
-          <color rgba="1 1 0 1"/>
-        </material>
-      </visual>
-      <collision>
-        <origin rpy="0 0 0" xyz="0 0 0"/>
-        <geometry>
-          <mesh filename="package://ar_description/meshes/ar4/link_3.STL"/>
+          <mesh filename="file://$(find ar_description)/meshes/ar4/link_3.STL"/>
+        </geometry>
+        <material name="">
+          <color rgba="1 1 0 1"/>
+        </material>
+      </visual>
+      <collision>
+        <origin rpy="0 0 0" xyz="0 0 0"/>
+        <geometry>
+          <mesh filename="file://$(find ar_description)/meshes/ar4/link_3.STL"/>
         </geometry>
       </collision>
@@ -125,14 +125,14 @@
         <origin rpy="0 0 0" xyz="0 0 0"/>
         <geometry>
-          <mesh filename="package://ar_description/meshes/ar4/link_4.STL"/>
-        </geometry>
-        <material name="">
-          <color rgba="1 1 0 1"/>
-        </material>
-      </visual>
-      <collision>
-        <origin rpy="0 0 0" xyz="0 0 0"/>
-        <geometry>
-          <mesh filename="package://ar_description/meshes/ar4/link_4.STL"/>
+          <mesh filename="file://$(find ar_description)/meshes/ar4/link_4.STL"/>
+        </geometry>
+        <material name="">
+          <color rgba="1 1 0 1"/>
+        </material>
+      </visual>
+      <collision>
+        <origin rpy="0 0 0" xyz="0 0 0"/>
+        <geometry>
+          <mesh filename="file://$(find ar_description)/meshes/ar4/link_4.STL"/>
         </geometry>
       </collision>
@@ -154,14 +154,14 @@
         <origin rpy="0 0 0" xyz="0 0 0"/>
         <geometry>
-          <mesh filename="package://ar_description/meshes/ar4/link_5.STL"/>
-        </geometry>
-        <material name="">
-          <color rgba="1 1 0 1"/>
-        </material>
-      </visual>
-      <collision>
-        <origin rpy="0 0 0" xyz="0 0 0"/>
-        <geometry>
-          <mesh filename="package://ar_description/meshes/ar4/link_5.STL"/>
+          <mesh filename="file://$(find ar_description)/meshes/ar4/link_5.STL"/>
+        </geometry>
+        <material name="">
+          <color rgba="1 1 0 1"/>
+        </material>
+      </visual>
+      <collision>
+        <origin rpy="0 0 0" xyz="0 0 0"/>
+        <geometry>
+          <mesh filename="file://$(find ar_description)/meshes/ar4/link_5.STL"/>
         </geometry>
       </collision>
@@ -183,14 +183,14 @@
         <origin rpy="0 0 0" xyz="0 0 0"/>
         <geometry>
-          <mesh filename="package://ar_description/meshes/ar4/link_6.STL"/>
-        </geometry>
-        <material name="">
-          <color rgba="1 1 0 1"/>
-        </material>
-      </visual>
-      <collision>
-        <origin rpy="0 0 0" xyz="0 0 0"/>
-        <geometry>
-          <mesh filename="package://ar_description/meshes/ar4/link_6.STL"/>
+          <mesh filename="file://$(find ar_description)/meshes/ar4/link_6.STL"/>
+        </geometry>
+        <material name="">
+          <color rgba="1 1 0 1"/>
+        </material>
+      </visual>
+      <collision>
+        <origin rpy="0 0 0" xyz="0 0 0"/>
+        <geometry>
+          <mesh filename="file://$(find ar_description)/meshes/ar4/link_6.STL"/>
         </geometry>
       </collision>

File: ar_hardware_interface/urdf/ar.urdf.xacro (robot description, xacro)
@@ -4,5 +4,5 @@
   <xacro:arg name="calibrate" default="True"/>
   <xacro:include filename="$(find ar_description)/urdf/ar_macro.xacro"/>
-  <xacro:include filename="$(find ar_hardware_interface)/urdf/ar.ros2_control.xacro"/>
+  <xacro:include filename="$(find ar_description)/urdf/ar.ros2_control.xacro"/>
   <!-- initial position for simulations (Mock Hardware, Gazebo, Ignition) -->
   <xacro:arg name="initial_positions_file" default="$(find ar_description)/config/initial_positions.yaml"/>

File: ar_moveit_config/urdf/fake_ar.urdf.xacro (robot description, xacro)
@@ -2,5 +2,5 @@
 <robot xmlns:xacro="http://wiki.ros.org/xacro" name="$(arg name)">
   <xacro:include filename="$(find ar_description)/urdf/ar_macro.xacro"/>
-  <xacro:include filename="$(find ar_hardware_interface)/urdf/ar.ros2_control.xacro"/>
+  <xacro:include filename="$(find ar_description)/urdf/ar.ros2_control.xacro"/>
   <link name="world" />
   <xacro:ar_robot parent="world">
