Commit message: debug planning failure

File: ar_description/urdf/ar_gripper.ros2_control.xacro (robot description, xacro)
@@ -20,4 +20,15 @@
         </state_interface>
       </joint>
+      <joint name="gripper_jaw2_joint">
+        <param name="mimic">gripper_jaw1_joint</param>
+        <param name="multiplier">1</param>
+        <command_interface name="position">
+          <param name="min">-0.014</param>
+          <param name="max">0.0</param>
+        </command_interface>
+        <state_interface name="position">
+          <param name="initial_value">0.0</param>
+        </state_interface>
+      </joint>
     </ros2_control>
   </xacro:macro>

File: ar_moveit_config/srdf/ar_gripper_macro.srdf.xacro (robot description, xacro)
@@ -7,6 +7,9 @@
   <xacro:macro name="ar_gripper_srdf">
     <group name="ar_gripper">
+      <link name="gripper_base_link" />
+      <link name="gripper_jaw1_link" />
+      <link name="gripper_jaw2_link" />
       <joint name="gripper_jaw1_joint" />
-      <joint name="gripper_jaw2_joint" />
+      <passive_joint name="gripper_jaw2_joint" />
     </group>
     <group_state name="open" group="ar_gripper">
@@ -19,4 +22,5 @@
     <disable_collisions link1="gripper_base_link" link2="gripper_jaw2_link" reason="Adjacent" />
     <disable_collisions link1="gripper_jaw1_link" link2="gripper_jaw2_link" reason="Adjacent" />
+    <disable_collisions link1="link_6" link2="gripper_base_link" reason="Adjacent" />
   </xacro:macro>
 </robot>
