Commit message: increase velocity limit of J5 and J6

File: ar_description/urdf/ar_macro.xacro (robot description, xacro)
@@ -85,5 +85,5 @@
       <child link="link_2"/>
       <axis xyz="0 0 -1"/>
-      <limit lower="${-42.0 / 180.0 * pi}" upper="${90.0 / 180.0 * pi}" effort="0.5" velocity="0"/>
+      <limit lower="${-42.0 / 180.0 * pi}" upper="${90.0 / 180.0 * pi}" effort="0.5" velocity="0.5"/>
     </joint>
     <link name="link_3">
@@ -172,5 +172,5 @@
       <child link="link_5"/>
       <axis xyz="1 0 0"/>
-      <limit lower="${-105.0 / 180.0 * pi}" upper="${105.0 / 180.0 * pi}" effort="0" velocity="0.5"/>
+      <limit lower="${-105.0 / 180.0 * pi}" upper="${105.0 / 180.0 * pi}" effort="0" velocity="1.0"/>
     </joint>
     <link name="link_6">
@@ -201,5 +201,5 @@
       <child link="link_6"/>
       <axis xyz="0 0 1"/>
-      <limit lower="${-155.0 / 180.0 * pi}" upper="${155.0 / 180.0 * pi}" effort="0" velocity="0.5"/>
+      <limit lower="${-155.0 / 180.0 * pi}" upper="${155.0 / 180.0 * pi}" effort="0" velocity="1.0"/>
     </joint>
     <!-- center of the end effector mounting surface on link_6 -->

Commit message: hopefully more accurate kinematics

File: ar_description/urdf/ar_macro.xacro (robot description, xacro)
@@ -52,5 +52,5 @@
     </link>
     <joint name="joint_1" type="revolute">
-      <origin rpy="${pi} 0 0" xyz="0 0 0.003445"/>
+      <origin rpy="${pi} 0 0" xyz="0 0 0"/>
       <parent link="base_link"/>
       <child link="link_1"/>
@@ -81,5 +81,5 @@
     </link>
     <joint name="joint_2" type="revolute">
-      <origin rpy="1.5708 0.5236 -1.5708" xyz="0 0.064146 -0.16608"/>
+      <origin rpy="1.5708 0 -1.5708" xyz="0 0.0642 -0.16977"/>
       <parent link="link_1"/>
       <child link="link_2"/>
@@ -110,5 +110,5 @@
     </link>
     <joint name="joint_3" type="revolute">
-      <origin rpy="0 0 -2.61799" xyz="0.1525 -0.26414 0"/>
+      <origin rpy="0 0 3.1416" xyz="0 -0.305 0"/>
       <parent link="link_2"/>
       <child link="link_3"/>
@@ -139,5 +139,5 @@
     </link>
     <joint name="joint_4" type="revolute">
-      <origin rpy="1.5708 -1.2554 -1.5708" xyz="0 0 0.00675"/>
+      <origin rpy="1.5708 0 -1.5708" xyz="0 0 0.0"/>
       <parent link="link_3"/>
       <child link="link_4"/>
@@ -168,5 +168,5 @@
     </link>
     <joint name="joint_5" type="revolute">
-      <origin rpy="${pi} 0 -2.8262" xyz="0 0 -0.22225"/>
+      <origin rpy="${pi} 0 -1.5708" xyz="0 0 -0.22263"/>
       <parent link="link_4"/>
       <child link="link_5"/>
@@ -197,5 +197,5 @@
     </link>
     <joint name="joint_6" type="revolute">
-      <origin rpy="0 0 3.1416" xyz="-0.000294 0 0.02117"/>
+      <origin rpy="0 0 3.1416" xyz="0.000 0 0.03625"/>
       <parent link="link_5"/>
       <child link="link_6"/>
@@ -208,5 +208,5 @@
       <parent link="link_6" />
       <child link="ee_link" />
-      <origin xyz="0 0 0.016" rpy="0 0 0" />
+      <origin xyz="0 0 0.0" rpy="0 0 0" />
     </joint>
   </xacro:macro>

Commit message: WIP more accurate kinematics

File: ar_description/urdf/ar_macro.xacro (robot description, xacro)
@@ -52,5 +52,5 @@
     </link>
     <joint name="joint_1" type="revolute">
-      <origin rpy="${pi} 0 0" xyz="0 0 0"/>
+      <origin rpy="${pi} 0 0" xyz="0 0 0.0"/>
       <parent link="base_link"/>
       <child link="link_1"/>

Commit message: more accurate kinematics

File: ar_description/urdf/ar_macro.xacro (robot description, xacro)
@@ -110,5 +110,5 @@
     </link>
     <joint name="joint_3" type="revolute">
-      <origin rpy="0 0 3.1416" xyz="0 -0.305 0"/>
+      <origin rpy="0 0 3.1416" xyz="0 -0.305 0.007"/>
       <parent link="link_2"/>
       <child link="link_3"/>

Commit message: support MK3

File: ar_description/urdf/ar_macro.xacro (robot description, xacro)
@@ -1,5 +1,10 @@
 <?xml version="1.0" encoding="utf-8"?>
 <robot xmlns:xacro="http://wiki.ros.org/xacro">
-  <xacro:macro name="ar_robot" params="parent *origin">
+  <xacro:macro name="ar_robot" params="
+    parent
+    *origin
+    robot_parameters_file
+  ">
+    <xacro:property name="robot_parameters" value="${xacro.load_yaml(robot_parameters_file)}"/>
     <joint name="base_joint" type="fixed">
       <xacro:insert_block name="origin" />
@@ -16,14 +21,14 @@
         <origin rpy="0 0 0" xyz="0 0 0"/>
         <geometry>
-          <mesh filename="file://$(find ar_description)/meshes/ar4/base_link.STL"/>
-        </geometry>
-        <material name="">
-          <color rgba="1 1 0 1"/>
-        </material>
-      </visual>
-      <collision>
-        <origin rpy="0 0 0" xyz="0 0 0"/>
-        <geometry>
-          <mesh filename="file://$(find ar_description)/meshes/ar4/base_link.STL"/>
+          <mesh filename="file://$(find ar_description)/meshes/${robot_parameters['mesh_dir']}/base_link.STL"/>
+        </geometry>
+        <material name="">
+          <color rgba="1 1 0 1"/>
+        </material>
+      </visual>
+      <collision>
+        <origin rpy="0 0 0" xyz="0 0 0"/>
+        <geometry>
+          <mesh filename="file://$(find ar_description)/meshes/${robot_parameters['mesh_dir']}/base_link.STL"/>
         </geometry>
       </collision>
@@ -38,14 +43,14 @@
         <origin rpy="0 0 0" xyz="0 0 0"/>
         <geometry>
-          <mesh filename="file://$(find ar_description)/meshes/ar4/link_1.STL"/>
-        </geometry>
-        <material name="">
-          <color rgba="1 1 0 1"/>
-        </material>
-      </visual>
-      <collision>
-        <origin rpy="0 0 0" xyz="0 0 0"/>
-        <geometry>
-          <mesh filename="file://$(find ar_description)/meshes/ar4/link_1.STL"/>
+          <mesh filename="file://$(find ar_description)/meshes/${robot_parameters['mesh_dir']}/link_1.STL"/>
+        </geometry>
+        <material name="">
+          <color rgba="1 1 0 1"/>
+        </material>
+      </visual>
+      <collision>
+        <origin rpy="0 0 0" xyz="0 0 0"/>
+        <geometry>
+          <mesh filename="file://$(find ar_description)/meshes/${robot_parameters['mesh_dir']}/link_1.STL"/>
         </geometry>
       </collision>
@@ -67,14 +72,14 @@
         <origin rpy="0 0 0" xyz="0 0 0"/>
         <geometry>
-          <mesh filename="file://$(find ar_description)/meshes/ar4/link_2.STL"/>
-        </geometry>
-        <material name="">
-          <color rgba="1 1 0 1"/>
-        </material>
-      </visual>
-      <collision>
-        <origin rpy="0 0 0" xyz="0 0 0"/>
-        <geometry>
-          <mesh filename="file://$(find ar_description)/meshes/ar4/link_2.STL"/>
+          <mesh filename="file://$(find ar_description)/meshes/${robot_parameters['mesh_dir']}/link_2.STL"/>
+        </geometry>
+        <material name="">
+          <color rgba="1 1 0 1"/>
+        </material>
+      </visual>
+      <collision>
+        <origin rpy="0 0 0" xyz="0 0 0"/>
+        <geometry>
+          <mesh filename="file://$(find ar_description)/meshes/${robot_parameters['mesh_dir']}/link_2.STL"/>
         </geometry>
       </collision>
@@ -96,14 +101,14 @@
         <origin rpy="0 0 0" xyz="0 0 0"/>
         <geometry>
-          <mesh filename="file://$(find ar_description)/meshes/ar4/link_3.STL"/>
-        </geometry>
-        <material name="">
-          <color rgba="1 1 0 1"/>
-        </material>
-      </visual>
-      <collision>
-        <origin rpy="0 0 0" xyz="0 0 0"/>
-        <geometry>
-          <mesh filename="file://$(find ar_description)/meshes/ar4/link_3.STL"/>
+          <mesh filename="file://$(find ar_description)/meshes/${robot_parameters['mesh_dir']}/link_3.STL"/>
+        </geometry>
+        <material name="">
+          <color rgba="1 1 0 1"/>
+        </material>
+      </visual>
+      <collision>
+        <origin rpy="0 0 0" xyz="0 0 0"/>
+        <geometry>
+          <mesh filename="file://$(find ar_description)/meshes/${robot_parameters['mesh_dir']}/link_3.STL"/>
         </geometry>
       </collision>
@@ -125,14 +130,14 @@
         <origin rpy="0 0 0" xyz="0 0 0"/>
         <geometry>
-          <mesh filename="file://$(find ar_description)/meshes/ar4/link_4.STL"/>
-        </geometry>
-        <material name="">
-          <color rgba="1 1 0 1"/>
-        </material>
-      </visual>
-      <collision>
-        <origin rpy="0 0 0" xyz="0 0 0"/>
-        <geometry>
-          <mesh filename="file://$(find ar_description)/meshes/ar4/link_4.STL"/>
+          <mesh filename="file://$(find ar_description)/meshes/${robot_parameters['mesh_dir']}/link_4.STL"/>
+        </geometry>
+        <material name="">
+          <color rgba="1 1 0 1"/>
+        </material>
+      </visual>
+      <collision>
+        <origin rpy="0 0 0" xyz="0 0 0"/>
+        <geometry>
+          <mesh filename="file://$(find ar_description)/meshes/${robot_parameters['mesh_dir']}/link_4.STL"/>
         </geometry>
       </collision>
@@ -143,5 +148,5 @@
       <child link="link_4"/>
       <axis xyz="0 0 -1"/>
-      <limit lower="${-165.0 / 180.0 * pi}" upper="${165.0 / 180.0 * pi}" effort="0" velocity="0.5"/>
+      <limit lower="${-1 * robot_parameters['j4_limit']}" upper="${robot_parameters['j4_limit']}" effort="0" velocity="0.5"/>
     </joint>
     <link name="link_5">
@@ -154,14 +159,14 @@
         <origin rpy="0 0 0" xyz="0 0 0"/>
         <geometry>
-          <mesh filename="file://$(find ar_description)/meshes/ar4/link_5.STL"/>
-        </geometry>
-        <material name="">
-          <color rgba="1 1 0 1"/>
-        </material>
-      </visual>
-      <collision>
-        <origin rpy="0 0 0" xyz="0 0 0"/>
-        <geometry>
-          <mesh filename="file://$(find ar_description)/meshes/ar4/link_5.STL"/>
+          <mesh filename="file://$(find ar_description)/meshes/${robot_parameters['mesh_dir']}/link_5.STL"/>
+        </geometry>
+        <material name="">
+          <color rgba="1 1 0 1"/>
+        </material>
+      </visual>
+      <collision>
+        <origin rpy="0 0 0" xyz="0 0 0"/>
+        <geometry>
+          <mesh filename="file://$(find ar_description)/meshes/${robot_parameters['mesh_dir']}/link_5.STL"/>
         </geometry>
       </collision>
@@ -183,23 +188,23 @@
         <origin rpy="0 0 0" xyz="0 0 0"/>
         <geometry>
-          <mesh filename="file://$(find ar_description)/meshes/ar4/link_6.STL"/>
-        </geometry>
-        <material name="">
-          <color rgba="1 1 0 1"/>
-        </material>
-      </visual>
-      <collision>
-        <origin rpy="0 0 0" xyz="0 0 0"/>
-        <geometry>
-          <mesh filename="file://$(find ar_description)/meshes/ar4/link_6.STL"/>
+          <mesh filename="file://$(find ar_description)/meshes/${robot_parameters['mesh_dir']}/link_6.STL"/>
+        </geometry>
+        <material name="">
+          <color rgba="1 1 0 1"/>
+        </material>
+      </visual>
+      <collision>
+        <origin rpy="0 0 0" xyz="0 0 0"/>
+        <geometry>
+          <mesh filename="file://$(find ar_description)/meshes/${robot_parameters['mesh_dir']}/link_6.STL"/>
         </geometry>
       </collision>
     </link>
     <joint name="joint_6" type="revolute">
-      <origin rpy="0 0 3.1416" xyz="0.000 0 0.03625"/>
+      <origin rpy="0 0 3.1416" xyz="0.000 0 ${robot_parameters['l6_length']}"/>
       <parent link="link_5"/>
       <child link="link_6"/>
       <axis xyz="0 0 1"/>
-      <limit lower="${-155.0 / 180.0 * pi}" upper="${155.0 / 180.0 * pi}" effort="0" velocity="1.0"/>
+      <limit lower="${-1.0 * robot_parameters['j6_limit']}" upper="${robot_parameters['j6_limit']}" effort="0" velocity="1.0"/>
     </joint>
     <!-- center of the end effector mounting surface on link_6 -->

File: ar_moveit_config/srdf/ar_gripper_macro.srdf.xacro (robot description, xacro)
@@ -23,4 +23,5 @@
     <disable_collisions link1="gripper_jaw1_link" link2="gripper_jaw2_link" reason="Default" />
     <disable_collisions link1="link_6" link2="gripper_base_link" reason="Adjacent" />
+    <disable_collisions link1="link_5" link2="gripper_base_link" reason="Adjacent" />
   </xacro:macro>
 </robot>

File: ar_moveit_config/urdf/fake_ar.urdf.xacro (robot description, xacro)
@@ -1,4 +1,4 @@
 <?xml version="1.0"?>
-<robot xmlns:xacro="http://wiki.ros.org/xacro" name="$(arg name)">
+<robot xmlns:xacro="http://wiki.ros.org/xacro" name="$(arg ar_model)">
   <xacro:include filename="$(find ar_description)/urdf/ar_macro.xacro"/>
   <xacro:include filename="$(find ar_description)/urdf/ar_gripper_macro.xacro"/>
@@ -6,5 +6,8 @@
   <xacro:include filename="$(find ar_description)/urdf/ar_gripper.ros2_control.xacro"/>
   <link name="world" />
-  <xacro:ar_robot parent="world">
+  <xacro:ar_robot
+    parent="world"
+    robot_parameters_file="$(find ar_description)/config/$(arg ar_model).yaml"
+  >
     <origin xyz="0 0 0" rpy="0 0 0" />
   </xacro:ar_robot>
