Commit message: fix gripper alignment and change its color

File: ar_description/urdf/ar_gripper_macro.xacro (robot description, xacro)
@@ -12,4 +12,7 @@
           <mesh filename="file://$(find ar_description)/meshes/ar4_gripper/gripper_base_link.stl" />
         </geometry>
+        <material name="">
+          <color rgba="1 1 0 1"/>
+        </material>
       </visual>
       <collision>
@@ -29,4 +32,7 @@
           <mesh filename="file://$(find ar_description)/meshes/ar4_gripper/gripper_jaw1_link.stl" />
         </geometry>
+        <material name="">
+          <color rgba="1 1 0 1"/>
+        </material>
       </visual>
       <collision>
@@ -46,4 +52,7 @@
           <mesh filename="file://$(find ar_description)/meshes/ar4_gripper/gripper_jaw2_link.stl" />
         </geometry>
+        <material name="">
+          <color rgba="1 1 0 1"/>
+        </material>
       </visual>
       <collision>
@@ -59,5 +68,5 @@
     </link>
     <joint name="gripper_jaw1_joint" type="prismatic">
-      <origin xyz="0.0 -0.036 -0.0155" rpy="0.0 0.0 0.0"/>
+      <origin xyz="0.0 -0.036 0" rpy="0.0 0.0 0.0"/>
       <parent link="gripper_base_link"/>
       <child link="gripper_jaw1_link"/>
@@ -66,5 +75,5 @@
     </joint>
     <joint name="gripper_jaw2_joint" type="prismatic">
-      <origin xyz="0.0 -0.036 0.0097" rpy="0.0 ${-pi} 0.0"/>
+      <origin xyz="0.0 -0.036 0" rpy="0.0 ${-pi} 0.0"/>
       <parent link="gripper_base_link"/>
       <child link="gripper_jaw2_link"/>

Commit message: working gripper

File: ar_description/urdf/ar_gripper_macro.xacro (robot description, xacro)
@@ -72,5 +72,5 @@
       <child link="gripper_jaw1_link"/>
       <axis xyz="1 0 0"/>
-      <limit lower="-0.014" upper="0" effort="0" velocity="0.1"/>
+      <limit lower="-0.014" upper="0" effort="-1" velocity="1.0"/>
     </joint>
     <joint name="gripper_jaw2_joint" type="prismatic">
@@ -79,5 +79,5 @@
       <child link="gripper_jaw2_link"/>
       <axis xyz="1 0 0"/>
-      <limit lower="-0.014" upper="0" effort="0" velocity="0.1"/>
+      <limit lower="-0.014" upper="0" effort="-1" velocity="1.0"/>
       <mimic joint="gripper_jaw1_joint" multiplier="1" offset="0"/>
     </joint>
