Commit message: rename AR

File: ar_description/urdf/ar.urdf.xacro (robot description, xacro)
@@ -1,9 +1,8 @@
 <?xml version="1.0"?>
 <robot xmlns:xacro="http://wiki.ros.org/xacro" name="$(arg name)">
-  <xacro:arg name="ar_type" default="ar3"/>
-  <xacro:include filename="$(find ar_description)/urdf/$(arg ar_type)_macro.xacro"/>
+  <xacro:include filename="$(find ar_description)/urdf/ar_macro.xacro"/>
   <link name="world" />
-  <xacro:ar3_robot parent="world">
+  <xacro:ar_robot parent="world">
     <origin xyz="0 0 0" rpy="0 0 0" />
-  </xacro:ar3_robot>
+  </xacro:ar_robot>
 </robot>

File: ar_description/urdf/ar_gazebo.urdf.xacro (robot description, xacro)
@@ -1,8 +1,8 @@
 <?xml version="1.0" encoding="utf-8"?>
 <!-- =================================================================================== -->
-<!-- |    This document was autogenerated by xacro from ar3.urdf                       | -->
+<!-- |    This document was autogenerated by xacro from ar4.urdf                       | -->
 <!-- |    EDITING THIS FILE BY HAND IS NOT RECOMMENDED but it was unfortunately        | -->
 <!-- =================================================================================== -->
-<robot name="ar3">
+<robot name="ar">
   <link name="world" />
   <link name="base_link">
@@ -15,14 +15,14 @@
       <origin rpy="0 0 0" xyz="0 0 0"/>
       <geometry>
-        <mesh filename="package://ar_description/meshes/ar3/base_link.STL"/>
-      </geometry>
-      <material name="">
-        <color rgba="1 1 0 1"/>
-      </material>
-    </visual>
-    <collision>
-      <origin rpy="0 0 0" xyz="0 0 0"/>
-      <geometry>
-        <mesh filename="package://ar_description/meshes/ar3/base_link.STL"/>
+        <mesh filename="package://ar_description/meshes/ar4/base_link.STL"/>
+      </geometry>
+      <material name="">
+        <color rgba="1 1 0 1"/>
+      </material>
+    </visual>
+    <collision>
+      <origin rpy="0 0 0" xyz="0 0 0"/>
+      <geometry>
+        <mesh filename="package://ar_description/meshes/ar4/base_link.STL"/>
       </geometry>
     </collision>
@@ -42,14 +42,14 @@
       <origin rpy="0 0 0" xyz="0 0 0"/>
       <geometry>
-        <mesh filename="package://ar_description/meshes/ar3/link_1.STL"/>
-      </geometry>
-      <material name="">
-        <color rgba="1 1 0 1"/>
-      </material>
-    </visual>
-    <collision>
-      <origin rpy="0 0 0" xyz="0 0 0"/>
-      <geometry>
-        <mesh filename="package://ar_description/meshes/ar3/link_1.STL"/>
+        <mesh filename="package://ar_description/meshes/ar4/link_1.STL"/>
+      </geometry>
+      <material name="">
+        <color rgba="1 1 0 1"/>
+      </material>
+    </visual>
+    <collision>
+      <origin rpy="0 0 0" xyz="0 0 0"/>
+      <geometry>
+        <mesh filename="package://ar_description/meshes/ar4/link_1.STL"/>
       </geometry>
     </collision>
@@ -71,14 +71,14 @@
       <origin rpy="0 0 0" xyz="0 0 0"/>
       <geometry>
-        <mesh filename="package://ar_description/meshes/ar3/link_2.STL"/>
-      </geometry>
-      <material name="">
-        <color rgba="1 1 0 1"/>
-      </material>
-    </visual>
-    <collision>
-      <origin rpy="0 0 0" xyz="0 0 0"/>
-      <geometry>
-        <mesh filename="package://ar_description/meshes/ar3/link_2.STL"/>
+        <mesh filename="package://ar_description/meshes/ar4/link_2.STL"/>
+      </geometry>
+      <material name="">
+        <color rgba="1 1 0 1"/>
+      </material>
+    </visual>
+    <collision>
+      <origin rpy="0 0 0" xyz="0 0 0"/>
+      <geometry>
+        <mesh filename="package://ar_description/meshes/ar4/link_2.STL"/>
       </geometry>
     </collision>
@@ -100,14 +100,14 @@
       <origin rpy="0 0 0" xyz="0 0 0"/>
       <geometry>
-        <mesh filename="package://ar_description/meshes/ar3/link_3.STL"/>
-      </geometry>
-      <material name="">
-        <color rgba="1 1 0 1"/>
-      </material>
-    </visual>
-    <collision>
-      <origin rpy="0 0 0" xyz="0 0 0"/>
-      <geometry>
-        <mesh filename="package://ar_description/meshes/ar3/link_3.STL"/>
+        <mesh filename="package://ar_description/meshes/ar4/link_3.STL"/>
+      </geometry>
+      <material name="">
+        <color rgba="1 1 0 1"/>
+      </material>
+    </visual>
+    <collision>
+      <origin rpy="0 0 0" xyz="0 0 0"/>
+      <geometry>
+        <mesh filename="package://ar_description/meshes/ar4/link_3.STL"/>
       </geometry>
     </collision>
@@ -129,14 +129,14 @@
       <origin rpy="0 0 0" xyz="0 0 0"/>
       <geometry>
-        <mesh filename="package://ar_description/meshes/ar3/link_4.STL"/>
-      </geometry>
-      <material name="">
-        <color rgba="1 1 0 1"/>
-      </material>
-    </visual>
-    <collision>
-      <origin rpy="0 0 0" xyz="0 0 0"/>
-      <geometry>
-        <mesh filename="package://ar_description/meshes/ar3/link_4.STL"/>
+        <mesh filename="package://ar_description/meshes/ar4/link_4.STL"/>
+      </geometry>
+      <material name="">
+        <color rgba="1 1 0 1"/>
+      </material>
+    </visual>
+    <collision>
+      <origin rpy="0 0 0" xyz="0 0 0"/>
+      <geometry>
+        <mesh filename="package://ar_description/meshes/ar4/link_4.STL"/>
       </geometry>
     </collision>
@@ -158,14 +158,14 @@
       <origin rpy="0 0 0" xyz="0 0 0"/>
       <geometry>
-        <mesh filename="package://ar_description/meshes/ar3/link_5.STL"/>
-      </geometry>
-      <material name="">
-        <color rgba="1 1 0 1"/>
-      </material>
-    </visual>
-    <collision>
-      <origin rpy="0 0 0" xyz="0 0 0"/>
-      <geometry>
-        <mesh filename="package://ar_description/meshes/ar3/link_5.STL"/>
+        <mesh filename="package://ar_description/meshes/ar4/link_5.STL"/>
+      </geometry>
+      <material name="">
+        <color rgba="1 1 0 1"/>
+      </material>
+    </visual>
+    <collision>
+      <origin rpy="0 0 0" xyz="0 0 0"/>
+      <geometry>
+        <mesh filename="package://ar_description/meshes/ar4/link_5.STL"/>
       </geometry>
     </collision>
@@ -187,14 +187,14 @@
       <origin rpy="0 0 0" xyz="0 0 0"/>
       <geometry>
-        <mesh filename="package://ar_description/meshes/ar3/link_6.STL"/>
-      </geometry>
-      <material name="">
-        <color rgba="1 1 0 1"/>
-      </material>
-    </visual>
-    <collision>
-      <origin rpy="0 0 0" xyz="0 0 0"/>
-      <geometry>
-        <mesh filename="package://ar_description/meshes/ar3/link_6.STL"/>
+        <mesh filename="package://ar_description/meshes/ar4/link_6.STL"/>
+      </geometry>
+      <material name="">
+        <color rgba="1 1 0 1"/>
+      </material>
+    </visual>
+    <collision>
+      <origin rpy="0 0 0" xyz="0 0 0"/>
+      <geometry>
+        <mesh filename="package://ar_description/meshes/ar4/link_6.STL"/>
       </geometry>
     </collision>

File: ar_description/urdf/ar_macro.xacro (robot description, xacro)
@@ -1,5 +1,5 @@
 <?xml version="1.0" encoding="utf-8"?>
 <robot xmlns:xacro="http://wiki.ros.org/xacro">
-  <xacro:macro name="ar3_robot" params="parent *origin">
+  <xacro:macro name="ar_robot" params="parent *origin">
     <joint name="base_joint" type="fixed">
       <xacro:insert_block name="origin" />
@@ -16,14 +16,14 @@
         <origin rpy="0 0 0" xyz="0 0 0"/>
         <geometry>
-          <mesh filename="package://ar_description/meshes/ar3/base_link.STL"/>
-        </geometry>
-        <material name="">
-          <color rgba="1 1 0 1"/>
-        </material>
-      </visual>
-      <collision>
-        <origin rpy="0 0 0" xyz="0 0 0"/>
-        <geometry>
-          <mesh filename="package://ar_description/meshes/ar3/base_link.STL"/>
+          <mesh filename="package://ar_description/meshes/ar4/base_link.STL"/>
+        </geometry>
+        <material name="">
+          <color rgba="1 1 0 1"/>
+        </material>
+      </visual>
+      <collision>
+        <origin rpy="0 0 0" xyz="0 0 0"/>
+        <geometry>
+          <mesh filename="package://ar_description/meshes/ar4/base_link.STL"/>
         </geometry>
       </collision>
@@ -38,14 +38,14 @@
         <origin rpy="0 0 0" xyz="0 0 0"/>
         <geometry>
-          <mesh filename="package://ar_description/meshes/ar3/link_1.STL"/>
-        </geometry>
-        <material name="">
-          <color rgba="1 1 0 1"/>
-        </material>
-      </visual>
-      <collision>
-        <origin rpy="0 0 0" xyz="0 0 0"/>
-        <geometry>
-          <mesh filename="package://ar_description/meshes/ar3/link_1.STL"/>
+          <mesh filename="package://ar_description/meshes/ar4/link_1.STL"/>
+        </geometry>
+        <material name="">
+          <color rgba="1 1 0 1"/>
+        </material>
+      </visual>
+      <collision>
+        <origin rpy="0 0 0" xyz="0 0 0"/>
+        <geometry>
+          <mesh filename="package://ar_description/meshes/ar4/link_1.STL"/>
         </geometry>
       </collision>
@@ -67,14 +67,14 @@
         <origin rpy="0 0 0" xyz="0 0 0"/>
         <geometry>
-          <mesh filename="package://ar_description/meshes/ar3/link_2.STL"/>
-        </geometry>
-        <material name="">
-          <color rgba="1 1 0 1"/>
-        </material>
-      </visual>
-      <collision>
-        <origin rpy="0 0 0" xyz="0 0 0"/>
-        <geometry>
-          <mesh filename="package://ar_description/meshes/ar3/link_2.STL"/>
+          <mesh filename="package://ar_description/meshes/ar4/link_2.STL"/>
+        </geometry>
+        <material name="">
+          <color rgba="1 1 0 1"/>
+        </material>
+      </visual>
+      <collision>
+        <origin rpy="0 0 0" xyz="0 0 0"/>
+        <geometry>
+          <mesh filename="package://ar_description/meshes/ar4/link_2.STL"/>
         </geometry>
       </collision>
@@ -96,14 +96,14 @@
         <origin rpy="0 0 0" xyz="0 0 0"/>
         <geometry>
-          <mesh filename="package://ar_description/meshes/ar3/link_3.STL"/>
-        </geometry>
-        <material name="">
-          <color rgba="1 1 0 1"/>
-        </material>
-      </visual>
-      <collision>
-        <origin rpy="0 0 0" xyz="0 0 0"/>
-        <geometry>
-          <mesh filename="package://ar_description/meshes/ar3/link_3.STL"/>
+          <mesh filename="package://ar_description/meshes/ar4/link_3.STL"/>
+        </geometry>
+        <material name="">
+          <color rgba="1 1 0 1"/>
+        </material>
+      </visual>
+      <collision>
+        <origin rpy="0 0 0" xyz="0 0 0"/>
+        <geometry>
+          <mesh filename="package://ar_description/meshes/ar4/link_3.STL"/>
         </geometry>
       </collision>
@@ -125,14 +125,14 @@
         <origin rpy="0 0 0" xyz="0 0 0"/>
         <geometry>
-          <mesh filename="package://ar_description/meshes/ar3/link_4.STL"/>
-        </geometry>
-        <material name="">
-          <color rgba="1 1 0 1"/>
-        </material>
-      </visual>
-      <collision>
-        <origin rpy="0 0 0" xyz="0 0 0"/>
-        <geometry>
-          <mesh filename="package://ar_description/meshes/ar3/link_4.STL"/>
+          <mesh filename="package://ar_description/meshes/ar4/link_4.STL"/>
+        </geometry>
+        <material name="">
+          <color rgba="1 1 0 1"/>
+        </material>
+      </visual>
+      <collision>
+        <origin rpy="0 0 0" xyz="0 0 0"/>
+        <geometry>
+          <mesh filename="package://ar_description/meshes/ar4/link_4.STL"/>
         </geometry>
       </collision>
@@ -154,14 +154,14 @@
         <origin rpy="0 0 0" xyz="0 0 0"/>
         <geometry>
-          <mesh filename="package://ar_description/meshes/ar3/link_5.STL"/>
-        </geometry>
-        <material name="">
-          <color rgba="1 1 0 1"/>
-        </material>
-      </visual>
-      <collision>
-        <origin rpy="0 0 0" xyz="0 0 0"/>
-        <geometry>
-          <mesh filename="package://ar_description/meshes/ar3/link_5.STL"/>
+          <mesh filename="package://ar_description/meshes/ar4/link_5.STL"/>
+        </geometry>
+        <material name="">
+          <color rgba="1 1 0 1"/>
+        </material>
+      </visual>
+      <collision>
+        <origin rpy="0 0 0" xyz="0 0 0"/>
+        <geometry>
+          <mesh filename="package://ar_description/meshes/ar4/link_5.STL"/>
         </geometry>
       </collision>
@@ -183,14 +183,14 @@
         <origin rpy="0 0 0" xyz="0 0 0"/>
         <geometry>
-          <mesh filename="package://ar_description/meshes/ar3/link_6.STL"/>
-        </geometry>
-        <material name="">
-          <color rgba="1 1 0 1"/>
-        </material>
-      </visual>
-      <collision>
-        <origin rpy="0 0 0" xyz="0 0 0"/>
-        <geometry>
-          <mesh filename="package://ar_description/meshes/ar3/link_6.STL"/>
+          <mesh filename="package://ar_description/meshes/ar4/link_6.STL"/>
+        </geometry>
+        <material name="">
+          <color rgba="1 1 0 1"/>
+        </material>
+      </visual>
+      <collision>
+        <origin rpy="0 0 0" xyz="0 0 0"/>
+        <geometry>
+          <mesh filename="package://ar_description/meshes/ar4/link_6.STL"/>
         </geometry>
       </collision>

File: ar_hardware_interface/urdf/ar.urdf.xacro (robot description, xacro)
@@ -1,10 +1,7 @@
 <?xml version="1.0"?>
 <robot xmlns:xacro="http://wiki.ros.org/xacro" name="$(arg name)">
-  <!-- TODO: merge name and ar_type -->
-  <xacro:arg name="name" default="ar"/>
-  <xacro:arg name="ar_type" default="ar3"/>
   <xacro:arg name="serial_port" default="/dev/ttyACM0"/>
   <xacro:arg name="calibrate" default="True"/>
-  <xacro:include filename="$(find ar_description)/urdf/$(arg ar_type)_macro.xacro"/>
+  <xacro:include filename="$(find ar_description)/urdf/ar_macro.xacro"/>
   <xacro:include filename="$(find ar_hardware_interface)/urdf/ar.ros2_control.xacro"/>
   <!-- initial position for simulations (Mock Hardware, Gazebo, Ignition) -->
@@ -13,7 +10,7 @@
   <xacro:property name="initial_positions_file" default="$(arg initial_positions_file)"/>
   <link name="world" />
-  <xacro:ar3_robot parent="world">
+  <xacro:ar_robot parent="world">
     <origin xyz="0 0 0" rpy="0 0 0" />
-  </xacro:ar3_robot>
+  </xacro:ar_robot>
   <xacro:ar_ros2_control
     name="$(arg name)"

File: ar_moveit_config/urdf/fake_ar.urdf.xacro (robot description, xacro)
@@ -1,12 +1,10 @@
 <?xml version="1.0"?>
 <robot xmlns:xacro="http://wiki.ros.org/xacro" name="$(arg name)">
-  <!-- TODO: merge name and ar_type -->
-  <xacro:arg name="ar_type" default="ar3"/>
-  <xacro:include filename="$(find ar_description)/urdf/$(arg ar_type)_macro.xacro"/>
+  <xacro:include filename="$(find ar_description)/urdf/ar_macro.xacro"/>
   <xacro:include filename="$(find ar_hardware_interface)/urdf/ar.ros2_control.xacro"/>
   <link name="world" />
-  <xacro:ar3_robot parent="world">
+  <xacro:ar_robot parent="world">
     <origin xyz="0 0 0" rpy="0 0 0" />
-  </xacro:ar3_robot>
+  </xacro:ar_robot>
   <xacro:ar_ros2_control
     name="ARFakeSystem"

Commit message: begin adding ar gripper

File: ar_description/urdf/ar.urdf.xacro (robot description, xacro)
@@ -2,7 +2,7 @@
 <robot xmlns:xacro="http://wiki.ros.org/xacro" name="$(arg name)">
   <xacro:include filename="$(find ar_description)/urdf/ar_macro.xacro"/>
+  <xacro:include filename="$(find ar_description)/urdf/ar_gripper_macro.xacro"/>
   <link name="world" />
-  <xacro:ar_robot parent="world">
-    <origin xyz="0 0 0" rpy="0 0 0" />
-  </xacro:ar_robot>
+  <xacro:ar_robot parent="world" />
+  <xacro:ar_gripper parent="link_6" />
 </robot>

File: ar_hardware_interface/urdf/ar.urdf.xacro (robot description, xacro)
@@ -5,8 +5,4 @@
   <xacro:include filename="$(find ar_description)/urdf/ar_macro.xacro"/>
   <xacro:include filename="$(find ar_description)/urdf/ar.ros2_control.xacro"/>
-  <!-- initial position for simulations (Mock Hardware, Gazebo, Ignition) -->
-  <xacro:arg name="initial_positions_file" default="$(find ar_description)/config/initial_positions.yaml"/>
-  <!-- convert to property to use substitution in function -->
-  <xacro:property name="initial_positions_file" default="$(arg initial_positions_file)"/>
   <link name="world" />
   <xacro:ar_robot parent="world">

File: ar_moveit_config/srdf/ar.srdf.xacro (robot description, xacro)
@@ -2,4 +2,6 @@
 <robot xmlns:xacro="http://wiki.ros.org/xacro" name="$(arg name)">
   <xacro:include filename="$(find ar_moveit_config)/srdf/ar_macro.srdf.xacro"/>
+  <xacro:include filename="$(find ar_moveit_config)/srdf/ar_gripper_macro.srdf.xacro"/>
   <xacro:ar_srdf />
+  <xacro:ar_gripper_srdf />
 </robot>

File: ar_moveit_config/urdf/fake_ar.urdf.xacro (robot description, xacro)
@@ -2,9 +2,12 @@
 <robot xmlns:xacro="http://wiki.ros.org/xacro" name="$(arg name)">
   <xacro:include filename="$(find ar_description)/urdf/ar_macro.xacro"/>
+  <xacro:include filename="$(find ar_description)/urdf/ar_gripper_macro.xacro"/>
   <xacro:include filename="$(find ar_description)/urdf/ar.ros2_control.xacro"/>
+  <xacro:include filename="$(find ar_description)/urdf/ar_gripper.ros2_control.xacro"/>
   <link name="world" />
   <xacro:ar_robot parent="world">
     <origin xyz="0 0 0" rpy="0 0 0" />
   </xacro:ar_robot>
+  <xacro:ar_gripper parent="link_6" />
   <xacro:ar_ros2_control
     name="ARFakeSystem"
@@ -13,3 +16,8 @@
     calibrate="False"
   />
+  <xacro:ar_gripper_ros2_control
+    name="ARGripperFakeSystem"
+    plugin_name="mock_components/GenericSystem"
+    serial_port="/dev/ttyUSB0"
+  />
 </robot>

Commit message: working simulation and hardware grippers

File: ar_description/urdf/ar.urdf.xacro (robot description, xacro)
@@ -4,5 +4,7 @@
   <xacro:include filename="$(find ar_description)/urdf/ar_gripper_macro.xacro"/>
   <link name="world" />
-  <xacro:ar_robot parent="world" />
+  <xacro:ar_robot parent="world">
+    <origin xyz="0 0 0" rpy="0 0 0" />
+  </xacro:ar_robot>
   <xacro:ar_gripper parent="link_6" />
 </robot>

Commit message: introduce ee_link, calibration uses camera_color_frame

File: ar_description/urdf/ar.urdf.xacro (robot description, xacro)
@@ -9,5 +9,5 @@
   <xacro:if value="$(arg include_gripper)">
     <xacro:include filename="$(find ar_description)/urdf/ar_gripper_macro.xacro"/>
-    <xacro:ar_gripper parent="link_6" />
+    <xacro:ar_gripper parent="ee_link" />
   </xacro:if>
 </robot>

File: ar_description/urdf/ar_gazebo.urdf.xacro (robot description, xacro)
@@ -10,5 +10,5 @@
     <origin xyz="0 0 0" rpy="0 0 0" />
   </xacro:ar_robot>
-  <xacro:ar_gripper parent="link_6" />
+  <xacro:ar_gripper parent="ee_link" />
   <xacro:ar_ros2_control
     name="ARGazeboSystem"

File: ar_description/urdf/ar_gripper_macro.xacro (robot description, xacro)
@@ -3,5 +3,5 @@
   <xacro:macro name="ar_gripper" params="parent">
     <joint name="gripper_base_joint" type="fixed">
-      <origin xyz="0.0 0.0 0.016" rpy="-1.5708 0.0 0.0"/>
+      <origin xyz="0.0 0.0 0.0" rpy="-1.5708 0.0 0.0"/>
       <parent link="${parent}"/>
       <child link="gripper_base_link"/>

File: ar_description/urdf/ar_macro.xacro (robot description, xacro)
@@ -203,4 +203,11 @@
       <limit lower="${-155.0 / 180.0 * pi}" upper="${155.0 / 180.0 * pi}" effort="0" velocity="0.5"/>
     </joint>
+    <!-- center of the end effector mounting surface on link_6 -->
+    <link name="ee_link" />
+    <joint name="ee_joint" type="fixed">
+      <parent link="link_6" />
+      <child link="ee_link" />
+      <origin xyz="0 0 0.016" rpy="0 0 0" />
+    </joint>
   </xacro:macro>
 </robot>

File: ar_hardware_interface/urdf/ar.urdf.xacro (robot description, xacro)
@@ -21,5 +21,5 @@
     <xacro:include filename="$(find ar_description)/urdf/ar_gripper_macro.xacro"/>
     <xacro:include filename="$(find ar_description)/urdf/ar_gripper.ros2_control.xacro"/>
-    <xacro:ar_gripper parent="link_6" />
+    <xacro:ar_gripper parent="ee_link" />
     <xacro:ar_gripper_ros2_control
       name="ar_servo_gripper"

File: ar_moveit_config/srdf/ar_gripper_macro.srdf.xacro (robot description, xacro)
@@ -17,9 +17,9 @@
     </group_state>
     <group_state name="closed" group="ar_gripper">
-      <joint name="gripper_jaw1_joint" value="0" />
+      <joint name="gripper_jaw1_joint" value="-0.001" />
     </group_state>
     <disable_collisions link1="gripper_base_link" link2="gripper_jaw1_link" reason="Adjacent" />
     <disable_collisions link1="gripper_base_link" link2="gripper_jaw2_link" reason="Adjacent" />
-    <disable_collisions link1="gripper_jaw1_link" link2="gripper_jaw2_link" reason="Adjacent" />
+    <disable_collisions link1="gripper_jaw1_link" link2="gripper_jaw2_link" reason="Default" />
     <disable_collisions link1="link_6" link2="gripper_base_link" reason="Adjacent" />
   </xacro:macro>

File: ar_moveit_config/srdf/ar_macro.srdf.xacro (robot description, xacro)
@@ -13,4 +13,5 @@
       <joint name="joint_5" />
       <joint name="joint_6" />
+      <joint name="ee_joint"/>
     </group>
     <group_state name="home" group="ar_manipulator">

File: ar_moveit_config/urdf/fake_ar.urdf.xacro (robot description, xacro)
@@ -9,5 +9,5 @@
     <origin xyz="0 0 0" rpy="0 0 0" />
   </xacro:ar_robot>
-  <xacro:ar_gripper parent="link_6" />
+  <xacro:ar_gripper parent="ee_link" />
   <xacro:ar_ros2_control
     name="ARFakeSystem"
