Commit message: rename all files

File: ar_description/urdf/ar.urdf.xacro (robot description, xacro)
@@ -2,14 +2,14 @@
 <robot xmlns:xacro="http://wiki.ros.org/xacro" name="$(arg ar_model)">
   <xacro:arg name="include_gripper" default="true"/>
-  <xacro:include filename="$(find ar_description)/urdf/ar_macro.xacro"/>
+  <xacro:include filename="$(find annin_ar4_description)/urdf/ar_macro.xacro"/>
   <link name="world" />
   <xacro:ar_robot
     parent="world"
-    robot_parameters_file="$(find ar_description)/config/$(arg ar_model).yaml"
+    robot_parameters_file="$(find annin_ar4_description)/config/$(arg ar_model).yaml"
   >
     <origin xyz="0 0 0" rpy="0 0 0" />
   </xacro:ar_robot>
   <xacro:if value="$(arg include_gripper)">
-    <xacro:include filename="$(find ar_description)/urdf/ar_gripper_macro.xacro"/>
+    <xacro:include filename="$(find annin_ar4_description)/urdf/ar_gripper_macro.xacro"/>
     <xacro:ar_gripper parent="ee_link" />
   </xacro:if>

File: ar_description/urdf/ar_gazebo.urdf.xacro (robot description, xacro)
@@ -1,13 +1,13 @@
 <?xml version="1.0"?>
 <robot xmlns:xacro="http://wiki.ros.org/xacro" name="$(arg ar_model)">
-  <xacro:include filename="$(find ar_description)/urdf/ar_macro.xacro" />
-  <xacro:include filename="$(find ar_description)/urdf/ar_gripper_macro.xacro" />
-  <xacro:include filename="$(find ar_description)/urdf/ar.ros2_control.xacro" />
-  <xacro:include filename="$(find ar_description)/urdf/ar_gripper.ros2_control.xacro" />
+  <xacro:include filename="$(find annin_ar4_description)/urdf/ar_macro.xacro" />
+  <xacro:include filename="$(find annin_ar4_description)/urdf/ar_gripper_macro.xacro" />
+  <xacro:include filename="$(find annin_ar4_description)/urdf/ar.ros2_control.xacro" />
+  <xacro:include filename="$(find annin_ar4_description)/urdf/ar_gripper.ros2_control.xacro" />
   <xacro:arg name="simulation_controllers" default="" />
   <link name="world" />
   <xacro:ar_robot
     parent="world"
-    robot_parameters_file="$(find ar_description)/config/$(arg ar_model).yaml"
+    robot_parameters_file="$(find annin_ar4_description)/config/$(arg ar_model).yaml"
   >
     <origin xyz="0 0 0" rpy="0 0 0" />
@@ -19,7 +19,7 @@
     serial_port="None"
     calibrate="False"
-    robot_parameters_file="$(find ar_description)/config/$(arg ar_model).yaml"
-    joint_offset_parameters_file="$(find ar_hardware_interface)/config/joint_offsets/$(arg ar_model).yaml"
-    driver_parameters_file="$(find ar_hardware_interface)/config/driver.yaml"
+    robot_parameters_file="$(find annin_ar4_description)/config/$(arg ar_model).yaml"
+    joint_offset_parameters_file="$(find annin_ar4_driver)/config/joint_offsets/$(arg ar_model).yaml"
+    driver_parameters_file="$(find annin_ar4_driver)/config/driver.yaml"
   />
   <xacro:ar_gripper_ros2_control

File: ar_description/urdf/ar_gripper_macro.xacro (robot description, xacro)
@@ -10,5 +10,5 @@
       <visual>
         <geometry>
-          <mesh filename="file://$(find ar_description)/meshes/ar4_gripper/gripper_base_link.stl" />
+          <mesh filename="file://$(find annin_ar4_description)/meshes/ar4_gripper/gripper_base_link.stl" />
         </geometry>
         <material name="">
@@ -18,5 +18,5 @@
       <collision>
         <geometry>
-          <mesh filename="file://$(find ar_description)/meshes/ar4_gripper/gripper_base_link.stl" />
+          <mesh filename="file://$(find annin_ar4_description)/meshes/ar4_gripper/gripper_base_link.stl" />
         </geometry>
       </collision>
@@ -30,5 +30,5 @@
       <visual>
         <geometry>
-          <mesh filename="file://$(find ar_description)/meshes/ar4_gripper/gripper_jaw1_link.stl" />
+          <mesh filename="file://$(find annin_ar4_description)/meshes/ar4_gripper/gripper_jaw1_link.stl" />
         </geometry>
         <material name="">
@@ -38,5 +38,5 @@
       <collision>
         <geometry>
-          <mesh filename="file://$(find ar_description)/meshes/ar4_gripper/gripper_jaw1_link.stl" />
+          <mesh filename="file://$(find annin_ar4_description)/meshes/ar4_gripper/gripper_jaw1_link.stl" />
         </geometry>
       </collision>
@@ -50,5 +50,5 @@
       <visual>
         <geometry>
-          <mesh filename="file://$(find ar_description)/meshes/ar4_gripper/gripper_jaw2_link.stl" />
+          <mesh filename="file://$(find annin_ar4_description)/meshes/ar4_gripper/gripper_jaw2_link.stl" />
         </geometry>
         <material name="">
@@ -58,5 +58,5 @@
       <collision>
         <geometry>
-          <mesh filename="file://$(find ar_description)/meshes/ar4_gripper/gripper_jaw2_link.stl" />
+          <mesh filename="file://$(find annin_ar4_description)/meshes/ar4_gripper/gripper_jaw2_link.stl" />
         </geometry>
       </collision>

File: ar_description/urdf/ar_macro.xacro (robot description, xacro)
@@ -21,14 +21,14 @@
         <origin rpy="0 0 0" xyz="0 0 0"/>
         <geometry>
-          <mesh filename="file://$(find ar_description)/meshes/${robot_parameters['mesh_dir']}/base_link.STL"/>
-        </geometry>
-        <material name="">
-          <color rgba="1 1 0 1"/>
-        </material>
-      </visual>
-      <collision>
-        <origin rpy="0 0 0" xyz="0 0 0"/>
-        <geometry>
-          <mesh filename="file://$(find ar_description)/meshes/${robot_parameters['mesh_dir']}/base_link.STL"/>
+          <mesh filename="file://$(find annin_ar4_description)/meshes/${robot_parameters['mesh_dir']}/base_link.STL"/>
+        </geometry>
+        <material name="">
+          <color rgba="1 1 0 1"/>
+        </material>
+      </visual>
+      <collision>
+        <origin rpy="0 0 0" xyz="0 0 0"/>
+        <geometry>
+          <mesh filename="file://$(find annin_ar4_description)/meshes/${robot_parameters['mesh_dir']}/base_link.STL"/>
         </geometry>
       </collision>
@@ -43,14 +43,14 @@
         <origin rpy="0 0 0" xyz="0 0 0"/>
         <geometry>
-          <mesh filename="file://$(find ar_description)/meshes/${robot_parameters['mesh_dir']}/link_1.STL"/>
-        </geometry>
-        <material name="">
-          <color rgba="1 1 0 1"/>
-        </material>
-      </visual>
-      <collision>
-        <origin rpy="0 0 0" xyz="0 0 0"/>
-        <geometry>
-          <mesh filename="file://$(find ar_description)/meshes/${robot_parameters['mesh_dir']}/link_1.STL"/>
+          <mesh filename="file://$(find annin_ar4_description)/meshes/${robot_parameters['mesh_dir']}/link_1.STL"/>
+        </geometry>
+        <material name="">
+          <color rgba="1 1 0 1"/>
+        </material>
+      </visual>
+      <collision>
+        <origin rpy="0 0 0" xyz="0 0 0"/>
+        <geometry>
+          <mesh filename="file://$(find annin_ar4_description)/meshes/${robot_parameters['mesh_dir']}/link_1.STL"/>
         </geometry>
       </collision>
@@ -77,14 +77,14 @@
         <origin rpy="0 0 0" xyz="0 0 0"/>
         <geometry>
-          <mesh filename="file://$(find ar_description)/meshes/${robot_parameters['mesh_dir']}/link_2.STL"/>
-        </geometry>
-        <material name="">
-          <color rgba="1 1 0 1"/>
-        </material>
-      </visual>
-      <collision>
-        <origin rpy="0 0 0" xyz="0 0 0"/>
-        <geometry>
-          <mesh filename="file://$(find ar_description)/meshes/${robot_parameters['mesh_dir']}/link_2.STL"/>
+          <mesh filename="file://$(find annin_ar4_description)/meshes/${robot_parameters['mesh_dir']}/link_2.STL"/>
+        </geometry>
+        <material name="">
+          <color rgba="1 1 0 1"/>
+        </material>
+      </visual>
+      <collision>
+        <origin rpy="0 0 0" xyz="0 0 0"/>
+        <geometry>
+          <mesh filename="file://$(find annin_ar4_description)/meshes/${robot_parameters['mesh_dir']}/link_2.STL"/>
         </geometry>
       </collision>
@@ -111,14 +111,14 @@
         <origin rpy="0 0 0" xyz="0 0 0"/>
         <geometry>
-          <mesh filename="file://$(find ar_description)/meshes/${robot_parameters['mesh_dir']}/link_3.STL"/>
-        </geometry>
-        <material name="">
-          <color rgba="1 1 0 1"/>
-        </material>
-      </visual>
-      <collision>
-        <origin rpy="0 0 0" xyz="0 0 0"/>
-        <geometry>
-          <mesh filename="file://$(find ar_description)/meshes/${robot_parameters['mesh_dir']}/link_3.STL"/>
+          <mesh filename="file://$(find annin_ar4_description)/meshes/${robot_parameters['mesh_dir']}/link_3.STL"/>
+        </geometry>
+        <material name="">
+          <color rgba="1 1 0 1"/>
+        </material>
+      </visual>
+      <collision>
+        <origin rpy="0 0 0" xyz="0 0 0"/>
+        <geometry>
+          <mesh filename="file://$(find annin_ar4_description)/meshes/${robot_parameters['mesh_dir']}/link_3.STL"/>
         </geometry>
       </collision>
@@ -145,14 +145,14 @@
         <origin rpy="0 0 0" xyz="0 0 0"/>
         <geometry>
-          <mesh filename="file://$(find ar_description)/meshes/${robot_parameters['mesh_dir']}/link_4.STL"/>
-        </geometry>
-        <material name="">
-          <color rgba="1 1 0 1"/>
-        </material>
-      </visual>
-      <collision>
-        <origin rpy="0 0 0" xyz="0 0 0"/>
-        <geometry>
-          <mesh filename="file://$(find ar_description)/meshes/${robot_parameters['mesh_dir']}/link_4.STL"/>
+          <mesh filename="file://$(find annin_ar4_description)/meshes/${robot_parameters['mesh_dir']}/link_4.STL"/>
+        </geometry>
+        <material name="">
+          <color rgba="1 1 0 1"/>
+        </material>
+      </visual>
+      <collision>
+        <origin rpy="0 0 0" xyz="0 0 0"/>
+        <geometry>
+          <mesh filename="file://$(find annin_ar4_description)/meshes/${robot_parameters['mesh_dir']}/link_4.STL"/>
         </geometry>
       </collision>
@@ -179,14 +179,14 @@
         <origin rpy="0 0 0" xyz="0 0 0"/>
         <geometry>
-          <mesh filename="file://$(find ar_description)/meshes/${robot_parameters['mesh_dir']}/link_5.STL"/>
-        </geometry>
-        <material name="">
-          <color rgba="1 1 0 1"/>
-        </material>
-      </visual>
-      <collision>
-        <origin rpy="0 0 0" xyz="0 0 0"/>
-        <geometry>
-          <mesh filename="file://$(find ar_description)/meshes/${robot_parameters['mesh_dir']}/link_5.STL"/>
+          <mesh filename="file://$(find annin_ar4_description)/meshes/${robot_parameters['mesh_dir']}/link_5.STL"/>
+        </geometry>
+        <material name="">
+          <color rgba="1 1 0 1"/>
+        </material>
+      </visual>
+      <collision>
+        <origin rpy="0 0 0" xyz="0 0 0"/>
+        <geometry>
+          <mesh filename="file://$(find annin_ar4_description)/meshes/${robot_parameters['mesh_dir']}/link_5.STL"/>
         </geometry>
       </collision>
@@ -213,14 +213,14 @@
         <origin rpy="0 0 0" xyz="0 0 0"/>
         <geometry>
-          <mesh filename="file://$(find ar_description)/meshes/${robot_parameters['mesh_dir']}/link_6.STL"/>
-        </geometry>
-        <material name="">
-          <color rgba="1 1 0 1"/>
-        </material>
-      </visual>
-      <collision>
-        <origin rpy="0 0 0" xyz="0 0 0"/>
-        <geometry>
-          <mesh filename="file://$(find ar_description)/meshes/${robot_parameters['mesh_dir']}/link_6.STL"/>
+          <mesh filename="file://$(find annin_ar4_description)/meshes/${robot_parameters['mesh_dir']}/link_6.STL"/>
+        </geometry>
+        <material name="">
+          <color rgba="1 1 0 1"/>
+        </material>
+      </visual>
+      <collision>
+        <origin rpy="0 0 0" xyz="0 0 0"/>
+        <geometry>
+          <mesh filename="file://$(find annin_ar4_description)/meshes/${robot_parameters['mesh_dir']}/link_6.STL"/>
         </geometry>
       </collision>

File: ar_hardware_interface/urdf/ar.urdf.xacro (robot description, xacro)
@@ -5,10 +5,10 @@
   <xacro:arg name="calibrate" default="True"/>
   <xacro:arg name="include_gripper" default="true"/>
-  <xacro:include filename="$(find ar_description)/urdf/ar_macro.xacro"/>
-  <xacro:include filename="$(find ar_description)/urdf/ar.ros2_control.xacro"/>
+  <xacro:include filename="$(find annin_ar4_description)/urdf/ar_macro.xacro"/>
+  <xacro:include filename="$(find annin_ar4_description)/urdf/ar.ros2_control.xacro"/>
   <link name="world" />
   <xacro:ar_robot
     parent="world"
-    robot_parameters_file="$(find ar_description)/config/$(arg ar_model).yaml"
+    robot_parameters_file="$(find annin_ar4_description)/config/$(arg ar_model).yaml"
   >
     <origin xyz="0 0 0" rpy="0 0 0" />
@@ -16,18 +16,18 @@
   <xacro:ar_ros2_control
     ar_model="$(arg ar_model)"
-    plugin_name="ar_hardware_interface/ARHardwareInterface"
+    plugin_name="annin_ar4_driver/ARHardwareInterface"
     serial_port="$(arg serial_port)"
     calibrate="$(arg calibrate)"
-    robot_parameters_file="$(find ar_description)/config/$(arg ar_model).yaml"
-    joint_offset_parameters_file="$(find ar_hardware_interface)/config/joint_offsets/$(arg ar_model).yaml"
-    driver_parameters_file="$(find ar_hardware_interface)/config/driver.yaml"
+    robot_parameters_file="$(find annin_ar4_description)/config/$(arg ar_model).yaml"
+    joint_offset_parameters_file="$(find annin_ar4_driver)/config/joint_offsets/$(arg ar_model).yaml"
+    driver_parameters_file="$(find annin_ar4_driver)/config/driver.yaml"
   />
   <xacro:if value="$(arg include_gripper)">
-    <xacro:include filename="$(find ar_description)/urdf/ar_gripper_macro.xacro"/>
-    <xacro:include filename="$(find ar_description)/urdf/ar_gripper.ros2_control.xacro"/>
+    <xacro:include filename="$(find annin_ar4_description)/urdf/ar_gripper_macro.xacro"/>
+    <xacro:include filename="$(find annin_ar4_description)/urdf/ar_gripper.ros2_control.xacro"/>
     <xacro:ar_gripper parent="ee_link" />
     <xacro:ar_gripper_ros2_control
       name="ar_servo_gripper"
-      plugin_name="ar_hardware_interface/ARServoGripperHWInterface"
+      plugin_name="annin_ar4_driver/ARServoGripperHWInterface"
       serial_port="$(arg arduino_serial_port)"
     />

File: ar_moveit_config/srdf/ar.srdf.xacro (robot description, xacro)
@@ -2,8 +2,8 @@
 <robot xmlns:xacro="http://wiki.ros.org/xacro" name="$(arg name)">
   <xacro:arg name="include_gripper" default="true"/>
-  <xacro:include filename="$(find ar_moveit_config)/srdf/ar_macro.srdf.xacro"/>
+  <xacro:include filename="$(find annin_ar4_moveit_config)/srdf/ar_macro.srdf.xacro"/>
   <xacro:ar_srdf />
   <xacro:if value="$(arg include_gripper)">
-    <xacro:include filename="$(find ar_moveit_config)/srdf/ar_gripper_macro.srdf.xacro"/>
+    <xacro:include filename="$(find annin_ar4_moveit_config)/srdf/ar_gripper_macro.srdf.xacro"/>
     <xacro:ar_gripper_srdf />
   </xacro:if>

File: ar_moveit_config/urdf/fake_ar.urdf.xacro (robot description, xacro)
@@ -1,12 +1,12 @@
 <?xml version="1.0"?>
 <robot xmlns:xacro="http://wiki.ros.org/xacro" name="$(arg ar_model)">
-  <xacro:include filename="$(find ar_description)/urdf/ar_macro.xacro"/>
-  <xacro:include filename="$(find ar_description)/urdf/ar_gripper_macro.xacro"/>
-  <xacro:include filename="$(find ar_description)/urdf/ar.ros2_control.xacro"/>
-  <xacro:include filename="$(find ar_description)/urdf/ar_gripper.ros2_control.xacro"/>
+  <xacro:include filename="$(find annin_ar4_description)/urdf/ar_macro.xacro"/>
+  <xacro:include filename="$(find annin_ar4_description)/urdf/ar_gripper_macro.xacro"/>
+  <xacro:include filename="$(find annin_ar4_description)/urdf/ar.ros2_control.xacro"/>
+  <xacro:include filename="$(find annin_ar4_description)/urdf/ar_gripper.ros2_control.xacro"/>
   <link name="world" />
   <xacro:ar_robot
     parent="world"
-    robot_parameters_file="$(find ar_description)/config/$(arg ar_model).yaml"
+    robot_parameters_file="$(find annin_ar4_description)/config/$(arg ar_model).yaml"
   >
     <origin xyz="0 0 0" rpy="0 0 0" />
@@ -18,7 +18,7 @@
     serial_port="/dev/ttyACM0"
     calibrate="False"
-    robot_parameters_file="$(find ar_description)/config/$(arg ar_model).yaml"
-    joint_offset_parameters_file="$(find ar_hardware_interface)/config/joint_offsets/$(arg ar_model).yaml"
-    driver_parameters_file="$(find ar_hardware_interface)/config/driver.yaml"
+    robot_parameters_file="$(find annin_ar4_description)/config/$(arg ar_model).yaml"
+    joint_offset_parameters_file="$(find annin_ar4_driver)/config/joint_offsets/$(arg ar_model).yaml"
+    driver_parameters_file="$(find annin_ar4_driver)/config/driver.yaml"
   />
   <xacro:ar_gripper_ros2_control
