Commit message: read joint offsets from file

File: ar_description/urdf/ar.ros2_control.xacro (robot description, xacro)
@@ -6,5 +6,8 @@
     serial_port
     calibrate
+    joint_offset_parameters_file
   ">
+    <xacro:property name="joint_offset_parameters"
+      value="${xacro.load_yaml(joint_offset_parameters_file)}"/>
     <ros2_control name="${name}" type="system">
       <hardware>
@@ -21,4 +24,5 @@
           <param name="initial_value">0.0</param>
         </state_interface>
+        <param name="position_offset">${joint_offset_parameters['joint_1']}</param>
       </joint>
       <joint name="joint_2">
@@ -30,4 +34,5 @@
           <param name="initial_value">0.0</param>
         </state_interface>
+        <param name="position_offset">${joint_offset_parameters['joint_2']}</param>
       </joint>
       <joint name="joint_3">
@@ -39,4 +44,5 @@
           <param name="initial_value">0.0</param>
         </state_interface>
+        <param name="position_offset">${joint_offset_parameters['joint_3']}</param>
       </joint>
       <joint name="joint_4">
@@ -48,4 +54,5 @@
           <param name="initial_value">0.0</param>
         </state_interface>
+        <param name="position_offset">${joint_offset_parameters['joint_4']}</param>
       </joint>
       <joint name="joint_5">
@@ -57,4 +64,5 @@
           <param name="initial_value">0.0</param>
         </state_interface>
+        <param name="position_offset">${joint_offset_parameters['joint_5']}</param>
       </joint>
       <joint name="joint_6">
@@ -66,4 +74,5 @@
           <param name="initial_value">0.0</param>
         </state_interface>
+        <param name="position_offset">${joint_offset_parameters['joint_6']}</param>
       </joint>
     </ros2_control>

File: ar_hardware_interface/urdf/ar.urdf.xacro (robot description, xacro)
@@ -16,4 +16,5 @@
     serial_port="$(arg serial_port)"
     calibrate="$(arg calibrate)"
+    joint_offset_parameters_file="$(find ar_hardware_interface)/config/joint_offsets.yaml"
   />
   <xacro:if value="$(arg include_gripper)">

Commit message: Include gripper y/n in gazebo

File: ar_description/urdf/ar.ros2_control.xacro (robot description, xacro)
@@ -1,5 +1,6 @@
 <?xml version="1.0"?>
 <robot xmlns:xacro="http://www.ros.org/wiki/xacro">
-  <xacro:macro name="ar_ros2_control" params="
+  <xacro:macro name="ar_ros2_control"
+    params="
     name
     plugin_name
@@ -12,5 +13,8 @@
       value="${xacro.load_yaml(robot_parameters_file)}"/>
     <xacro:property name="joint_offset_parameters"
-      value="${xacro.load_yaml(joint_offset_parameters_file)}"/>
+      value="${xacro.load_yaml(joint_offset_parameters_file)}" />
+    <xacro:property name="robot_parameters_file"
+      value="$(find ar_description)/config/$(arg ar_model).yaml" />
+    <xacro:property name="robot_parameters" value="${xacro.load_yaml(robot_parameters_file)}" />
     <ros2_control name="${name}" type="system">
       <hardware>

File: ar_description/urdf/ar_gazebo.urdf.xacro (robot description, xacro)
@@ -1,17 +1,12 @@
 <?xml version="1.0"?>
 <robot xmlns:xacro="http://wiki.ros.org/xacro" name="$(arg ar_model)">
-  <xacro:include filename="$(find ar_description)/urdf/ar_macro.xacro" />
-  <xacro:include filename="$(find ar_description)/urdf/ar_gripper_macro.xacro" />
+  <xacro:arg name="simulation_controllers" default="" />
+  <xacro:arg name="include_gripper" default="True" />
+  <xacro:arg name="include_track" default="True" />
+  <xacro:include filename="$(find ar_description)/urdf/ar.urdf.xacro" />
+  <!--<xacro:include
+  filename="$(find ar_description)/urdf/ar_macro.xacro" />-->
   <xacro:include filename="$(find ar_description)/urdf/ar.ros2_control.xacro" />
   <xacro:include filename="$(find ar_description)/urdf/ar_gripper.ros2_control.xacro" />
-  <xacro:arg name="simulation_controllers" default="" />
-  <link name="world" />
-  <xacro:ar_robot
-    parent="world"
-    robot_parameters_file="$(find ar_description)/config/$(arg ar_model).yaml"
-  >
-    <origin xyz="0 0 0" rpy="0 0 0" />
-  </xacro:ar_robot>
-  <xacro:ar_gripper parent="ee_link" />
   <xacro:ar_ros2_control
     name="ARGazeboSystem"
@@ -22,9 +17,11 @@
     joint_offset_parameters_file="$(find ar_hardware_interface)/config/joint_offsets/$(arg ar_model).yaml"
   />
-  <xacro:ar_gripper_ros2_control
-    name="ARGripperGazeboSystem"
-    plugin_name="gazebo_ros2_control/GazeboSystem"
-    serial_port="None"
-  />
+  <xacro:if value="$(arg include_gripper)">
+    <xacro:ar_gripper_ros2_control
+      name="ARGripperGazeboSystem"
+      plugin_name="gazebo_ros2_control/GazeboSystem"
+      serial_port="None"
+    />
+  </xacro:if>
   <gazebo reference="world" />
   <gazebo>

Commit message: read j4 and j6 limits from config in ar.ros2_control.xacro

File: ar_description/urdf/ar.ros2_control.xacro (robot description, xacro)
@@ -6,6 +6,9 @@
     serial_port
     calibrate
+    robot_parameters_file
     joint_offset_parameters_file
   ">
+    <xacro:property name="robot_parameters"
+      value="${xacro.load_yaml(robot_parameters_file)}"/>
     <xacro:property name="joint_offset_parameters"
       value="${xacro.load_yaml(joint_offset_parameters_file)}"/>
@@ -48,6 +51,6 @@
       <joint name="joint_4">
         <command_interface name="position">
-          <param name="min">{-165*pi/180}</param>
-          <param name="max">{165*pi/180}</param>
+          <param name="min">${-robot_parameters['j4_limit']}</param>
+          <param name="max">${robot_parameters['j4_limit']}</param>
         </command_interface>
         <state_interface name="position">
@@ -68,6 +71,6 @@
       <joint name="joint_6">
         <command_interface name="position">
-          <param name="min">{-155*pi/180}</param>
-          <param name="max">{155*pi/180}</param>
+          <param name="min">${-robot_parameters['j4_limit']}</param>
+          <param name="max">${robot_parameters['j6_limit']}</param>
         </command_interface>
         <state_interface name="position">

File: ar_description/urdf/ar_gazebo.urdf.xacro (robot description, xacro)
@@ -19,4 +19,5 @@
     serial_port="None"
     calibrate="False"
+    robot_parameters_file="$(find ar_description)/config/$(arg ar_model).yaml"
     joint_offset_parameters_file="$(find ar_hardware_interface)/config/joint_offsets/$(arg ar_model).yaml"
   />

File: ar_hardware_interface/urdf/ar.urdf.xacro (robot description, xacro)
@@ -19,4 +19,5 @@
     serial_port="$(arg serial_port)"
     calibrate="$(arg calibrate)"
+    robot_parameters_file="$(find ar_description)/config/$(arg ar_model).yaml"
     joint_offset_parameters_file="$(find ar_hardware_interface)/config/joint_offsets/$(arg ar_model).yaml"
   />

File: ar_moveit_config/urdf/fake_ar.urdf.xacro (robot description, xacro)
@@ -18,4 +18,5 @@
     serial_port="/dev/ttyACM0"
     calibrate="False"
+    robot_parameters_file="$(find ar_description)/config/$(arg ar_model).yaml"
     joint_offset_parameters_file="$(find ar_hardware_interface)/config/joint_offsets/$(arg ar_model).yaml"
   />

Commit message: use robot parameters for every joint limit

File: ar_description/urdf/ar.ros2_control.xacro (robot description, xacro)
@@ -22,6 +22,6 @@
       <joint name="joint_1">
         <command_interface name="position">
-          <param name="min">{-170*pi/180}</param>
-          <param name="max">{170*pi/180}</param>
+          <param name="min">${robot_parameters['j1_limit_min']}</param>
+          <param name="max">${robot_parameters['j1_limit_max']}</param>
         </command_interface>
         <state_interface name="position">
@@ -32,6 +32,6 @@
       <joint name="joint_2">
         <command_interface name="position">
-          <param name="min">{-42*pi/180}</param>
-          <param name="max">{90*pi/180}</param>
+          <param name="min">${robot_parameters['j2_limit_min']}</param>
+          <param name="max">${robot_parameters['j2_limit_max']}</param>
         </command_interface>
         <state_interface name="position">
@@ -42,6 +42,6 @@
       <joint name="joint_3">
         <command_interface name="position">
-          <param name="min">{-89*pi/180}</param>
-          <param name="max">{52*pi/180}</param>
+          <param name="min">${robot_parameters['j3_limit_min']}</param>
+          <param name="max">${robot_parameters['j3_limit_max']}</param>
         </command_interface>
         <state_interface name="position">
@@ -52,6 +52,6 @@
       <joint name="joint_4">
         <command_interface name="position">
-          <param name="min">${-robot_parameters['j4_limit']}</param>
-          <param name="max">${robot_parameters['j4_limit']}</param>
+          <param name="min">${robot_parameters['j4_limit_min']}</param>
+          <param name="max">${robot_parameters['j4_limit_max']}</param>
         </command_interface>
         <state_interface name="position">
@@ -62,6 +62,6 @@
       <joint name="joint_5">
         <command_interface name="position">
-          <param name="min">{-105*pi/180}</param>
-          <param name="max">{105*pi/180}</param>
+          <param name="min">${robot_parameters['j5_limit_min']}</param>
+          <param name="max">${robot_parameters['j5_limit_max']}</param>
         </command_interface>
         <state_interface name="position">
@@ -72,6 +72,6 @@
       <joint name="joint_6">
         <command_interface name="position">
-          <param name="min">${-robot_parameters['j6_limit']}</param>
-          <param name="max">${robot_parameters['j6_limit']}</param>
+          <param name="min">${robot_parameters['j6_limit_min']}</param>
+          <param name="max">${robot_parameters['j6_limit_max']}</param>
         </command_interface>
         <state_interface name="position">

File: ar_description/urdf/ar_gripper.ros2_control.xacro (robot description, xacro)
@@ -23,5 +23,4 @@
         <param name="mimic">gripper_jaw1_joint</param>
         <param name="multiplier">1</param>
-        <command_interface name="position" />
         <state_interface name="position">
           <param name="initial_value">0.0</param>

File: ar_description/urdf/ar_macro.xacro (robot description, xacro)
@@ -61,5 +61,5 @@
       <child link="link_1"/>
       <axis xyz="0 0 1"/>
-      <limit lower="${-170.0 / 180.0 * pi}" upper="${170.0 / 180.0 * pi}" effort="0" velocity="0.5"/>
+      <limit lower="${robot_parameters['j1_limit_min']}" upper="${robot_parameters['j1_limit_max']}" effort="0" velocity="0.5"/>
     </joint>
     <link name="link_2">
@@ -90,5 +90,5 @@
       <child link="link_2"/>
       <axis xyz="0 0 -1"/>
-      <limit lower="${-42.0 / 180.0 * pi}" upper="${90.0 / 180.0 * pi}" effort="0.5" velocity="0.5"/>
+      <limit lower="${robot_parameters['j2_limit_min']}" upper="${robot_parameters['j2_limit_max']}" effort="0.5" velocity="0.5"/>
     </joint>
     <link name="link_3">
@@ -119,5 +119,5 @@
       <child link="link_3"/>
       <axis xyz="0 0 -1"/>
-      <limit lower="${-89.0 / 180.0 * pi}" upper="${52.0 / 180.0 * pi}" effort="0" velocity="0.5"/>
+      <limit lower="${robot_parameters['j3_limit_min']}" upper="${robot_parameters['j3_limit_max']}" effort="0" velocity="0.5"/>
     </joint>
     <link name="link_4">
@@ -148,5 +148,5 @@
       <child link="link_4"/>
       <axis xyz="0 0 -1"/>
-      <limit lower="${-1 * robot_parameters['j4_limit']}" upper="${robot_parameters['j4_limit']}" effort="0" velocity="0.5"/>
+      <limit lower="${robot_parameters['j4_limit_min']}" upper="${robot_parameters['j4_limit_max']}" effort="0" velocity="0.5"/>
     </joint>
     <link name="link_5">
@@ -177,5 +177,5 @@
       <child link="link_5"/>
       <axis xyz="1 0 0"/>
-      <limit lower="${-105.0 / 180.0 * pi}" upper="${105.0 / 180.0 * pi}" effort="0" velocity="1.0"/>
+      <limit lower="${robot_parameters['j5_limit_min']}" upper="${robot_parameters['j5_limit_max']}" effort="0" velocity="1.0"/>
     </joint>
     <link name="link_6">
@@ -206,5 +206,5 @@
       <child link="link_6"/>
       <axis xyz="0 0 1"/>
-      <limit lower="${-1.0 * robot_parameters['j6_limit']}" upper="${robot_parameters['j6_limit']}" effort="0" velocity="1.0"/>
+      <limit lower="${robot_parameters['j6_limit_min']}" upper="${robot_parameters['j6_limit_max']}" effort="0" velocity="1.0"/>
     </joint>
     <!-- center of the end effector mounting surface on link_6 -->

Commit message: velocity control

File: ar_description/urdf/ar.ros2_control.xacro (robot description, xacro)
@@ -8,4 +8,5 @@
     robot_parameters_file
     joint_offset_parameters_file
+    driver_parameters_file
   ">
     <xacro:property name="robot_parameters"
@@ -13,4 +14,6 @@
     <xacro:property name="joint_offset_parameters"
       value="${xacro.load_yaml(joint_offset_parameters_file)}"/>
+    <xacro:property name="driver_parameters"
+      value="${xacro.load_yaml(driver_parameters_file)}"/>
     <ros2_control name="${ar_model}" type="system">
       <hardware>
@@ -19,4 +22,5 @@
         <param name="serial_port">${serial_port}</param>
         <param name="calibrate">${calibrate}</param>
+        <param name="velocity_control_enabled">${driver_parameters['velocity_control_enabled']}</param>
       </hardware>
       <joint name="joint_1">
@@ -25,5 +29,9 @@
           <param name="max">${robot_parameters['j1_limit_max']}</param>
         </command_interface>
+        <command_interface name="velocity" />
         <state_interface name="position">
+          <param name="initial_value">0.0</param>
+        </state_interface>
+        <state_interface name="velocity">
           <param name="initial_value">0.0</param>
         </state_interface>
@@ -35,5 +43,9 @@
           <param name="max">${robot_parameters['j2_limit_max']}</param>
         </command_interface>
+        <command_interface name="velocity" />
         <state_interface name="position">
+          <param name="initial_value">0.0</param>
+        </state_interface>
+        <state_interface name="velocity">
           <param name="initial_value">0.0</param>
         </state_interface>
@@ -45,5 +57,9 @@
           <param name="max">${robot_parameters['j3_limit_max']}</param>
         </command_interface>
+        <command_interface name="velocity" />
         <state_interface name="position">
+          <param name="initial_value">0.0</param>
+        </state_interface>
+        <state_interface name="velocity">
           <param name="initial_value">0.0</param>
         </state_interface>
@@ -55,5 +71,9 @@
           <param name="max">${robot_parameters['j4_limit_max']}</param>
         </command_interface>
+        <command_interface name="velocity" />
         <state_interface name="position">
+          <param name="initial_value">0.0</param>
+        </state_interface>
+        <state_interface name="velocity">
           <param name="initial_value">0.0</param>
         </state_interface>
@@ -65,5 +85,9 @@
           <param name="max">${robot_parameters['j5_limit_max']}</param>
         </command_interface>
+        <command_interface name="velocity" />
         <state_interface name="position">
+          <param name="initial_value">0.0</param>
+        </state_interface>
+        <state_interface name="velocity">
           <param name="initial_value">0.0</param>
         </state_interface>
@@ -75,5 +99,9 @@
           <param name="max">${robot_parameters['j6_limit_max']}</param>
         </command_interface>
+        <command_interface name="velocity" />
         <state_interface name="position">
+          <param name="initial_value">0.0</param>
+        </state_interface>
+        <state_interface name="velocity">
           <param name="initial_value">0.0</param>
         </state_interface>

File: ar_description/urdf/ar_gazebo.urdf.xacro (robot description, xacro)
@@ -21,4 +21,5 @@
     robot_parameters_file="$(find ar_description)/config/$(arg ar_model).yaml"
     joint_offset_parameters_file="$(find ar_hardware_interface)/config/joint_offsets/$(arg ar_model).yaml"
+    driver_parameters_file="$(find ar_hardware_interface)/config/driver.yaml"
   />
   <xacro:ar_gripper_ros2_control

File: ar_description/urdf/ar_macro.xacro (robot description, xacro)
@@ -61,5 +61,10 @@
       <child link="link_1"/>
       <axis xyz="0 0 1"/>
-      <limit lower="${robot_parameters['j1_limit_min']}" upper="${robot_parameters['j1_limit_max']}" effort="0" velocity="0.5"/>
+      <limit
+        lower="${robot_parameters['j1_limit_min']}"
+        upper="${robot_parameters['j1_limit_max']}"
+        effort="-1"
+        velocity="1.0472"
+      />
     </joint>
     <link name="link_2">
@@ -90,5 +95,10 @@
       <child link="link_2"/>
       <axis xyz="0 0 -1"/>
-      <limit lower="${robot_parameters['j2_limit_min']}" upper="${robot_parameters['j2_limit_max']}" effort="0.5" velocity="0.5"/>
+      <limit
+        lower="${robot_parameters['j2_limit_min']}"
+        upper="${robot_parameters['j2_limit_max']}"
+        effort="-1"
+        velocity="1.0472"
+      />
     </joint>
     <link name="link_3">
@@ -119,5 +129,10 @@
       <child link="link_3"/>
       <axis xyz="0 0 -1"/>
-      <limit lower="${robot_parameters['j3_limit_min']}" upper="${robot_parameters['j3_limit_max']}" effort="0" velocity="0.5"/>
+      <limit
+        lower="${robot_parameters['j3_limit_min']}"
+        upper="${robot_parameters['j3_limit_max']}"
+        effort="-1"
+        velocity="1.0472"
+      />
     </joint>
     <link name="link_4">
@@ -148,5 +163,10 @@
       <child link="link_4"/>
       <axis xyz="0 0 -1"/>
-      <limit lower="${robot_parameters['j4_limit_min']}" upper="${robot_parameters['j4_limit_max']}" effort="0" velocity="0.5"/>
+      <limit
+        lower="${robot_parameters['j4_limit_min']}"
+        upper="${robot_parameters['j4_limit_max']}"
+        effort="-1"
+        velocity="1.0472"
+      />
     </joint>
     <link name="link_5">
@@ -177,5 +197,10 @@
       <child link="link_5"/>
       <axis xyz="1 0 0"/>
-      <limit lower="${robot_parameters['j5_limit_min']}" upper="${robot_parameters['j5_limit_max']}" effort="0" velocity="1.0"/>
+      <limit
+        lower="${robot_parameters['j5_limit_min']}"
+        upper="${robot_parameters['j5_limit_max']}"
+        effort="-1"
+        velocity="1.0472"
+      />
     </joint>
     <link name="link_6">
@@ -206,5 +231,10 @@
       <child link="link_6"/>
       <axis xyz="0 0 1"/>
-      <limit lower="${robot_parameters['j6_limit_min']}" upper="${robot_parameters['j6_limit_max']}" effort="0" velocity="1.0"/>
+      <limit
+        lower="${robot_parameters['j6_limit_min']}"
+        upper="${robot_parameters['j6_limit_max']}"
+        effort="-1"
+        velocity="1.0472"
+      />
     </joint>
     <!-- center of the end effector mounting surface on link_6 -->

File: ar_hardware_interface/urdf/ar.urdf.xacro (robot description, xacro)
@@ -21,4 +21,5 @@
     robot_parameters_file="$(find ar_description)/config/$(arg ar_model).yaml"
     joint_offset_parameters_file="$(find ar_hardware_interface)/config/joint_offsets/$(arg ar_model).yaml"
+    driver_parameters_file="$(find ar_hardware_interface)/config/driver.yaml"
   />
   <xacro:if value="$(arg include_gripper)">

File: ar_moveit_config/srdf/ar_macro.srdf.xacro (robot description, xacro)
@@ -26,5 +26,5 @@
       <joint name="joint_1" value="0" />
       <joint name="joint_2" value="-0.087" />
-      <joint name="joint_3" value="-1.34" />
+      <joint name="joint_3" value="-1.4" />
       <joint name="joint_4" value="0" />
       <joint name="joint_5" value="0" />

File: ar_moveit_config/urdf/fake_ar.urdf.xacro (robot description, xacro)
@@ -20,4 +20,5 @@
     robot_parameters_file="$(find ar_description)/config/$(arg ar_model).yaml"
     joint_offset_parameters_file="$(find ar_hardware_interface)/config/joint_offsets/$(arg ar_model).yaml"
+    driver_parameters_file="$(find ar_hardware_interface)/config/driver.yaml"
   />
   <xacro:ar_gripper_ros2_control
