Commit message: added tf_prefix/prefix variable to .urdf and .srdf + made demo.launch.py compatible with the changes

File: ar_description/urdf/ar.ros2_control.xacro (robot description, xacro)
@@ -9,4 +9,5 @@
     joint_offset_parameters_file
     driver_parameters_file
+    tf_prefix
   ">
     <xacro:property name="robot_parameters"
@@ -23,6 +24,7 @@
         <param name="calibrate">${calibrate}</param>
         <param name="velocity_control_enabled">${driver_parameters['velocity_control_enabled']}</param>
+        <param name="tf_prefix">${tf_prefix}</param>
       </hardware>
-      <joint name="joint_1">
+      <joint name="${tf_prefix}joint_1">
         <command_interface name="position">
           <param name="min">${robot_parameters['j1_limit_min']}</param>
@@ -38,5 +40,5 @@
         <param name="position_offset">${joint_offset_parameters['joint_1']}</param>
       </joint>
-      <joint name="joint_2">
+      <joint name="${tf_prefix}joint_2">
         <command_interface name="position">
           <param name="min">${robot_parameters['j2_limit_min']}</param>
@@ -52,5 +54,5 @@
         <param name="position_offset">${joint_offset_parameters['joint_2']}</param>
       </joint>
-      <joint name="joint_3">
+      <joint name="${tf_prefix}joint_3">
         <command_interface name="position">
           <param name="min">${robot_parameters['j3_limit_min']}</param>
@@ -66,5 +68,5 @@
         <param name="position_offset">${joint_offset_parameters['joint_3']}</param>
       </joint>
-      <joint name="joint_4">
+      <joint name="${tf_prefix}joint_4">
         <command_interface name="position">
           <param name="min">${robot_parameters['j4_limit_min']}</param>
@@ -80,5 +82,5 @@
         <param name="position_offset">${joint_offset_parameters['joint_4']}</param>
       </joint>
-      <joint name="joint_5">
+      <joint name="${tf_prefix}joint_5">
         <command_interface name="position">
           <param name="min">${robot_parameters['j5_limit_min']}</param>
@@ -94,5 +96,5 @@
         <param name="position_offset">${joint_offset_parameters['joint_5']}</param>
       </joint>
-      <joint name="joint_6">
+      <joint name="${tf_prefix}joint_6">
         <command_interface name="position">
           <param name="min">${robot_parameters['j6_limit_min']}</param>

File: ar_description/urdf/ar.urdf.xacro (robot description, xacro)
@@ -1,8 +1,10 @@
 <?xml version="1.0"?>
 <robot xmlns:xacro="http://wiki.ros.org/xacro" name="$(arg ar_model)">
+  <xacro:arg name="tf_prefix" default="" />
   <xacro:arg name="include_gripper" default="true"/>
   <xacro:include filename="$(find ar_description)/urdf/ar_macro.xacro"/>
   <link name="world" />
   <xacro:ar_robot
+    tf_prefix="$(arg tf_prefix)"
     parent="world"
     robot_parameters_file="$(find ar_description)/config/$(arg ar_model).yaml"
@@ -12,5 +14,5 @@
   <xacro:if value="$(arg include_gripper)">
     <xacro:include filename="$(find ar_description)/urdf/ar_gripper_macro.xacro"/>
-    <xacro:ar_gripper parent="ee_link" />
+    <xacro:ar_gripper parent="$(arg tf_prefix)ee_link" />
   </xacro:if>
 </robot>

File: ar_description/urdf/ar_macro.xacro (robot description, xacro)
@@ -2,4 +2,5 @@
 <robot xmlns:xacro="http://wiki.ros.org/xacro">
   <xacro:macro name="ar_robot" params="
+    tf_prefix
     parent
     *origin
@@ -7,10 +8,10 @@
   ">
     <xacro:property name="robot_parameters" value="${xacro.load_yaml(robot_parameters_file)}"/>
-    <joint name="base_joint" type="fixed">
+    <joint name="${tf_prefix}base_joint" type="fixed">
       <xacro:insert_block name="origin" />
       <parent link="${parent}"/>
-      <child link="base_link" />
-    </joint>
-    <link name="base_link">
+      <child link="${tf_prefix}base_link" />
+    </joint>
+    <link name="${tf_prefix}base_link">
       <inertial>
         <origin rpy="0 0 0" xyz="-4.6941E-06 0.054174 0.038824"/>
@@ -34,5 +35,5 @@
       </collision>
     </link>
-    <link name="link_1">
+    <link name="${tf_prefix}link_1">
       <inertial>
         <origin rpy="0 0 0" xyz="-0.022706 0.04294 -0.12205"/>
@@ -56,8 +57,8 @@
       </collision>
     </link>
-    <joint name="joint_1" type="revolute">
+    <joint name="${tf_prefix}joint_1" type="revolute">
       <origin rpy="${pi} 0 0" xyz="0 0 0"/>
-      <parent link="base_link"/>
-      <child link="link_1"/>
+      <parent link="${tf_prefix}base_link"/>
+      <child link="${tf_prefix}link_1"/>
       <axis xyz="0 0 1"/>
       <limit
@@ -68,5 +69,5 @@
       />
     </joint>
-    <link name="link_2">
+    <link name="${tf_prefix}link_2">
       <inertial>
         <origin rpy="0 0 0" xyz="0.064818 -0.11189 -0.038671"/>
@@ -90,8 +91,8 @@
       </collision>
     </link>
-    <joint name="joint_2" type="revolute">
+    <joint name="${tf_prefix}joint_2" type="revolute">
       <origin rpy="1.5708 0 -1.5708" xyz="0 0.0642 -0.16977"/>
-      <parent link="link_1"/>
-      <child link="link_2"/>
+      <parent link="${tf_prefix}link_1"/>
+      <child link="${tf_prefix}link_2"/>
       <axis xyz="0 0 -1"/>
       <limit
@@ -102,5 +103,5 @@
       />
     </joint>
-    <link name="link_3">
+    <link name="${tf_prefix}link_3">
       <inertial>
         <origin rpy="0 0 0" xyz="-0.00029765 -0.023661 -0.0019125"/>
@@ -124,8 +125,8 @@
       </collision>
     </link>
-    <joint name="joint_3" type="revolute">
+    <joint name="${tf_prefix}joint_3" type="revolute">
       <origin rpy="0 0 3.1416" xyz="0 -0.305 0.007"/>
-      <parent link="link_2"/>
-      <child link="link_3"/>
+      <parent link="${tf_prefix}link_2"/>
+      <child link="${tf_prefix}link_3"/>
       <axis xyz="0 0 -1"/>
       <limit
@@ -136,5 +137,5 @@
       />
     </joint>
-    <link name="link_4">
+    <link name="${tf_prefix}link_4">
       <inertial>
         <origin rpy="0 0 0" xyz="-0.0016798 -0.00057319 -0.074404"/>
@@ -158,8 +159,8 @@
       </collision>
     </link>
-    <joint name="joint_4" type="revolute">
+    <joint name="${tf_prefix}joint_4" type="revolute">
       <origin rpy="1.5708 0 -1.5708" xyz="0 0 0.0"/>
-      <parent link="link_3"/>
-      <child link="link_4"/>
+      <parent link="${tf_prefix}link_3"/>
+      <child link="${tf_prefix}link_4"/>
       <axis xyz="0 0 -1"/>
       <limit
@@ -170,5 +171,5 @@
       />
     </joint>
-    <link name="link_5">
+    <link name="${tf_prefix}link_5">
       <inertial>
         <origin rpy="0 0 0" xyz="0.0015066 -1.3102E-05 -0.012585"/>
@@ -192,8 +193,8 @@
       </collision>
     </link>
-    <joint name="joint_5" type="revolute">
+    <joint name="${tf_prefix}joint_5" type="revolute">
       <origin rpy="${pi} 0 -1.5708" xyz="0 0 -0.22263"/>
-      <parent link="link_4"/>
-      <child link="link_5"/>
+      <parent link="${tf_prefix}link_4"/>
+      <child link="${tf_prefix}link_5"/>
       <axis xyz="1 0 0"/>
       <limit
@@ -204,5 +205,5 @@
       />
     </joint>
-    <link name="link_6">
+    <link name="${tf_prefix}link_6">
       <inertial>
         <origin rpy="0 0 0" xyz="2.9287E-10 -1.6472E-09 0.0091432"/>
@@ -226,8 +227,8 @@
       </collision>
     </link>
-    <joint name="joint_6" type="revolute">
+    <joint name="${tf_prefix}joint_6" type="revolute">
       <origin rpy="0 0 3.1416" xyz="0.000 0 ${robot_parameters['l6_length']}"/>
-      <parent link="link_5"/>
-      <child link="link_6"/>
+      <parent link="${tf_prefix}link_5"/>
+      <child link="${tf_prefix}link_6"/>
       <axis xyz="0 0 1"/>
       <limit
@@ -239,8 +240,8 @@
     </joint>
     <!-- center of the end effector mounting surface on link_6 -->
-    <link name="ee_link" />
-    <joint name="ee_joint" type="fixed">
-      <parent link="link_6" />
-      <child link="ee_link" />
+    <link name="${tf_prefix}ee_link" />
+    <joint name="${tf_prefix}ee_joint" type="fixed">
+      <parent link="${tf_prefix}link_6" />
+      <child link="${tf_prefix}ee_link" />
       <origin xyz="0 0 0.0" rpy="0 0 0" />
     </joint>

File: ar_moveit_config/srdf/ar.srdf.xacro (robot description, xacro)
@@ -2,9 +2,10 @@
 <robot xmlns:xacro="http://wiki.ros.org/xacro" name="$(arg name)">
   <xacro:arg name="include_gripper" default="true"/>
+  <xacro:arg name="prefix" default="" />
   <xacro:include filename="$(find ar_moveit_config)/srdf/ar_macro.srdf.xacro"/>
-  <xacro:ar_srdf />
+  <xacro:ar_srdf prefix="$(arg prefix)"/>
   <xacro:if value="$(arg include_gripper)">
     <xacro:include filename="$(find ar_moveit_config)/srdf/ar_gripper_macro.srdf.xacro"/>
-    <xacro:ar_gripper_srdf />
+    <xacro:ar_gripper_srdf prefix="$(arg prefix)"/>
   </xacro:if>
 </robot>

File: ar_moveit_config/srdf/ar_gripper_macro.srdf.xacro (robot description, xacro)
@@ -5,5 +5,5 @@
 -->
 <robot xmlns:xacro="http://wiki.ros.org/xacro">
-  <xacro:macro name="ar_gripper_srdf">
+  <xacro:macro name="ar_gripper_srdf" params="prefix">
     <group name="ar_gripper">
       <link name="gripper_base_link" />
@@ -22,6 +22,6 @@
     <disable_collisions link1="gripper_base_link" link2="gripper_jaw2_link" reason="Adjacent" />
     <disable_collisions link1="gripper_jaw1_link" link2="gripper_jaw2_link" reason="Default" />
-    <disable_collisions link1="link_6" link2="gripper_base_link" reason="Adjacent" />
-    <disable_collisions link1="link_5" link2="gripper_base_link" reason="Adjacent" />
+    <disable_collisions link1="${prefix}link_6" link2="gripper_base_link" reason="Adjacent" />
+    <disable_collisions link1="${prefix}link_5" link2="gripper_base_link" reason="Adjacent" />
   </xacro:macro>
 </robot>

File: ar_moveit_config/srdf/ar_macro.srdf.xacro (robot description, xacro)
@@ -5,39 +5,39 @@
 -->
 <robot xmlns:xacro="http://wiki.ros.org/xacro">
-  <xacro:macro name="ar_srdf">
+  <xacro:macro name="ar_srdf" params="prefix">
     <group name="ar_manipulator">
-      <joint name="joint_1" />
-      <joint name="joint_2" />
-      <joint name="joint_3" />
-      <joint name="joint_4" />
-      <joint name="joint_5" />
-      <joint name="joint_6" />
-      <joint name="ee_joint"/>
+      <joint name="${prefix}joint_1" />
+      <joint name="${prefix}joint_2" />
+      <joint name="${prefix}joint_3" />
+      <joint name="${prefix}joint_4" />
+      <joint name="${prefix}joint_5" />
+      <joint name="${prefix}joint_6" />
+      <joint name="${prefix}ee_joint"/>
     </group>
     <group_state name="home" group="ar_manipulator">
-      <joint name="joint_1" value="0" />
-      <joint name="joint_2" value="0" />
-      <joint name="joint_3" value="0" />
-      <joint name="joint_4" value="0" />
-      <joint name="joint_5" value="0" />
-      <joint name="joint_6" value="0" />
+      <joint name="${prefix}joint_1" value="0" />
+      <joint name="${prefix}joint_2" value="0" />
+      <joint name="${prefix}joint_3" value="0" />
+      <joint name="${prefix}joint_4" value="0" />
+      <joint name="${prefix}joint_5" value="0" />
+      <joint name="${prefix}joint_6" value="0" />
     </group_state>
     <group_state name="upright" group="ar_manipulator">
-      <joint name="joint_1" value="0" />
-      <joint name="joint_2" value="-0.087" />
-      <joint name="joint_3" value="-1.4" />
-      <joint name="joint_4" value="0" />
-      <joint name="joint_5" value="0" />
-      <joint name="joint_6" value="0" />
+      <joint name="${prefix}joint_1" value="0" />
+      <joint name="${prefix}joint_2" value="-0.087" />
+      <joint name="${prefix}joint_3" value="-1.4" />
+      <joint name="${prefix}joint_4" value="0" />
+      <joint name="${prefix}joint_5" value="0" />
+      <joint name="${prefix}joint_6" value="0" />
     </group_state>
-    <disable_collisions link1="base_link" link2="link_1" reason="Adjacent" />
-    <disable_collisions link1="link_1" link2="link_2" reason="Adjacent" />
-    <disable_collisions link1="link_1" link2="link_3" reason="Never" />
-    <disable_collisions link1="link_2" link2="link_3" reason="Adjacent" />
-    <disable_collisions link1="link_3" link2="link_4" reason="Adjacent" />
-    <disable_collisions link1="link_3" link2="link_5" reason="Never" />
-    <disable_collisions link1="link_3" link2="link_6" reason="Never" />
-    <disable_collisions link1="link_4" link2="link_5" reason="Adjacent" />
-    <disable_collisions link1="link_5" link2="link_6" reason="Adjacent" />
+    <disable_collisions link1="${prefix}base_link" link2="${prefix}link_1" reason="Adjacent" />
+    <disable_collisions link1="${prefix}link_1" link2="${prefix}link_2" reason="Adjacent" />
+    <disable_collisions link1="${prefix}link_1" link2="${prefix}link_3" reason="Never" />
+    <disable_collisions link1="${prefix}link_2" link2="${prefix}link_3" reason="Adjacent" />
+    <disable_collisions link1="${prefix}link_3" link2="${prefix}link_4" reason="Adjacent" />
+    <disable_collisions link1="${prefix}link_3" link2="${prefix}link_5" reason="Never" />
+    <disable_collisions link1="${prefix}link_3" link2="${prefix}link_6" reason="Never" />
+    <disable_collisions link1="${prefix}link_4" link2="${prefix}link_5" reason="Adjacent" />
+    <disable_collisions link1="${prefix}link_5" link2="${prefix}link_6" reason="Adjacent" />
   </xacro:macro>
 </robot>

File: ar_moveit_config/urdf/fake_ar.urdf.xacro (robot description, xacro)
@@ -5,6 +5,8 @@
   <xacro:include filename="$(find ar_description)/urdf/ar.ros2_control.xacro"/>
   <xacro:include filename="$(find ar_description)/urdf/ar_gripper.ros2_control.xacro"/>
+  <xacro:arg name="tf_prefix" default="" />
   <link name="world" />
   <xacro:ar_robot
+    tf_prefix="$(arg tf_prefix)"
     parent="world"
     robot_parameters_file="$(find ar_description)/config/$(arg ar_model).yaml"
@@ -12,5 +14,5 @@
     <origin xyz="0 0 0" rpy="0 0 0" />
   </xacro:ar_robot>
-  <xacro:ar_gripper parent="ee_link" />
+  <xacro:ar_gripper parent="$(arg tf_prefix)ee_link" />
   <xacro:ar_ros2_control
     ar_model="$(arg ar_model)"
@@ -21,4 +23,5 @@
     joint_offset_parameters_file="$(find ar_hardware_interface)/config/joint_offsets/$(arg ar_model).yaml"
     driver_parameters_file="$(find ar_hardware_interface)/config/driver.yaml"
+    tf_prefix="$(arg tf_prefix)"
   />
   <xacro:ar_gripper_ros2_control
