Commit message: add stow pos, video link, tune controller params

File: ar_moveit_config/srdf/ar_macro.srdf.xacro (robot description, xacro)
@@ -22,4 +22,12 @@
       <joint name="joint_6" value="0" />
     </group_state>
+    <group_state name="stow" group="ar_manipulator">
+      <joint name="joint_1" value="0" />
+      <joint name="joint_2" value="-9" />
+      <joint name="joint_3" value="-69" />
+      <joint name="joint_4" value="0" />
+      <joint name="joint_5" value="0" />
+      <joint name="joint_6" value="0" />
+    </group_state>
     <disable_collisions link1="base_link" link2="link_1" reason="Adjacent" />
     <disable_collisions link1="link_1" link2="link_2" reason="Adjacent" />

Commit message: update upright preset position

File: ar_moveit_config/srdf/ar_macro.srdf.xacro (robot description, xacro)
@@ -22,8 +22,8 @@
       <joint name="joint_6" value="0" />
     </group_state>
-    <group_state name="stow" group="ar_manipulator">
+    <group_state name="upright" group="ar_manipulator">
       <joint name="joint_1" value="0" />
-      <joint name="joint_2" value="-9" />
-      <joint name="joint_3" value="-69" />
+      <joint name="joint_2" value="-0.157" />
+      <joint name="joint_3" value="-1.2" />
       <joint name="joint_4" value="0" />
       <joint name="joint_5" value="0" />
