Commit message: tune upright and gripper open positions

File: ar_moveit_config/srdf/ar_gripper_macro.srdf.xacro (robot description, xacro)
@@ -14,5 +14,5 @@
     </group>
     <group_state name="open" group="ar_gripper">
-      <joint name="gripper_jaw1_joint" value="-0.014" />
+      <joint name="gripper_jaw1_joint" value="-0.012" />
     </group_state>
     <group_state name="closed" group="ar_gripper">

File: ar_moveit_config/srdf/ar_macro.srdf.xacro (robot description, xacro)
@@ -24,6 +24,6 @@
     <group_state name="upright" group="ar_manipulator">
       <joint name="joint_1" value="0" />
-      <joint name="joint_2" value="-0.157" />
-      <joint name="joint_3" value="-1.2" />
+      <joint name="joint_2" value="-0.087" />
+      <joint name="joint_3" value="-1.34" />
       <joint name="joint_4" value="0" />
       <joint name="joint_5" value="0" />
