Commit message: Adding tf_prefix to .urdf, .srdf and launch files

File: annin_ar4_description/urdf/ar.urdf.xacro (robot description, xacro)
@@ -1,8 +1,10 @@
 <?xml version="1.0"?>
 <robot xmlns:xacro="http://wiki.ros.org/xacro" name="$(arg ar_model)">
+  <xacro:arg name="tf_prefix" default="" />
   <xacro:arg name="include_gripper" default="true"/>
   <xacro:include filename="$(find annin_ar4_description)/urdf/ar_macro.xacro"/>
   <link name="world" />
   <xacro:ar_robot
+    tf_prefix="$(arg tf_prefix)"
     parent="world"
     robot_parameters_file="$(find annin_ar4_description)/config/$(arg ar_model).yaml"
@@ -12,5 +14,5 @@
   <xacro:if value="$(arg include_gripper)">
     <xacro:include filename="$(find annin_ar4_description)/urdf/ar_gripper_macro.xacro"/>
-    <xacro:ar_gripper parent="ee_link" />
+    <xacro:ar_gripper parent="$(arg tf_prefix)ee_link" />
   </xacro:if>
 </robot>

File: annin_ar4_description/urdf/ar_gazebo.urdf.xacro (robot description, xacro)
@@ -6,6 +6,8 @@
   <xacro:include filename="$(find annin_ar4_description)/urdf/ar_gripper.ros2_control.xacro" />
   <xacro:arg name="simulation_controllers" default="" />
+  <xacro:arg name="tf_prefix" default="" />
   <link name="world" />
   <xacro:ar_robot
+    tf_prefix="$(arg tf_prefix)"
     parent="world"
     robot_parameters_file="$(find annin_ar4_description)/config/$(arg ar_model).yaml"
@@ -13,5 +15,5 @@
     <origin xyz="0 0 0" rpy="0 0 0" />
   </xacro:ar_robot>
-  <xacro:ar_gripper parent="ee_link" />
+  <xacro:ar_gripper parent="$(arg tf_prefix)ee_link" />
   <xacro:ar_ros2_control
     ar_model="$(arg ar_model)"
@@ -22,4 +24,5 @@
     joint_offset_parameters_file="$(find annin_ar4_driver)/config/joint_offsets/$(arg ar_model).yaml"
     driver_parameters_file="$(find annin_ar4_driver)/config/driver.yaml"
+    tf_prefix="$(arg tf_prefix)"
   />
   <xacro:ar_gripper_ros2_control

File: annin_ar4_description/urdf/ar_macro.xacro (robot description, xacro)
@@ -2,4 +2,5 @@
 <robot xmlns:xacro="http://wiki.ros.org/xacro">
   <xacro:macro name="ar_robot" params="
+    tf_prefix
     parent
     *origin
@@ -7,10 +8,10 @@
   ">
     <xacro:property name="robot_parameters" value="${xacro.load_yaml(robot_parameters_file)}"/>
-    <joint name="base_joint" type="fixed">
+    <joint name="${tf_prefix}base_joint" type="fixed">
       <xacro:insert_block name="origin" />
       <parent link="${parent}"/>
-      <child link="base_link" />
-    </joint>
-    <link name="base_link">
+      <child link="${tf_prefix}base_link" />
+    </joint>
+    <link name="${tf_prefix}base_link">
       <inertial>
         <origin rpy="0 0 0" xyz="-4.6941E-06 0.054174 0.038824"/>
@@ -34,5 +35,5 @@
       </collision>
     </link>
-    <link name="link_1">
+    <link name="${tf_prefix}link_1">
       <inertial>
         <origin rpy="0 0 0" xyz="-0.022706 0.04294 -0.12205"/>
@@ -56,8 +57,8 @@
       </collision>
     </link>
-    <joint name="joint_1" type="revolute">
+    <joint name="${tf_prefix}joint_1" type="revolute">
       <origin rpy="${pi} 0 0" xyz="0 0 0"/>
-      <parent link="base_link"/>
-      <child link="link_1"/>
+      <parent link="${tf_prefix}base_link"/>
+      <child link="${tf_prefix}link_1"/>
       <axis xyz="0 0 1"/>
       <limit
@@ -68,5 +69,5 @@
       />
     </joint>
-    <link name="link_2">
+    <link name="${tf_prefix}link_2">
       <inertial>
         <origin rpy="0 0 0" xyz="0.064818 -0.11189 -0.038671"/>
@@ -90,8 +91,8 @@
       </collision>
     </link>
-    <joint name="joint_2" type="revolute">
+    <joint name="${tf_prefix}joint_2" type="revolute">
       <origin rpy="1.5708 0 -1.5708" xyz="0 0.0642 -0.16977"/>
-      <parent link="link_1"/>
-      <child link="link_2"/>
+      <parent link="${tf_prefix}link_1"/>
+      <child link="${tf_prefix}link_2"/>
       <axis xyz="0 0 -1"/>
       <limit
@@ -102,5 +103,5 @@
       />
     </joint>
-    <link name="link_3">
+    <link name="${tf_prefix}link_3">
       <inertial>
         <origin rpy="0 0 0" xyz="-0.00029765 -0.023661 -0.0019125"/>
@@ -124,8 +125,8 @@
       </collision>
     </link>
-    <joint name="joint_3" type="revolute">
+    <joint name="${tf_prefix}joint_3" type="revolute">
       <origin rpy="0 0 3.1416" xyz="0 -0.305 0.007"/>
-      <parent link="link_2"/>
-      <child link="link_3"/>
+      <parent link="${tf_prefix}link_2"/>
+      <child link="${tf_prefix}link_3"/>
       <axis xyz="0 0 -1"/>
       <limit
@@ -136,5 +137,5 @@
       />
     </joint>
-    <link name="link_4">
+    <link name="${tf_prefix}link_4">
       <inertial>
         <origin rpy="0 0 0" xyz="-0.0016798 -0.00057319 -0.074404"/>
@@ -158,8 +159,8 @@
       </collision>
     </link>
-    <joint name="joint_4" type="revolute">
+    <joint name="${tf_prefix}joint_4" type="revolute">
       <origin rpy="1.5708 0 -1.5708" xyz="0 0 0.0"/>
-      <parent link="link_3"/>
-      <child link="link_4"/>
+      <parent link="${tf_prefix}link_3"/>
+      <child link="${tf_prefix}link_4"/>
       <axis xyz="0 0 -1"/>
       <limit
@@ -170,5 +171,5 @@
       />
     </joint>
-    <link name="link_5">
+    <link name="${tf_prefix}link_5">
       <inertial>
         <origin rpy="0 0 0" xyz="0.0015066 -1.3102E-05 -0.012585"/>
@@ -192,8 +193,8 @@
       </collision>
     </link>
-    <joint name="joint_5" type="revolute">
+    <joint name="${tf_prefix}joint_5" type="revolute">
       <origin rpy="${pi} 0 -1.5708" xyz="0 0 -0.22263"/>
-      <parent link="link_4"/>
-      <child link="link_5"/>
+      <parent link="${tf_prefix}link_4"/>
+      <child link="${tf_prefix}link_5"/>
       <axis xyz="1 0 0"/>
       <limit
@@ -204,5 +205,5 @@
       />
     </joint>
-    <link name="link_6">
+    <link name="${tf_prefix}link_6">
       <inertial>
         <origin rpy="0 0 0" xyz="2.9287E-10 -1.6472E-09 0.0091432"/>
@@ -226,8 +227,8 @@
       </collision>
     </link>
-    <joint name="joint_6" type="revolute">
+    <joint name="${tf_prefix}joint_6" type="revolute">
       <origin rpy="0 0 3.1416" xyz="0.000 0 ${robot_parameters['l6_length']}"/>
-      <parent link="link_5"/>
-      <child link="link_6"/>
+      <parent link="${tf_prefix}link_5"/>
+      <child link="${tf_prefix}link_6"/>
       <axis xyz="0 0 1"/>
       <limit
@@ -239,8 +240,8 @@
     </joint>
     <!-- center of the end effector mounting surface on link_6 -->
-    <link name="ee_link" />
-    <joint name="ee_joint" type="fixed">
-      <parent link="link_6" />
-      <child link="ee_link" />
+    <link name="${tf_prefix}ee_link" />
+    <joint name="${tf_prefix}ee_joint" type="fixed">
+      <parent link="${tf_prefix}link_6" />
+      <child link="${tf_prefix}ee_link" />
       <origin xyz="0 0 0.0" rpy="0 0 0" />
     </joint>

File: annin_ar4_driver/urdf/ar.urdf.xacro (robot description, xacro)
@@ -4,4 +4,5 @@
   <xacro:arg name="arduino_serial_port" default="/dev/ttyUSB0"/>
   <xacro:arg name="calibrate" default="True"/>
+  <xacro:arg name="tf_prefix" default="" />
   <xacro:arg name="include_gripper" default="true"/>
   <xacro:include filename="$(find annin_ar4_description)/urdf/ar_macro.xacro"/>
@@ -9,4 +10,5 @@
   <link name="world" />
   <xacro:ar_robot
+    tf_prefix="$(arg tf_prefix)"
     parent="world"
     robot_parameters_file="$(find annin_ar4_description)/config/$(arg ar_model).yaml"
@@ -22,9 +24,10 @@
     joint_offset_parameters_file="$(find annin_ar4_driver)/config/joint_offsets/$(arg ar_model).yaml"
     driver_parameters_file="$(find annin_ar4_driver)/config/driver.yaml"
+    tf_prefix="$(arg tf_prefix)"
   />
   <xacro:if value="$(arg include_gripper)">
     <xacro:include filename="$(find annin_ar4_description)/urdf/ar_gripper_macro.xacro"/>
     <xacro:include filename="$(find annin_ar4_description)/urdf/ar_gripper.ros2_control.xacro"/>
-    <xacro:ar_gripper parent="ee_link" />
+    <xacro:ar_gripper parent="$(arg tf_prefix)ee_link" />
     <xacro:ar_gripper_ros2_control
       name="ar_servo_gripper"

File: annin_ar4_moveit_config/srdf/ar.srdf.xacro (robot description, xacro)
@@ -2,9 +2,10 @@
 <robot xmlns:xacro="http://wiki.ros.org/xacro" name="$(arg name)">
   <xacro:arg name="include_gripper" default="true"/>
+  <xacro:arg name="prefix" default="" />
   <xacro:include filename="$(find annin_ar4_moveit_config)/srdf/ar_macro.srdf.xacro"/>
-  <xacro:ar_srdf />
+  <xacro:ar_srdf prefix="$(arg prefix)"/>
   <xacro:if value="$(arg include_gripper)">
     <xacro:include filename="$(find annin_ar4_moveit_config)/srdf/ar_gripper_macro.srdf.xacro"/>
-    <xacro:ar_gripper_srdf />
+    <xacro:ar_gripper_srdf prefix="$(arg prefix)"/>
   </xacro:if>
 </robot>

File: annin_ar4_moveit_config/urdf/fake_ar.urdf.xacro (robot description, xacro)
@@ -5,6 +5,8 @@
   <xacro:include filename="$(find annin_ar4_description)/urdf/ar.ros2_control.xacro"/>
   <xacro:include filename="$(find annin_ar4_description)/urdf/ar_gripper.ros2_control.xacro"/>
+  <xacro:arg name="tf_prefix" default="" />
   <link name="world" />
   <xacro:ar_robot
+    tf_prefix="$(arg tf_prefix)"
     parent="world"
     robot_parameters_file="$(find annin_ar4_description)/config/$(arg ar_model).yaml"
@@ -12,5 +14,5 @@
     <origin xyz="0 0 0" rpy="0 0 0" />
   </xacro:ar_robot>
-  <xacro:ar_gripper parent="ee_link" />
+  <xacro:ar_gripper parent="$(arg tf_prefix)ee_link" />
   <xacro:ar_ros2_control
     ar_model="$(arg ar_model)"
@@ -21,4 +23,5 @@
     joint_offset_parameters_file="$(find annin_ar4_driver)/config/joint_offsets/$(arg ar_model).yaml"
     driver_parameters_file="$(find annin_ar4_driver)/config/driver.yaml"
+    tf_prefix="$(arg tf_prefix)"
   />
   <xacro:ar_gripper_ros2_control

Commit message: adding option to prepend gripper links with tf_prefix

File: annin_ar4_description/urdf/ar.urdf.xacro (robot description, xacro)
@@ -14,5 +14,8 @@
   <xacro:if value="$(arg include_gripper)">
     <xacro:include filename="$(find annin_ar4_description)/urdf/ar_gripper_macro.xacro"/>
-    <xacro:ar_gripper parent="$(arg tf_prefix)ee_link" />
+    <xacro:ar_gripper
+      tf_prefix="$(arg tf_prefix)"
+      parent="$(arg tf_prefix)ee_link"
+    />
   </xacro:if>
 </robot>

File: annin_ar4_description/urdf/ar_gazebo.urdf.xacro (robot description, xacro)
@@ -15,5 +15,8 @@
     <origin xyz="0 0 0" rpy="0 0 0" />
   </xacro:ar_robot>
-  <xacro:ar_gripper parent="$(arg tf_prefix)ee_link" />
+  <xacro:ar_gripper
+    tf_prefix="$(arg tf_prefix)"
+    parent="$(arg tf_prefix)ee_link"
+  />
   <xacro:ar_ros2_control
     ar_model="$(arg ar_model)"
@@ -30,4 +33,5 @@
     plugin_name="ign_ros2_control/IgnitionSystem"
     serial_port="None"
+    tf_prefix="$(arg tf_prefix)"
   />
   <gazebo reference="world" />

File: annin_ar4_description/urdf/ar_gripper.ros2_control.xacro (robot description, xacro)
@@ -5,4 +5,5 @@
     plugin_name
     serial_port
+    tf_prefix
   ">
     <ros2_control name="${name}" type="system">
@@ -10,6 +11,7 @@
         <plugin>${plugin_name}</plugin>
         <param name="serial_port">${serial_port}</param>
+        <param name="tf_prefix">${tf_prefix}</param>
       </hardware>
-      <joint name="gripper_jaw1_joint">
+      <joint name="${tf_prefix}gripper_jaw1_joint">
         <command_interface name="position" />
         <state_interface name="position">
@@ -20,6 +22,6 @@
         </state_interface>
       </joint>
-      <joint name="gripper_jaw2_joint">
-        <param name="mimic">gripper_jaw1_joint</param>
+      <joint name="${tf_prefix}gripper_jaw2_joint">
+        <param name="mimic">${tf_prefix}gripper_jaw1_joint</param>
         <param name="multiplier">1</param>
         <state_interface name="position">

File: annin_ar4_description/urdf/ar_gripper_macro.xacro (robot description, xacro)
@@ -1,11 +1,14 @@
 <?xml version="1.0" encoding="utf-8"?>
 <robot xmlns:xacro="http://wiki.ros.org/xacro">
-  <xacro:macro name="ar_gripper" params="parent">
-    <joint name="gripper_base_joint" type="fixed">
+  <xacro:macro name="ar_gripper" params="
+    tf_prefix
+    parent
+  ">
+    <joint name="${tf_prefix}gripper_base_joint" type="fixed">
       <origin xyz="0.0 0.0 0.0" rpy="-1.5708 0.0 0.0"/>
       <parent link="${parent}"/>
-      <child link="gripper_base_link"/>
+      <child link="${tf_prefix}gripper_base_link"/>
     </joint>
-    <link name="gripper_base_link">
+    <link name="${tf_prefix}gripper_base_link">
       <visual>
         <geometry>
@@ -27,5 +30,5 @@
       </inertial>
     </link>
-    <link name="gripper_jaw1_link">
+    <link name="${tf_prefix}gripper_jaw1_link">
       <visual>
         <geometry>
@@ -47,5 +50,5 @@
       </inertial>
     </link>
-    <link name="gripper_jaw2_link">
+    <link name="${tf_prefix}gripper_jaw2_link">
       <visual>
         <geometry>
@@ -67,24 +70,24 @@
       </inertial>
     </link>
-    <joint name="gripper_jaw1_joint" type="prismatic">
+    <joint name="${tf_prefix}gripper_jaw1_joint" type="prismatic">
       <origin xyz="0.0 -0.036 0" rpy="0.0 0.0 0.0"/>
-      <parent link="gripper_base_link"/>
-      <child link="gripper_jaw1_link"/>
+      <parent link="${tf_prefix}gripper_base_link"/>
+      <child link="${tf_prefix}gripper_jaw1_link"/>
       <axis xyz="1 0 0"/>
       <limit lower="-0.014" upper="0" effort="1000" velocity="1.0"/>
     </joint>
-    <joint name="gripper_jaw2_joint" type="prismatic">
+    <joint name="${tf_prefix}gripper_jaw2_joint" type="prismatic">
       <origin xyz="0.0 -0.036 0" rpy="0.0 ${-pi} 0.0"/>
-      <parent link="gripper_base_link"/>
-      <child link="gripper_jaw2_link"/>
+      <parent link="${tf_prefix}gripper_base_link"/>
+      <child link="${tf_prefix}gripper_jaw2_link"/>
       <axis xyz="1 0 0"/>
       <limit lower="-0.014" upper="0" effort="1000" velocity="1.0"/>
-      <mimic joint="gripper_jaw1_joint" multiplier="1" offset="0"/>
+      <mimic joint="${tf_prefix}gripper_jaw1_joint" multiplier="1" offset="0"/>
     </joint>
     <!-- Fix for https://github.com/ros-controls/gz_ros2_control/issues/96 when running in sim -->
-    <link name="dummy_mimic_fix"/>
-    <joint name="gripper_jaw2_joint_mimic" type="fixed">
-      <parent link="gripper_base_link" />
-      <child link="dummy_mimic_fix" />
+    <link name="${tf_prefix}dummy_mimic_fix"/>
+    <joint name="${tf_prefix}gripper_jaw2_joint_mimic" type="fixed">
+      <parent link="${tf_prefix}gripper_base_link" />
+      <child link="${tf_prefix}dummy_mimic_fix" />
     </joint>
   </xacro:macro>

File: annin_ar4_driver/urdf/ar.urdf.xacro (robot description, xacro)
@@ -29,9 +29,13 @@
     <xacro:include filename="$(find annin_ar4_description)/urdf/ar_gripper_macro.xacro"/>
     <xacro:include filename="$(find annin_ar4_description)/urdf/ar_gripper.ros2_control.xacro"/>
-    <xacro:ar_gripper parent="$(arg tf_prefix)ee_link" />
+    <xacro:ar_gripper
+      tf_prefix="$(arg tf_prefix)"
+      parent="$(arg tf_prefix)ee_link"
+    />
     <xacro:ar_gripper_ros2_control
       name="ar_servo_gripper"
       plugin_name="annin_ar4_driver/ARServoGripperHWInterface"
       serial_port="$(arg arduino_serial_port)"
+      tf_prefix="$(arg tf_prefix)"
     />
   </xacro:if>

File: annin_ar4_moveit_config/srdf/ar_gripper_macro.srdf.xacro (robot description, xacro)
@@ -7,21 +7,21 @@
   <xacro:macro name="ar_gripper_srdf" params="prefix">
     <group name="ar_gripper">
-      <link name="gripper_base_link" />
-      <link name="gripper_jaw1_link" />
-      <link name="gripper_jaw2_link" />
-      <joint name="gripper_jaw1_joint" />
-      <passive_joint name="gripper_jaw2_joint" />
+      <link name="${prefix}gripper_base_link" />
+      <link name="${prefix}gripper_jaw1_link" />
+      <link name="${prefix}gripper_jaw2_link" />
+      <joint name="${prefix}gripper_jaw1_joint" />
+      <passive_joint name="${prefix}gripper_jaw2_joint" />
     </group>
     <group_state name="open" group="ar_gripper">
-      <joint name="gripper_jaw1_joint" value="-0.012" />
+      <joint name="${prefix}gripper_jaw1_joint" value="-0.012" />
     </group_state>
     <group_state name="closed" group="ar_gripper">
-      <joint name="gripper_jaw1_joint" value="-0.001" />
+      <joint name="${prefix}gripper_jaw1_joint" value="-0.001" />
     </group_state>
-    <disable_collisions link1="gripper_base_link" link2="gripper_jaw1_link" reason="Adjacent" />
-    <disable_collisions link1="gripper_base_link" link2="gripper_jaw2_link" reason="Adjacent" />
-    <disable_collisions link1="gripper_jaw1_link" link2="gripper_jaw2_link" reason="Default" />
-    <disable_collisions link1="${prefix}link_6" link2="gripper_base_link" reason="Adjacent" />
-    <disable_collisions link1="${prefix}link_5" link2="gripper_base_link" reason="Adjacent" />
+    <disable_collisions link1="${prefix}gripper_base_link" link2="${prefix}gripper_jaw1_link" reason="Adjacent" />
+    <disable_collisions link1="${prefix}gripper_base_link" link2="${prefix}gripper_jaw2_link" reason="Adjacent" />
+    <disable_collisions link1="${prefix}gripper_jaw1_link" link2="${prefix}gripper_jaw2_link" reason="Default" />
+    <disable_collisions link1="${prefix}link_6" link2="${prefix}gripper_base_link" reason="Adjacent" />
+    <disable_collisions link1="${prefix}link_5" link2="${prefix}gripper_base_link" reason="Adjacent" />
   </xacro:macro>
 </robot>

File: annin_ar4_moveit_config/urdf/fake_ar.urdf.xacro (robot description, xacro)
@@ -14,5 +14,8 @@
     <origin xyz="0 0 0" rpy="0 0 0" />
   </xacro:ar_robot>
-  <xacro:ar_gripper parent="$(arg tf_prefix)ee_link" />
+  <xacro:ar_gripper
+    tf_prefix="$(arg tf_prefix)"
+    parent="$(arg tf_prefix)ee_link"
+  />
   <xacro:ar_ros2_control
     ar_model="$(arg ar_model)"
@@ -29,4 +32,5 @@
     plugin_name="mock_components/GenericSystem"
     serial_port="/dev/ttyUSB0"
+    tf_prefix="$(arg tf_prefix)"
   />
 </robot>
