Commit message: Adding tf_prefix to .urdf, .srdf and launch files to humble branch (#37)
* Adding tf_prefix to .urdf, .srdf and launch files

* adding option to prepend gripper links with tf_prefix

* dynamic driver controllers.yaml, updates to demo.launch & driver.launch for using it. added config folder for gazebo with separate controllers.yaml and updated gazebo.launch

* remove commented code, light clean up

---------

Co-authored-by: Yifei Cheng <ycheng517@gmail.com>

File: annin_ar4_description/urdf/ar.urdf.xacro (robot description, xacro)
@@ -1,8 +1,10 @@
 <?xml version="1.0"?>
 <robot xmlns:xacro="http://wiki.ros.org/xacro" name="$(arg ar_model)">
+  <xacro:arg name="tf_prefix" default="" />
   <xacro:arg name="include_gripper" default="true"/>
   <xacro:include filename="$(find annin_ar4_description)/urdf/ar_macro.xacro"/>
   <link name="world" />
   <xacro:ar_robot
+    tf_prefix="$(arg tf_prefix)"
     parent="world"
     robot_parameters_file="$(find annin_ar4_description)/config/$(arg ar_model).yaml"
@@ -12,5 +14,8 @@
   <xacro:if value="$(arg include_gripper)">
     <xacro:include filename="$(find annin_ar4_description)/urdf/ar_gripper_macro.xacro"/>
-    <xacro:ar_gripper parent="ee_link" />
+    <xacro:ar_gripper
+      tf_prefix="$(arg tf_prefix)"
+      parent="$(arg tf_prefix)ee_link"
+    />
   </xacro:if>
 </robot>

File: annin_ar4_description/urdf/ar_gazebo.urdf.xacro (robot description, xacro)
@@ -6,6 +6,8 @@
   <xacro:include filename="$(find annin_ar4_description)/urdf/ar_gripper.ros2_control.xacro" />
   <xacro:arg name="simulation_controllers" default="" />
+  <xacro:arg name="tf_prefix" default="" />
   <link name="world" />
   <xacro:ar_robot
+    tf_prefix="$(arg tf_prefix)"
     parent="world"
     robot_parameters_file="$(find annin_ar4_description)/config/$(arg ar_model).yaml"
@@ -13,5 +15,8 @@
     <origin xyz="0 0 0" rpy="0 0 0" />
   </xacro:ar_robot>
-  <xacro:ar_gripper parent="ee_link" />
+  <xacro:ar_gripper
+    tf_prefix="$(arg tf_prefix)"
+    parent="$(arg tf_prefix)ee_link"
+  />
   <xacro:ar_ros2_control
     ar_model="$(arg ar_model)"
@@ -22,4 +27,5 @@
     joint_offset_parameters_file="$(find annin_ar4_driver)/config/joint_offsets/$(arg ar_model).yaml"
     driver_parameters_file="$(find annin_ar4_driver)/config/driver.yaml"
+    tf_prefix="$(arg tf_prefix)"
   />
   <xacro:ar_gripper_ros2_control
@@ -27,4 +33,5 @@
     plugin_name="ign_ros2_control/IgnitionSystem"
     serial_port="None"
+    tf_prefix="$(arg tf_prefix)"
   />
   <gazebo reference="world" />

File: annin_ar4_driver/urdf/ar.urdf.xacro (robot description, xacro)
@@ -4,4 +4,5 @@
   <xacro:arg name="arduino_serial_port" default="/dev/ttyUSB0"/>
   <xacro:arg name="calibrate" default="True"/>
+  <xacro:arg name="tf_prefix" default="" />
   <xacro:arg name="include_gripper" default="true"/>
   <xacro:include filename="$(find annin_ar4_description)/urdf/ar_macro.xacro"/>
@@ -9,4 +10,5 @@
   <link name="world" />
   <xacro:ar_robot
+    tf_prefix="$(arg tf_prefix)"
     parent="world"
     robot_parameters_file="$(find annin_ar4_description)/config/$(arg ar_model).yaml"
@@ -22,13 +24,18 @@
     joint_offset_parameters_file="$(find annin_ar4_driver)/config/joint_offsets/$(arg ar_model).yaml"
     driver_parameters_file="$(find annin_ar4_driver)/config/driver.yaml"
+    tf_prefix="$(arg tf_prefix)"
   />
   <xacro:if value="$(arg include_gripper)">
     <xacro:include filename="$(find annin_ar4_description)/urdf/ar_gripper_macro.xacro"/>
     <xacro:include filename="$(find annin_ar4_description)/urdf/ar_gripper.ros2_control.xacro"/>
-    <xacro:ar_gripper parent="ee_link" />
+    <xacro:ar_gripper
+      tf_prefix="$(arg tf_prefix)"
+      parent="$(arg tf_prefix)ee_link"
+    />
     <xacro:ar_gripper_ros2_control
       name="ar_servo_gripper"
       plugin_name="annin_ar4_driver/ARServoGripperHWInterface"
       serial_port="$(arg arduino_serial_port)"
+      tf_prefix="$(arg tf_prefix)"
     />
   </xacro:if>

File: annin_ar4_moveit_config/srdf/ar_gripper_macro.srdf.xacro (robot description, xacro)
@@ -5,23 +5,23 @@
 -->
 <robot xmlns:xacro="http://wiki.ros.org/xacro">
-  <xacro:macro name="ar_gripper_srdf">
+  <xacro:macro name="ar_gripper_srdf" params="prefix">
     <group name="ar_gripper">
-      <link name="gripper_base_link" />
-      <link name="gripper_jaw1_link" />
-      <link name="gripper_jaw2_link" />
-      <joint name="gripper_jaw1_joint" />
-      <passive_joint name="gripper_jaw2_joint" />
+      <link name="${prefix}gripper_base_link" />
+      <link name="${prefix}gripper_jaw1_link" />
+      <link name="${prefix}gripper_jaw2_link" />
+      <joint name="${prefix}gripper_jaw1_joint" />
+      <passive_joint name="${prefix}gripper_jaw2_joint" />
     </group>
     <group_state name="open" group="ar_gripper">
-      <joint name="gripper_jaw1_joint" value="-0.012" />
+      <joint name="${prefix}gripper_jaw1_joint" value="-0.012" />
     </group_state>
     <group_state name="closed" group="ar_gripper">
-      <joint name="gripper_jaw1_joint" value="-0.001" />
+      <joint name="${prefix}gripper_jaw1_joint" value="-0.001" />
     </group_state>
-    <disable_collisions link1="gripper_base_link" link2="gripper_jaw1_link" reason="Adjacent" />
-    <disable_collisions link1="gripper_base_link" link2="gripper_jaw2_link" reason="Adjacent" />
-    <disable_collisions link1="gripper_jaw1_link" link2="gripper_jaw2_link" reason="Default" />
-    <disable_collisions link1="link_6" link2="gripper_base_link" reason="Adjacent" />
-    <disable_collisions link1="link_5" link2="gripper_base_link" reason="Adjacent" />
+    <disable_collisions link1="${prefix}gripper_base_link" link2="${prefix}gripper_jaw1_link" reason="Adjacent" />
+    <disable_collisions link1="${prefix}gripper_base_link" link2="${prefix}gripper_jaw2_link" reason="Adjacent" />
+    <disable_collisions link1="${prefix}gripper_jaw1_link" link2="${prefix}gripper_jaw2_link" reason="Default" />
+    <disable_collisions link1="${prefix}link_6" link2="${prefix}gripper_base_link" reason="Adjacent" />
+    <disable_collisions link1="${prefix}link_5" link2="${prefix}gripper_base_link" reason="Adjacent" />
   </xacro:macro>
 </robot>

File: annin_ar4_moveit_config/urdf/fake_ar.urdf.xacro (robot description, xacro)
@@ -5,6 +5,8 @@
   <xacro:include filename="$(find annin_ar4_description)/urdf/ar.ros2_control.xacro"/>
   <xacro:include filename="$(find annin_ar4_description)/urdf/ar_gripper.ros2_control.xacro"/>
+  <xacro:arg name="tf_prefix" default="" />
   <link name="world" />
   <xacro:ar_robot
+    tf_prefix="$(arg tf_prefix)"
     parent="world"
     robot_parameters_file="$(find annin_ar4_description)/config/$(arg ar_model).yaml"
@@ -12,5 +14,8 @@
     <origin xyz="0 0 0" rpy="0 0 0" />
   </xacro:ar_robot>
-  <xacro:ar_gripper parent="ee_link" />
+  <xacro:ar_gripper
+    tf_prefix="$(arg tf_prefix)"
+    parent="$(arg tf_prefix)ee_link"
+  />
   <xacro:ar_ros2_control
     ar_model="$(arg ar_model)"
@@ -21,4 +26,5 @@
     joint_offset_parameters_file="$(find annin_ar4_driver)/config/joint_offsets/$(arg ar_model).yaml"
     driver_parameters_file="$(find annin_ar4_driver)/config/driver.yaml"
+    tf_prefix="$(arg tf_prefix)"
   />
   <xacro:ar_gripper_ros2_control
@@ -26,4 +32,5 @@
     plugin_name="mock_components/GenericSystem"
     serial_port="/dev/ttyUSB0"
+    tf_prefix="$(arg tf_prefix)"
   />
 </robot>
