Commit message: make gripper open position positive and not negative

File: annin_ar4_description/urdf/ar_gripper_macro.xacro (robot description, xacro)
@@ -74,6 +74,6 @@
       <parent link="${tf_prefix}gripper_base_link"/>
       <child link="${tf_prefix}gripper_jaw1_link"/>
-      <axis xyz="1 0 0"/>
-      <limit lower="-0.014" upper="0" effort="-1" velocity="1.0"/>
+      <axis xyz="-1 0 0"/>
+      <limit lower="0" upper="0.014" effort="-1" velocity="1.0"/>
     </joint>
     <joint name="${tf_prefix}gripper_jaw2_joint" type="prismatic">
@@ -81,6 +81,6 @@
       <parent link="${tf_prefix}gripper_base_link"/>
       <child link="${tf_prefix}gripper_jaw2_link"/>
-      <axis xyz="1 0 0"/>
-      <limit lower="-0.014" upper="0" effort="1000" velocity="1.0"/>
+      <axis xyz="-1 0 0"/>
+      <limit lower="0" upper="0.014" effort="1000" velocity="1.0"/>
       <mimic joint="${tf_prefix}gripper_jaw1_joint" multiplier="1" offset="0"/>
     </joint>

File: annin_ar4_moveit_config/srdf/ar_gripper_macro.srdf.xacro (robot description, xacro)
@@ -14,8 +14,8 @@
     </group>
     <group_state name="open" group="ar_gripper">
-      <joint name="${tf_prefix}gripper_jaw1_joint" value="-0.012" />
+      <joint name="${tf_prefix}gripper_jaw1_joint" value="0.012" />
     </group_state>
     <group_state name="closed" group="ar_gripper">
-      <joint name="${tf_prefix}gripper_jaw1_joint" value="-0.001" />
+      <joint name="${tf_prefix}gripper_jaw1_joint" value="0.001" />
     </group_state>
     <disable_collisions link1="${tf_prefix}gripper_base_link" link2="${tf_prefix}gripper_jaw1_link" reason="Adjacent" />

Commit message: make gripper open position positive and not negative (#48)

File: annin_ar4_description/urdf/ar_gripper_macro.xacro (robot description, xacro)
@@ -74,6 +74,6 @@
       <parent link="${tf_prefix}gripper_base_link"/>
       <child link="${tf_prefix}gripper_jaw1_link"/>
-      <axis xyz="1 0 0"/>
-      <limit lower="-0.014" upper="0" effort="1000" velocity="1.0"/>
+      <axis xyz="-1 0 0"/>
+      <limit lower="0" upper="0.014" effort="1000" velocity="1.0"/>
     </joint>
     <joint name="${tf_prefix}gripper_jaw2_joint" type="prismatic">
@@ -81,6 +81,6 @@
       <parent link="${tf_prefix}gripper_base_link"/>
       <child link="${tf_prefix}gripper_jaw2_link"/>
-      <axis xyz="1 0 0"/>
-      <limit lower="-0.014" upper="0" effort="1000" velocity="1.0"/>
+      <axis xyz="-1 0 0"/>
+      <limit lower="0" upper="0.014" effort="1000" velocity="1.0"/>
       <mimic joint="${tf_prefix}gripper_jaw1_joint" multiplier="1" offset="0"/>
     </joint>

Commit message: normalized gripper position

File: annin_ar4_description/urdf/ar_gripper_macro.xacro (robot description, xacro)
@@ -75,5 +75,5 @@
       <child link="${tf_prefix}gripper_jaw1_link"/>
       <axis xyz="-1 0 0"/>
-      <limit lower="0" upper="0.014" effort="-1" velocity="1.0"/>
+      <limit lower="0" upper="1" effort="-1" velocity="1.0"/>
     </joint>
     <joint name="${tf_prefix}gripper_jaw2_joint" type="prismatic">
@@ -82,5 +82,5 @@
       <child link="${tf_prefix}gripper_jaw2_link"/>
       <axis xyz="-1 0 0"/>
-      <limit lower="0" upper="0.014" effort="1000" velocity="1.0"/>
+      <limit lower="0" upper="1" effort="1000" velocity="1.0"/>
       <mimic joint="${tf_prefix}gripper_jaw1_joint" multiplier="1" offset="0"/>
     </joint>

File: annin_ar4_moveit_config/srdf/ar_gripper_macro.srdf.xacro (robot description, xacro)
@@ -14,8 +14,8 @@
     </group>
     <group_state name="open" group="ar_gripper">
-      <joint name="${tf_prefix}gripper_jaw1_joint" value="0.012" />
+      <joint name="${tf_prefix}gripper_jaw1_joint" value="1" />
     </group_state>
     <group_state name="closed" group="ar_gripper">
-      <joint name="${tf_prefix}gripper_jaw1_joint" value="0.001" />
+      <joint name="${tf_prefix}gripper_jaw1_joint" value="0" />
     </group_state>
     <disable_collisions link1="${tf_prefix}gripper_base_link" link2="${tf_prefix}gripper_jaw1_link" reason="Adjacent" />

Commit message: cant normalize, make open/close same scale as AR gripper

File: annin_ar4_description/urdf/ar_gripper_macro.xacro (robot description, xacro)
@@ -75,5 +75,5 @@
       <child link="${tf_prefix}gripper_jaw1_link"/>
       <axis xyz="-1 0 0"/>
-      <limit lower="0" upper="1" effort="-1" velocity="1.0"/>
+      <limit lower="0" upper="0.014" effort="-1" velocity="1.0"/>
     </joint>
     <joint name="${tf_prefix}gripper_jaw2_joint" type="prismatic">
@@ -82,5 +82,5 @@
       <child link="${tf_prefix}gripper_jaw2_link"/>
       <axis xyz="-1 0 0"/>
-      <limit lower="0" upper="1" effort="1000" velocity="1.0"/>
+      <limit lower="0" upper="0.014" effort="1000" velocity="1.0"/>
       <mimic joint="${tf_prefix}gripper_jaw1_joint" multiplier="1" offset="0"/>
     </joint>

File: annin_ar4_moveit_config/srdf/ar_gripper_macro.srdf.xacro (robot description, xacro)
@@ -14,8 +14,8 @@
     </group>
     <group_state name="open" group="ar_gripper">
-      <joint name="${tf_prefix}gripper_jaw1_joint" value="1" />
+      <joint name="${tf_prefix}gripper_jaw1_joint" value="0.014" />
     </group_state>
     <group_state name="closed" group="ar_gripper">
-      <joint name="${tf_prefix}gripper_jaw1_joint" value="0" />
+      <joint name="${tf_prefix}gripper_jaw1_joint" value="0.000" />
     </group_state>
     <disable_collisions link1="${tf_prefix}gripper_base_link" link2="${tf_prefix}gripper_jaw1_link" reason="Adjacent" />
