Commit message: branch that supports ROS 2 humble

File: annin_ar4_description/urdf/ar_gazebo.urdf.xacro (robot description, xacro)
@@ -16,5 +16,5 @@
   <xacro:ar_ros2_control
     ar_model="$(arg ar_model)"
-    plugin_name="gz_ros2_control/GazeboSimSystem"
+    plugin_name="ign_ros2_control/IgnitionSystem"
     serial_port="None"
     calibrate="False"
@@ -25,10 +25,10 @@
   <xacro:ar_gripper_ros2_control
     name="ARGripperGazeboSystem"
-    plugin_name="gz_ros2_control/GazeboSimSystem"
+    plugin_name="ign_ros2_control/IgnitionSystem"
     serial_port="None"
   />
   <gazebo reference="world" />
   <gazebo>
-    <plugin filename="libgz_ros2_control-system" name="gz_ros2_control::GazeboSimROS2ControlPlugin">
+    <plugin filename="libign_ros2_control-system" name="ign_ros2_control::IgnitionROS2ControlPlugin">
       <parameters>$(arg simulation_controllers)</parameters>
     </plugin>

File: annin_ar4_description/urdf/ar_gripper_macro.xacro (robot description, xacro)
@@ -72,5 +72,5 @@
       <child link="gripper_jaw1_link"/>
       <axis xyz="1 0 0"/>
-      <limit lower="-0.014" upper="0" effort="-1" velocity="1.0"/>
+      <limit lower="-0.014" upper="0" effort="1000" velocity="1.0"/>
     </joint>
     <joint name="gripper_jaw2_joint" type="prismatic">
@@ -79,6 +79,12 @@
       <child link="gripper_jaw2_link"/>
       <axis xyz="1 0 0"/>
-      <limit lower="-0.014" upper="0" effort="-1" velocity="1.0"/>
+      <limit lower="-0.014" upper="0" effort="1000" velocity="1.0"/>
       <mimic joint="gripper_jaw1_joint" multiplier="1" offset="0"/>
+    </joint>
+    <!-- Fix for https://github.com/ros-controls/gz_ros2_control/issues/96 when running in sim -->
+    <link name="dummy_mimic_fix"/>
+    <joint name="gripper_jaw2_joint_mimic" type="fixed">
+      <parent link="gripper_base_link" />
+      <child link="dummy_mimic_fix" />
     </joint>
   </xacro:macro>

File: annin_ar4_description/urdf/ar_macro.xacro (robot description, xacro)
@@ -64,5 +64,5 @@
         lower="${robot_parameters['j1_limit_min']}"
         upper="${robot_parameters['j1_limit_max']}"
-        effort="-1"
+        effort="1000"
         velocity="1.0472"
       />
@@ -98,5 +98,5 @@
         lower="${robot_parameters['j2_limit_min']}"
         upper="${robot_parameters['j2_limit_max']}"
-        effort="-1"
+        effort="1000"
         velocity="1.0472"
       />
@@ -132,5 +132,5 @@
         lower="${robot_parameters['j3_limit_min']}"
         upper="${robot_parameters['j3_limit_max']}"
-        effort="-1"
+        effort="1000"
         velocity="1.0472"
       />
@@ -166,5 +166,5 @@
         lower="${robot_parameters['j4_limit_min']}"
         upper="${robot_parameters['j4_limit_max']}"
-        effort="-1"
+        effort="1000"
         velocity="1.0472"
       />
@@ -200,5 +200,5 @@
         lower="${robot_parameters['j5_limit_min']}"
         upper="${robot_parameters['j5_limit_max']}"
-        effort="-1"
+        effort="1000"
         velocity="1.0472"
       />
@@ -234,5 +234,5 @@
         lower="${robot_parameters['j6_limit_min']}"
         upper="${robot_parameters['j6_limit_max']}"
-        effort="-1"
+        effort="1000"
         velocity="1.0472"
       />

Commit message: Adding tf_prefix to .urdf, .srdf and launch files to humble branch (#37)
* Adding tf_prefix to .urdf, .srdf and launch files

* adding option to prepend gripper links with tf_prefix

* dynamic driver controllers.yaml, updates to demo.launch & driver.launch for using it. added config folder for gazebo with separate controllers.yaml and updated gazebo.launch

* remove commented code, light clean up

---------

Co-authored-by: Yifei Cheng <ycheng517@gmail.com>

File: annin_ar4_description/urdf/ar_gazebo.urdf.xacro (robot description, xacro)
@@ -6,6 +6,8 @@
   <xacro:include filename="$(find annin_ar4_description)/urdf/ar_gripper.ros2_control.xacro" />
   <xacro:arg name="simulation_controllers" default="" />
+  <xacro:arg name="tf_prefix" default="" />
   <link name="world" />
   <xacro:ar_robot
+    tf_prefix="$(arg tf_prefix)"
     parent="world"
     robot_parameters_file="$(find annin_ar4_description)/config/$(arg ar_model).yaml"
@@ -13,5 +15,8 @@
     <origin xyz="0 0 0" rpy="0 0 0" />
   </xacro:ar_robot>
-  <xacro:ar_gripper parent="ee_link" />
+  <xacro:ar_gripper
+    tf_prefix="$(arg tf_prefix)"
+    parent="$(arg tf_prefix)ee_link"
+  />
   <xacro:ar_ros2_control
     ar_model="$(arg ar_model)"
@@ -22,4 +27,5 @@
     joint_offset_parameters_file="$(find annin_ar4_driver)/config/joint_offsets/$(arg ar_model).yaml"
     driver_parameters_file="$(find annin_ar4_driver)/config/driver.yaml"
+    tf_prefix="$(arg tf_prefix)"
   />
   <xacro:ar_gripper_ros2_control
@@ -27,4 +33,5 @@
     plugin_name="gz_ros2_control/GazeboSimSystem"
     serial_port="None"
+    tf_prefix="$(arg tf_prefix)"
   />
   <gazebo reference="world" />

File: annin_ar4_description/urdf/ar_gripper_macro.xacro (robot description, xacro)
@@ -1,11 +1,14 @@
 <?xml version="1.0" encoding="utf-8"?>
 <robot xmlns:xacro="http://wiki.ros.org/xacro">
-  <xacro:macro name="ar_gripper" params="parent">
-    <joint name="gripper_base_joint" type="fixed">
+  <xacro:macro name="ar_gripper" params="
+    tf_prefix
+    parent
+  ">
+    <joint name="${tf_prefix}gripper_base_joint" type="fixed">
       <origin xyz="0.0 0.0 0.0" rpy="-1.5708 0.0 0.0"/>
       <parent link="${parent}"/>
-      <child link="gripper_base_link"/>
+      <child link="${tf_prefix}gripper_base_link"/>
     </joint>
-    <link name="gripper_base_link">
+    <link name="${tf_prefix}gripper_base_link">
       <visual>
         <geometry>
@@ -27,5 +30,5 @@
       </inertial>
     </link>
-    <link name="gripper_jaw1_link">
+    <link name="${tf_prefix}gripper_jaw1_link">
       <visual>
         <geometry>
@@ -47,5 +50,5 @@
       </inertial>
     </link>
-    <link name="gripper_jaw2_link">
+    <link name="${tf_prefix}gripper_jaw2_link">
       <visual>
         <geometry>
@@ -67,18 +70,18 @@
       </inertial>
     </link>
-    <joint name="gripper_jaw1_joint" type="prismatic">
+    <joint name="${tf_prefix}gripper_jaw1_joint" type="prismatic">
       <origin xyz="0.0 -0.036 0" rpy="0.0 0.0 0.0"/>
-      <parent link="gripper_base_link"/>
-      <child link="gripper_jaw1_link"/>
+      <parent link="${tf_prefix}gripper_base_link"/>
+      <child link="${tf_prefix}gripper_jaw1_link"/>
       <axis xyz="1 0 0"/>
       <limit lower="-0.014" upper="0" effort="-1" velocity="1.0"/>
     </joint>
-    <joint name="gripper_jaw2_joint" type="prismatic">
+    <joint name="${tf_prefix}gripper_jaw2_joint" type="prismatic">
       <origin xyz="0.0 -0.036 0" rpy="0.0 ${-pi} 0.0"/>
-      <parent link="gripper_base_link"/>
-      <child link="gripper_jaw2_link"/>
+      <parent link="${tf_prefix}gripper_base_link"/>
+      <child link="${tf_prefix}gripper_jaw2_link"/>
       <axis xyz="1 0 0"/>
-      <limit lower="-0.014" upper="0" effort="-1" velocity="1.0"/>
-      <mimic joint="gripper_jaw1_joint" multiplier="1" offset="0"/>
+      <limit lower="-0.014" upper="0" effort="1000" velocity="1.0"/>
+      <mimic joint="${tf_prefix}gripper_jaw1_joint" multiplier="1" offset="0"/>
     </joint>
   </xacro:macro>

File: annin_ar4_description/urdf/ar_macro.xacro (robot description, xacro)
@@ -2,4 +2,5 @@
 <robot xmlns:xacro="http://wiki.ros.org/xacro">
   <xacro:macro name="ar_robot" params="
+    tf_prefix
     parent
     *origin
@@ -7,10 +8,10 @@
   ">
     <xacro:property name="robot_parameters" value="${xacro.load_yaml(robot_parameters_file)}"/>
-    <joint name="base_joint" type="fixed">
+    <joint name="${tf_prefix}base_joint" type="fixed">
       <xacro:insert_block name="origin" />
       <parent link="${parent}"/>
-      <child link="base_link" />
-    </joint>
-    <link name="base_link">
+      <child link="${tf_prefix}base_link" />
+    </joint>
+    <link name="${tf_prefix}base_link">
       <inertial>
         <origin rpy="0 0 0" xyz="-4.6941E-06 0.054174 0.038824"/>
@@ -34,5 +35,5 @@
       </collision>
     </link>
-    <link name="link_1">
+    <link name="${tf_prefix}link_1">
       <inertial>
         <origin rpy="0 0 0" xyz="-0.022706 0.04294 -0.12205"/>
@@ -56,8 +57,8 @@
       </collision>
     </link>
-    <joint name="joint_1" type="revolute">
+    <joint name="${tf_prefix}joint_1" type="revolute">
       <origin rpy="${pi} 0 0" xyz="0 0 0"/>
-      <parent link="base_link"/>
-      <child link="link_1"/>
+      <parent link="${tf_prefix}base_link"/>
+      <child link="${tf_prefix}link_1"/>
       <axis xyz="0 0 1"/>
       <limit
@@ -68,5 +69,5 @@
       />
     </joint>
-    <link name="link_2">
+    <link name="${tf_prefix}link_2">
       <inertial>
         <origin rpy="0 0 0" xyz="0.064818 -0.11189 -0.038671"/>
@@ -90,8 +91,8 @@
       </collision>
     </link>
-    <joint name="joint_2" type="revolute">
+    <joint name="${tf_prefix}joint_2" type="revolute">
       <origin rpy="1.5708 0 -1.5708" xyz="0 0.0642 -0.16977"/>
-      <parent link="link_1"/>
-      <child link="link_2"/>
+      <parent link="${tf_prefix}link_1"/>
+      <child link="${tf_prefix}link_2"/>
       <axis xyz="0 0 -1"/>
       <limit
@@ -102,5 +103,5 @@
       />
     </joint>
-    <link name="link_3">
+    <link name="${tf_prefix}link_3">
       <inertial>
         <origin rpy="0 0 0" xyz="-0.00029765 -0.023661 -0.0019125"/>
@@ -124,8 +125,8 @@
       </collision>
     </link>
-    <joint name="joint_3" type="revolute">
+    <joint name="${tf_prefix}joint_3" type="revolute">
       <origin rpy="0 0 3.1416" xyz="0 -0.305 0.007"/>
-      <parent link="link_2"/>
-      <child link="link_3"/>
+      <parent link="${tf_prefix}link_2"/>
+      <child link="${tf_prefix}link_3"/>
       <axis xyz="0 0 -1"/>
       <limit
@@ -136,5 +137,5 @@
       />
     </joint>
-    <link name="link_4">
+    <link name="${tf_prefix}link_4">
       <inertial>
         <origin rpy="0 0 0" xyz="-0.0016798 -0.00057319 -0.074404"/>
@@ -158,8 +159,8 @@
       </collision>
     </link>
-    <joint name="joint_4" type="revolute">
+    <joint name="${tf_prefix}joint_4" type="revolute">
       <origin rpy="1.5708 0 -1.5708" xyz="0 0 0.0"/>
-      <parent link="link_3"/>
-      <child link="link_4"/>
+      <parent link="${tf_prefix}link_3"/>
+      <child link="${tf_prefix}link_4"/>
       <axis xyz="0 0 -1"/>
       <limit
@@ -170,5 +171,5 @@
       />
     </joint>
-    <link name="link_5">
+    <link name="${tf_prefix}link_5">
       <inertial>
         <origin rpy="0 0 0" xyz="0.0015066 -1.3102E-05 -0.012585"/>
@@ -192,8 +193,8 @@
       </collision>
     </link>
-    <joint name="joint_5" type="revolute">
+    <joint name="${tf_prefix}joint_5" type="revolute">
       <origin rpy="${pi} 0 -1.5708" xyz="0 0 -0.22263"/>
-      <parent link="link_4"/>
-      <child link="link_5"/>
+      <parent link="${tf_prefix}link_4"/>
+      <child link="${tf_prefix}link_5"/>
       <axis xyz="1 0 0"/>
       <limit
@@ -204,5 +205,5 @@
       />
     </joint>
-    <link name="link_6">
+    <link name="${tf_prefix}link_6">
       <inertial>
         <origin rpy="0 0 0" xyz="2.9287E-10 -1.6472E-09 0.0091432"/>
@@ -226,8 +227,8 @@
       </collision>
     </link>
-    <joint name="joint_6" type="revolute">
+    <joint name="${tf_prefix}joint_6" type="revolute">
       <origin rpy="0 0 3.1416" xyz="0.000 0 ${robot_parameters['l6_length']}"/>
-      <parent link="link_5"/>
-      <child link="link_6"/>
+      <parent link="${tf_prefix}link_5"/>
+      <child link="${tf_prefix}link_6"/>
       <axis xyz="0 0 1"/>
       <limit
@@ -239,8 +240,8 @@
     </joint>
     <!-- center of the end effector mounting surface on link_6 -->
-    <link name="ee_link" />
-    <joint name="ee_joint" type="fixed">
-      <parent link="link_6" />
-      <child link="ee_link" />
+    <link name="${tf_prefix}ee_link" />
+    <joint name="${tf_prefix}ee_joint" type="fixed">
+      <parent link="${tf_prefix}link_6" />
+      <child link="${tf_prefix}ee_link" />
       <origin xyz="0 0 0.0" rpy="0 0 0" />
     </joint>

Commit message: fully support overcurrent option

File: annin_ar4_description/urdf/ar_gazebo.urdf.xacro (robot description, xacro)
@@ -34,4 +34,5 @@
     plugin_name="gz_ros2_control/GazeboSimSystem"
     serial_port="None"
+    driver_parameters_file="$(find annin_ar4_driver)/config/gripper_driver.yaml"
     tf_prefix="$(arg tf_prefix)"
   />

File: annin_ar4_description/urdf/ar_gripper.ros2_control.xacro (robot description, xacro)
@@ -5,10 +5,14 @@
     plugin_name
     serial_port
+    driver_parameters_file
     tf_prefix
   ">
+    <xacro:property name="driver_parameters"
+      value="${xacro.load_yaml(driver_parameters_file)}"/>
     <ros2_control name="${name}" type="system">
       <hardware>
         <plugin>${plugin_name}</plugin>
         <param name="serial_port">${serial_port}</param>
+        <param name="use_overcurrent_protection">${driver_parameters['use_overcurrent_protection']}</param>
         <param name="tf_prefix">${tf_prefix}</param>
       </hardware>

File: annin_ar4_driver/urdf/ar.urdf.xacro (robot description, xacro)
@@ -37,4 +37,5 @@
       plugin_name="annin_ar4_driver/ARServoGripperHWInterface"
       serial_port="$(arg arduino_serial_port)"
+      driver_parameters_file="$(find annin_ar4_driver)/config/gripper_driver.yaml"
       tf_prefix="$(arg tf_prefix)"
     />

File: annin_ar4_moveit_config/urdf/fake_ar.urdf.xacro (robot description, xacro)
@@ -32,4 +32,5 @@
     plugin_name="mock_components/GenericSystem"
     serial_port="/dev/ttyUSB0"
+    driver_parameters_file="$(find annin_ar4_driver)/config/gripper_driver.yaml"
     tf_prefix="$(arg tf_prefix)"
   />
