Commit message: Gripper Overcurrent Protection (#49)
* gripper current sensing

* normalized gripper position

* cant normalize, make open/close same scale as AR gripper

* finetuning

* move thermal protection to separate file

* rename thermal to over current

* fully support overcurrent option

* make min/max servo angle configurable

* use ar4 servo gripper defaults

* polish

* don't read current if overcurrent protection disabled

* clean up and tuning

* add docs, final polish

* final polish

* mention in main readme

* minor polish

File: annin_ar4_description/urdf/ar_gripper.ros2_control.xacro (robot description, xacro)
@@ -5,10 +5,16 @@
     plugin_name
     serial_port
+    driver_parameters_file
     tf_prefix
   ">
+    <xacro:property name="driver_parameters"
+      value="${xacro.load_yaml(driver_parameters_file)}"/>
     <ros2_control name="${name}" type="system">
       <hardware>
         <plugin>${plugin_name}</plugin>
         <param name="serial_port">${serial_port}</param>
+        <param name="use_overcurrent_protection">${driver_parameters['use_overcurrent_protection']}</param>
+        <param name="closed_servo_angle">${driver_parameters['closed_servo_angle']}</param>
+        <param name="open_servo_angle">${driver_parameters['open_servo_angle']}</param>
         <param name="tf_prefix">${tf_prefix}</param>
       </hardware>

File: annin_ar4_moveit_config/srdf/ar_gripper_macro.srdf.xacro (robot description, xacro)
@@ -14,8 +14,8 @@
     </group>
     <group_state name="open" group="ar_gripper">
-      <joint name="${tf_prefix}gripper_jaw1_joint" value="0.012" />
+      <joint name="${tf_prefix}gripper_jaw1_joint" value="0.014" />
     </group_state>
     <group_state name="closed" group="ar_gripper">
-      <joint name="${tf_prefix}gripper_jaw1_joint" value="0.001" />
+      <joint name="${tf_prefix}gripper_jaw1_joint" value="0.000" />
     </group_state>
     <disable_collisions link1="${tf_prefix}gripper_base_link" link2="${tf_prefix}gripper_jaw1_link" reason="Adjacent" />
