Commit message: rename prefix to tf_prefix

File: annin_ar4_moveit_config/srdf/ar.srdf.xacro (robot description, xacro)
@@ -2,10 +2,10 @@
 <robot xmlns:xacro="http://wiki.ros.org/xacro" name="$(arg name)">
   <xacro:arg name="include_gripper" default="true"/>
-  <xacro:arg name="prefix" default="" />
+  <xacro:arg name="tf_prefix" default="" />
   <xacro:include filename="$(find annin_ar4_moveit_config)/srdf/ar_macro.srdf.xacro"/>
-  <xacro:ar_srdf prefix="$(arg prefix)"/>
+  <xacro:ar_srdf tf_prefix="$(arg tf_prefix)"/>
   <xacro:if value="$(arg include_gripper)">
     <xacro:include filename="$(find annin_ar4_moveit_config)/srdf/ar_gripper_macro.srdf.xacro"/>
-    <xacro:ar_gripper_srdf prefix="$(arg prefix)"/>
+    <xacro:ar_gripper_srdf tf_prefix="$(arg tf_prefix)"/>
   </xacro:if>
 </robot>

File: annin_ar4_moveit_config/srdf/ar_gripper_macro.srdf.xacro (robot description, xacro)
@@ -5,23 +5,23 @@
 -->
 <robot xmlns:xacro="http://wiki.ros.org/xacro">
-  <xacro:macro name="ar_gripper_srdf" params="prefix">
+  <xacro:macro name="ar_gripper_srdf" params="tf_prefix">
     <group name="ar_gripper">
-      <link name="${prefix}gripper_base_link" />
-      <link name="${prefix}gripper_jaw1_link" />
-      <link name="${prefix}gripper_jaw2_link" />
-      <joint name="${prefix}gripper_jaw1_joint" />
-      <passive_joint name="${prefix}gripper_jaw2_joint" />
+      <link name="${tf_prefix}gripper_base_link" />
+      <link name="${tf_prefix}gripper_jaw1_link" />
+      <link name="${tf_prefix}gripper_jaw2_link" />
+      <joint name="${tf_prefix}gripper_jaw1_joint" />
+      <passive_joint name="${tf_prefix}gripper_jaw2_joint" />
     </group>
     <group_state name="open" group="ar_gripper">
-      <joint name="${prefix}gripper_jaw1_joint" value="-0.012" />
+      <joint name="${tf_prefix}gripper_jaw1_joint" value="-0.012" />
     </group_state>
     <group_state name="closed" group="ar_gripper">
-      <joint name="${prefix}gripper_jaw1_joint" value="-0.001" />
+      <joint name="${tf_prefix}gripper_jaw1_joint" value="-0.001" />
     </group_state>
-    <disable_collisions link1="${prefix}gripper_base_link" link2="${prefix}gripper_jaw1_link" reason="Adjacent" />
-    <disable_collisions link1="${prefix}gripper_base_link" link2="${prefix}gripper_jaw2_link" reason="Adjacent" />
-    <disable_collisions link1="${prefix}gripper_jaw1_link" link2="${prefix}gripper_jaw2_link" reason="Default" />
-    <disable_collisions link1="${prefix}link_6" link2="${prefix}gripper_base_link" reason="Adjacent" />
-    <disable_collisions link1="${prefix}link_5" link2="${prefix}gripper_base_link" reason="Adjacent" />
+    <disable_collisions link1="${tf_prefix}gripper_base_link" link2="${tf_prefix}gripper_jaw1_link" reason="Adjacent" />
+    <disable_collisions link1="${tf_prefix}gripper_base_link" link2="${tf_prefix}gripper_jaw2_link" reason="Adjacent" />
+    <disable_collisions link1="${tf_prefix}gripper_jaw1_link" link2="${tf_prefix}gripper_jaw2_link" reason="Default" />
+    <disable_collisions link1="${tf_prefix}link_6" link2="${tf_prefix}gripper_base_link" reason="Adjacent" />
+    <disable_collisions link1="${tf_prefix}link_5" link2="${tf_prefix}gripper_base_link" reason="Adjacent" />
   </xacro:macro>
 </robot>

File: annin_ar4_moveit_config/srdf/ar_macro.srdf.xacro (robot description, xacro)
@@ -5,39 +5,39 @@
 -->
 <robot xmlns:xacro="http://wiki.ros.org/xacro">
-  <xacro:macro name="ar_srdf" params="prefix">
+  <xacro:macro name="ar_srdf" params="tf_prefix">
     <group name="ar_manipulator">
-      <joint name="${prefix}joint_1" />
-      <joint name="${prefix}joint_2" />
-      <joint name="${prefix}joint_3" />
-      <joint name="${prefix}joint_4" />
-      <joint name="${prefix}joint_5" />
-      <joint name="${prefix}joint_6" />
-      <joint name="${prefix}ee_joint"/>
+      <joint name="${tf_prefix}joint_1" />
+      <joint name="${tf_prefix}joint_2" />
+      <joint name="${tf_prefix}joint_3" />
+      <joint name="${tf_prefix}joint_4" />
+      <joint name="${tf_prefix}joint_5" />
+      <joint name="${tf_prefix}joint_6" />
+      <joint name="${tf_prefix}ee_joint"/>
     </group>
     <group_state name="home" group="ar_manipulator">
-      <joint name="${prefix}joint_1" value="0" />
-      <joint name="${prefix}joint_2" value="0" />
-      <joint name="${prefix}joint_3" value="0" />
-      <joint name="${prefix}joint_4" value="0" />
-      <joint name="${prefix}joint_5" value="0" />
-      <joint name="${prefix}joint_6" value="0" />
+      <joint name="${tf_prefix}joint_1" value="0" />
+      <joint name="${tf_prefix}joint_2" value="0" />
+      <joint name="${tf_prefix}joint_3" value="0" />
+      <joint name="${tf_prefix}joint_4" value="0" />
+      <joint name="${tf_prefix}joint_5" value="0" />
+      <joint name="${tf_prefix}joint_6" value="0" />
     </group_state>
     <group_state name="upright" group="ar_manipulator">
-      <joint name="${prefix}joint_1" value="0" />
-      <joint name="${prefix}joint_2" value="-0.087" />
-      <joint name="${prefix}joint_3" value="-1.4" />
-      <joint name="${prefix}joint_4" value="0" />
-      <joint name="${prefix}joint_5" value="0" />
-      <joint name="${prefix}joint_6" value="0" />
+      <joint name="${tf_prefix}joint_1" value="0" />
+      <joint name="${tf_prefix}joint_2" value="-0.087" />
+      <joint name="${tf_prefix}joint_3" value="-1.4" />
+      <joint name="${tf_prefix}joint_4" value="0" />
+      <joint name="${tf_prefix}joint_5" value="0" />
+      <joint name="${tf_prefix}joint_6" value="0" />
     </group_state>
-    <disable_collisions link1="${prefix}base_link" link2="${prefix}link_1" reason="Adjacent" />
-    <disable_collisions link1="${prefix}link_1" link2="${prefix}link_2" reason="Adjacent" />
-    <disable_collisions link1="${prefix}link_1" link2="${prefix}link_3" reason="Never" />
-    <disable_collisions link1="${prefix}link_2" link2="${prefix}link_3" reason="Adjacent" />
-    <disable_collisions link1="${prefix}link_3" link2="${prefix}link_4" reason="Adjacent" />
-    <disable_collisions link1="${prefix}link_3" link2="${prefix}link_5" reason="Never" />
-    <disable_collisions link1="${prefix}link_3" link2="${prefix}link_6" reason="Never" />
-    <disable_collisions link1="${prefix}link_4" link2="${prefix}link_5" reason="Adjacent" />
-    <disable_collisions link1="${prefix}link_5" link2="${prefix}link_6" reason="Adjacent" />
+    <disable_collisions link1="${tf_prefix}base_link" link2="${tf_prefix}link_1" reason="Adjacent" />
+    <disable_collisions link1="${tf_prefix}link_1" link2="${tf_prefix}link_2" reason="Adjacent" />
+    <disable_collisions link1="${tf_prefix}link_1" link2="${tf_prefix}link_3" reason="Never" />
+    <disable_collisions link1="${tf_prefix}link_2" link2="${tf_prefix}link_3" reason="Adjacent" />
+    <disable_collisions link1="${tf_prefix}link_3" link2="${tf_prefix}link_4" reason="Adjacent" />
+    <disable_collisions link1="${tf_prefix}link_3" link2="${tf_prefix}link_5" reason="Never" />
+    <disable_collisions link1="${tf_prefix}link_3" link2="${tf_prefix}link_6" reason="Never" />
+    <disable_collisions link1="${tf_prefix}link_4" link2="${tf_prefix}link_5" reason="Adjacent" />
+    <disable_collisions link1="${tf_prefix}link_5" link2="${tf_prefix}link_6" reason="Adjacent" />
   </xacro:macro>
 </robot>
